File: sch/carrier/_autosave-CM4.kicad_sch (KiCad schematic)
At the start: 4 parts

Commit message: hhhhhhhhhhhhhhhhh
Changed lines of the file:
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@@
     (effects (font (size 1.27 1.27)) (justify left))
   )
-  (hierarchical_label "DPAD_DOWN" (shape input) (at 139.7 86.36 0)
+  (hierarchical_label "DPAD_DOWN" (shape input) (at 142.24 80.01 0)
     (effects (font (size 1.27 1.27)) (justify left))
   )
-  (hierarchical_label "DPAD_LEFT" (shape input) (at 139.7 96.52 0)
+  (hierarchical_label "DPAD_LEFT" (shape input) (at 142.24 90.17 0)
     (effects (font (size 1.27 1.27)) (justify left))
   )
-  (hierarchical_label "BTN_A" (shape input) (at 139.7 109.855 0)
+  (hierarchical_label "BTN_A" (shape input) (at 142.24 103.505 0)
     (effects (font (size 1.27 1.27)) (justify left))
   )
-  (hierarchical_label "DPAD_UP" (shape input) (at 140.97 81.28 0)
+  (hierarchical_label "DPAD_UP" (shape input) (at 143.51 74.93 0)
     (effects (font (size 1.27 1.27)) (justify left))
   )
-  (hierarchical_label "DPAD_RIGHT" (shape input) (at 140.97 103.505 0)
+  (hierarchical_label "DPAD_RIGHT" (shape input) (at 143.51 97.155 0)
     (effects (font (size 1.27 1.27)) (justify left))
   )
-  (hierarchical_label "BTN_B" (shape input) (at 141.605 118.11 0)
+  (hierarchical_label "BTN_B" (shape input) (at 144.145 111.76 0)
     (effects (font (size 1.27 1.27)) (justify left))
   )
