File: sch/carrier/carrier.kicad_pcb (KiCad board)
At the start: 0 parts

Commit message: put some stuff on the pcb - it is going to kill me trying to get all on
Parts:
- added C1: 0.1uF, Capacitor_SMD:C_0504_1310Metric_Pad0.83x1.28mm_HandSolder, F.Cu at (38.2, 45.5)
- added C2: 0.1uF, Capacitor_SMD:C_0504_1310Metric_Pad0.83x1.28mm_HandSolder, F.Cu at (59.6, 120.9)
- added C3: 0.1uF, Capacitor_SMD:C_0504_1310Metric_Pad0.83x1.28mm_HandSolder, F.Cu at (44.4, 135.0)
- added C4: 0.1uF, Capacitor_SMD:C_0504_1310Metric_Pad0.83x1.28mm_HandSolder, F.Cu at (71.8, 120.5)
- added C5: 0.1uF, Capacitor_SMD:C_0504_1310Metric_Pad0.83x1.28mm_HandSolder, F.Cu at (67.0, 125.8)
- added C6: 0.1uF, Capacitor_SMD:C_0504_1310Metric_Pad0.83x1.28mm_HandSolder, F.Cu at (64.3, 116.8)
- added D1: LED, LED_SMD:LED_0805_2012Metric_Pad1.15x1.40mm_HandSolder, F.Cu at (134.0, 94.4)
- added D2: 5.1v, Diode_THT:D_DO-41_SOD81_P7.62mm_Horizontal, F.Cu at (257.8, 38.7)
- added J1: 1054500101, MOLEXC:Molex-1054500101-MFG, F.Cu at (55.0, 30.8)
- added J2: 1054500101, MOLEXC:Molex-1054500101-MFG, F.Cu at (72.2, 30.7)
- added J3: 52271-0879, MOLEXZIF:Molex-52271-0879-Manufacturer_Recommended, F.Cu at (156.0, 99.2)
- added Module0: ComputeModule4-CM4, CM4IO:Raspberry-Pi-4-Compute-Module, F.Cu at (111.0, 73.2)
- added Q1: BC557, Package_TO_SOT_THT:TO-92_Inline_Horizontal1, F.Cu at (269.1, 38.1)
- added Q2: BC557, Package_TO_SOT_THT:TO-92_Inline_Horizontal1, F.Cu at (257.7, 42.3)
- added R1: 1k, Resistor_SMD:R_0805_2012Metric_Pad1.20x1.40mm_HandSolder, F.Cu at (33.8, 45.5)
- added R10: 10k, Resistor_SMD:R_0805_2012Metric_Pad1.20x1.40mm_HandSolder, F.Cu at (56.2, 114.0)
- added R11: 1k, Resistor_SMD:R_0805_2012Metric_Pad1.20x1.40mm_HandSolder, F.Cu at (42.0, 130.4)
- added R12: 10k, Resistor_SMD:R_0805_2012Metric_Pad1.20x1.40mm_HandSolder, F.Cu at (37.2, 130.4)
- added R13: 220, Resistor_SMD:R_0805_2012Metric_Pad1.20x1.40mm_HandSolder, F.Cu at (175.3, 38.0)
- added R14: 5.1k, Resistor_SMD:R_0805_2012Metric_Pad1.20x1.40mm_HandSolder, F.Cu at (264.5, 45.2)
- added R15: 5.1k, Resistor_SMD:R_0805_2012Metric_Pad1.20x1.40mm_HandSolder, F.Cu at (258.3, 63.8)
- added R16: 2k, Resistor_SMD:R_0805_2012Metric_Pad1.20x1.40mm_HandSolder, F.Cu at (264.5, 42.3)
- added R17: 1k, Resistor_SMD:R_0805_2012Metric_Pad1.20x1.40mm_HandSolder, F.Cu at (264.5, 49.2)
- added R18: 6.2k, Resistor_SMD:R_0805_2012Metric_Pad1.20x1.40mm_HandSolder, F.Cu at (275.8, 38.0)
- added R19: 33, Resistor_SMD:R_0805_2012Metric_Pad1.20x1.40mm_HandSolder, F.Cu at (175.7, 90.5)
- added R2: 10k, Resistor_SMD:R_0805_2012Metric_Pad1.20x1.40mm_HandSolder, F.Cu at (33.8, 42.2)
- added R3: 1k, Resistor_SMD:R_0805_2012Metric_Pad1.20x1.40mm_HandSolder, F.Cu at (51.5, 125.2)
- added R4: 1k, Resistor_SMD:R_0805_2012Metric_Pad1.20x1.40mm_HandSolder, F.Cu at (56.2, 117.0)
- added R5: 10k, Resistor_SMD:R_0805_2012Metric_Pad1.20x1.40mm_HandSolder, F.Cu at (51.5, 122.2)
- added R6: 10k, Resistor_SMD:R_0805_2012Metric_Pad1.20x1.40mm_HandSolder, F.Cu at (46.7, 128.1)
- added R7: 1k, Resistor_SMD:R_0805_2012Metric_Pad1.20x1.40mm_HandSolder, F.Cu at (46.7, 125.2)
- added R8: 10k, Resistor_SMD:R_0805_2012Metric_Pad1.20x1.40mm_HandSolder, F.Cu at (123.0, 106.2)
- added R9: 1k, Resistor_SMD:R_0805_2012Metric_Pad1.20x1.40mm_HandSolder, F.Cu at (46.7, 122.2)
- added SW1: SKRRACE010, eec:ALPS-SKRRACE010-0-0-MFG, F.Cu at (35.8, 61.8)
- added SW2: SKRRACE010, eec:ALPS-SKRRACE010-0-0-MFG, F.Cu at (42.8, 54.5)
- added SW3: SKRRACE010, eec:ALPS-SKRRACE010-0-0-MFG, F.Cu at (42.8, 69.0)
- added SW4: SKRRACE010, eec:ALPS-SKRRACE010-0-0-MFG, F.Cu at (49.5, 61.8)
- added SW5: SKRRACE010, eec:ALPS-SKRRACE010-0-0-MFG, F.Cu at (47.0, 83.2)
- added SW6: SKRRACE010, eec:ALPS-SKRRACE010-0-0-MFG, F.Cu at (37.0, 93.2)
- added TP1: GND, TestPoint:TestPoint_Pad_2.0x2.0mm, F.Cu at (166.3, 97.8)
- added TP10: A, TestPoint:TestPoint_Pad_2.0x2.0mm, F.Cu at (55.9, 120.5)
- added TP11: B, TestPoint:TestPoint_Pad_2.0x2.0mm, F.Cu at (60.6, 117.5)
- added TP2: Activity, TestPoint:TestPoint_Pad_2.0x2.0mm, F.Cu at (133.6, 98.0)
- added TP6: UP, TestPoint:TestPoint_Pad_2.0x2.0mm, F.Cu at (55.9, 124.5)
- added TP7: DOWN, TestPoint:TestPoint_Pad_2.0x2.0mm, F.Cu at (62.6, 129.4)
- added TP8: LEFT, TestPoint:TestPoint_Pad_2.0x2.0mm, F.Cu at (46.4, 131.6)
- added TP9: RIGHT, TestPoint:TestPoint_Pad_2.0x2.0mm, F.Cu at (51.1, 128.7)
- added U1: SN74HC14N, TI74HC14N:Texas_Instruments-R_R-PDIP-T14-0-0-0, F.Cu at (-3.25, 54.5)
- added U2: ER-CON40HT-1, ER-CON40HT-1:ER-CON40HT-1, F.Cu at (160.5, 91.8)
Other:
- board outline added: 77.2 x 77.3 mm
- copper layers 0 -> 2
