File: sch/carrier/carrier.kicad_pcb (KiCad board)
At the start: 2 copper layers, 77.2 x 77.3 mm, 49 parts, among them J1 1054500101, J2 1054500101, J3 52271-0879, Q1 BC557, Q2 BC557, SW1 SKRRACE010, SW2 SKRRACE010, SW3 SKRRACE010, SW4 SKRRACE010, SW5 SKRRACE010, SW6 SKRRACE010, U1 SN74HC14N, U2 ER-CON40HT-1

Commit message: holy shit i hate chargers
Parts:
- moved Q2 95.4 mm to (163.5, 57.1)
- moved D2 95.4 mm to (163.6, 53.5)
- moved R14 95.4 mm to (170.2, 60.0)
- moved R15 95.4 mm to (164.1, 78.5)
- moved R16 95.4 mm to (170.2, 57.0)
- moved R17 95.4 mm to (170.2, 64.0)
- moved R18 95.4 mm to (181.6, 52.8)
- moved Q1 95.4 mm to (174.9, 52.9)
- moved U1 58.4 mm to (40.5, 93.2), turned to 0 degrees
- moved SW6 55.7 mm to (89.2, 74.0)
- moved SW5 32.9 mm to (79.5, 78.2)
- moved R8 19.7 mm to (138.8, 94.5)
- moved TP2 1.63 mm to (134.2, 99.5)

Commit message: pcb time?
Parts:
- removed Q1, Q2: BC557, Package_TO_SOT_THT:TO-92_Inline_Horizontal1
- added C10: 0.1uF, Capacitor_SMD:C_0402_1005Metric_Pad0.74x0.62mm_HandSolder, F.Cu at (217.0, 49.6)
- added C11: 0.1uF, Capacitor_SMD:C_0402_1005Metric_Pad0.74x0.62mm_HandSolder, F.Cu at (247.3, 19.3)
- added C12: 0.1uF, Capacitor_SMD:C_0402_1005Metric_Pad0.74x0.62mm_HandSolder, F.Cu at (220.2, 49.6)
- added C13: 0.1uF, Capacitor_SMD:C_0402_1005Metric_Pad0.74x0.62mm_HandSolder, F.Cu at (247.3, 21.3)
- added C14: 0.1uF, Capacitor_SMD:C_0402_1005Metric_Pad0.74x0.62mm_HandSolder, F.Cu at (227.1, 37.4)
- added C15: 10uF, Capacitor_SMD:C_01005_0402Metric_Pad0.57x0.30mm_HandSolder, F.Cu at (215.6, 95.7)
- added C16: 100nF, Capacitor_SMD:C_0603_1608Metric_Pad1.08x0.95mm_HandSolder, F.Cu at (218.3, 89.5)
- added C17: 100nf, Capacitor_SMD:C_0402_1005Metric_Pad0.74x0.62mm_HandSolder, F.Cu at (211.1, 99.8)
- added C18: 22u, Capacitor_SMD:C_01005_0402Metric_Pad0.57x0.30mm_HandSolder, F.Cu at (215.6, 94.1)
- added C19: 10u, Capacitor_SMD:C_01005_0402Metric_Pad0.57x0.30mm_HandSolder, F.Cu at (219.9, 91.5)
- added C20: 10u, Capacitor_SMD:C_01005_0402Metric_Pad0.57x0.30mm_HandSolder, F.Cu at (206.4, 104.9)
- added C21: 1uF, Capacitor_SMD:C_0603_1608Metric_Pad1.08x0.95mm_HandSolder, F.Cu at (118.6, 89.0)
- added C22: 0.47uF, Capacitor_SMD:C_0603_1608Metric_Pad1.08x0.95mm_HandSolder, F.Cu at (116.7, 93.7)
- added C23: 33n, Capacitor_SMD:C_0603_1608Metric_Pad1.08x0.95mm_HandSolder, F.Cu at (158.6, 43.1)
- added C24: 10u, Capacitor_SMD:C_0603_1608Metric_Pad1.08x0.95mm_HandSolder, F.Cu at (117.1, 80.4)
- added C25: 10u, Capacitor_SMD:C_01005_0402Metric_Pad0.57x0.30mm_HandSolder, F.Cu at (206.4, 103.2)
- added C26: 10u, Capacitor_SMD:C_01005_0402Metric_Pad0.57x0.30mm_HandSolder, F.Cu at (221.8, 87.5)
- added C7: 33n, Capacitor_SMD:C_0603_1608Metric_Pad1.08x0.95mm_HandSolder, F.Cu at (122.4, 75.9)
- added C8: 10uF, Capacitor_SMD:C_0603_1608Metric_Pad1.08x0.95mm_HandSolder, F.Cu at (153.7, 47.5)
- added C9: 10u, Capacitor_SMD:C_0603_1608Metric_Pad1.08x0.95mm_HandSolder, F.Cu at (121.5, 80.4)
- added D3: LED, LED_SMD:LED_0805_2012Metric_Pad1.15x1.40mm_HandSolder, F.Cu at (207.6, 93.4)
- added D4: BAV99, Package_TO_SOT_SMD:SOT-23, F.Cu at (153.9, 44.0)
- added D5: BAV99, Package_TO_SOT_SMD:SOT-23, F.Cu at (117.7, 76.9)
- added D6: 824011, tvs:SOT95P280X145-5N, F.Cu at (156.1, 108.9)
- added J4: HDMI_D_1.4, Connector_HDMI:HDMI_Micro-D_Molex_46765-1x01, F.Cu at (170.4, 94.0)
- added J5: USB_C_Receptacle_USB2.0, Connector_USB:USB_C_Receptacle_JAE_DX07S016JA1R1500, F.Cu at (159.5, 92.6)
- added J6: 52271-0879, MOLEXZIF:Molex-52271-0879-Manufacturer_Recommended, F.Cu at (261.0, 28.5)
- added J7: AudioJack3_Switch, audio:audio, F.Cu at (156.0, 25.8)
- added L1: 6.8uH, Inductor_SMD:L_Wuerth_WE-PD-Typ-M-Typ-S_Handsoldering, F.Cu at (212.0, 81.2)
- added NT1: NetTie, NetTie:NetTie-2_SMD_Pad0.5mm, F.Cu at (225.3, 85.7)
- added R22: 12k 1%, Resistor_SMD:R_0402_1005Metric_Pad0.72x0.64mm_HandSolder, F.Cu at (162.4, 42.8)
- added R23: 270, Resistor_SMD:R_0603_1608Metric_Pad0.98x0.95mm_HandSolder, F.Cu at (158.0, 47.5)
- added R24: 150, Resistor_SMD:R_0603_1608Metric_Pad0.98x0.95mm_HandSolder, F.Cu at (153.7, 50.0)
- added R25: 0, Resistor_SMD:R_0603_1608Metric_Pad0.98x0.95mm_HandSolder, F.Cu at (117.1, 82.9)
- added R26: 1k, Resistor_SMD:R_0402_1005Metric_Pad0.72x0.64mm_HandSolder, F.Cu at (217.0, 45.6)
- added R27: 10k, Resistor_SMD:R_0402_1005Metric_Pad0.72x0.64mm_HandSolder, F.Cu at (223.8, 41.4)
- added R28: 1k, Resistor_SMD:R_0402_1005Metric_Pad0.72x0.64mm_HandSolder, F.Cu at (230.3, 33.5)
- added R29: 1k, Resistor_SMD:R_0402_1005Metric_Pad0.72x0.64mm_HandSolder, F.Cu at (212.7, 54.3)
- added R30: 10k, Resistor_SMD:R_0402_1005Metric_Pad0.72x0.64mm_HandSolder, F.Cu at (234.1, 29.1)
- added R31: 10k, Resistor_SMD:R_0402_1005Metric_Pad0.72x0.64mm_HandSolder, F.Cu at (206.8, 64.5)
- added R32: 1k, Resistor_SMD:R_0402_1005Metric_Pad0.72x0.64mm_HandSolder, F.Cu at (234.7, 31.1)
- added R33: 10k, Resistor_SMD:R_0402_1005Metric_Pad0.72x0.64mm_HandSolder, F.Cu at (223.8, 35.4)
- added R34: 1k, Resistor_SMD:R_0402_1005Metric_Pad0.72x0.64mm_HandSolder, F.Cu at (220.2, 43.6)
- added R35: 10k, Resistor_SMD:R_0402_1005Metric_Pad0.72x0.64mm_HandSolder, F.Cu at (244.1, 19.3)
- added R36: 1k, Resistor_SMD:R_0402_1005Metric_Pad0.72x0.64mm_HandSolder, F.Cu at (229.1, 80.2)
- added R37: 9k, Resistor_SMD:R_0402_1005Metric_Pad0.72x0.64mm_HandSolder, F.Cu at (211.1, 97.9)
- added R38: 1.3k, Resistor_SMD:R_0402_1005Metric_Pad0.72x0.64mm_HandSolder, F.Cu at (233.9, 77.7)
- added R39: 1k, Resistor_SMD:R_0402_1005Metric_Pad0.72x0.64mm_HandSolder, F.Cu at (222.1, 85.7)
- added R40: 10.5k, Resistor_SMD:R_0603_1608Metric_Pad0.98x0.95mm_HandSolder, F.Cu at (221.0, 81.0)
- added R41: 10.5k, Resistor_SMD:R_0603_1608Metric_Pad0.98x0.95mm_HandSolder, F.Cu at (216.5, 92.0)
- added R42: 16k, Resistor_SMD:R_0603_1608Metric_Pad0.98x0.95mm_HandSolder, F.Cu at (214.0, 87.0)
- added R43: 10k, Resistor_SMD:R_0603_1608Metric_Pad0.98x0.95mm_HandSolder, F.Cu at (218.3, 87.0)
- added R44: 3k, Resistor_SMD:R_0603_1608Metric_Pad0.98x0.95mm_HandSolder, F.Cu at (207.3, 101.2)
- added R45: 55.2k, Resistor_SMD:R_0603_1608Metric_Pad0.98x0.95mm_HandSolder, F.Cu at (221.0, 83.5)
- added R46: 120k, Resistor_SMD:R_0603_1608Metric_Pad0.98x0.95mm_HandSolder, F.Cu at (214.0, 89.5)
- added R47: 20m, Resistor_SMD:R_0603_1608Metric_Pad0.98x0.95mm_HandSolder, F.Cu at (212.1, 95.6)
- added R48: 2.49k, Resistor_SMD:R_0603_1608Metric_Pad0.98x0.95mm_HandSolder, F.Cu at (212.1, 93.1)
- added R49: 2.49k, Resistor_SMD:R_0603_1608Metric_Pad0.98x0.95mm_HandSolder, F.Cu at (230.1, 77.9)
- added R50: 2.49k, Resistor_SMD:R_0603_1608Metric_Pad0.98x0.95mm_HandSolder, F.Cu at (207.3, 98.7)
- added R51: 10.5k, Resistor_SMD:R_0603_1608Metric_Pad0.98x0.95mm_HandSolder, F.Cu at (225.3, 81.0)
- added R52: 10.5k, Resistor_SMD:R_0603_1608Metric_Pad0.98x0.95mm_HandSolder, F.Cu at (225.3, 83.5)
- added R53: 10.5k, Resistor_SMD:R_0603_1608Metric_Pad0.98x0.95mm_HandSolder, F.Cu at (207.3, 96.2)
- added R54: 10.5k, Resistor_SMD:R_0603_1608Metric_Pad0.98x0.95mm_HandSolder, F.Cu at (225.8, 77.9)
- added R55: 0, Resistor_SMD:R_0603_1608Metric_Pad0.98x0.95mm_HandSolder, F.Cu at (167.7, 101.6)
- added R56: 5.1k, Resistor_SMD:R_0805_2012Metric_Pad1.20x1.40mm_HandSolder, F.Cu at (155.9, 112.6)
- added R57: 5.1k, Resistor_SMD:R_0805_2012Metric_Pad1.20x1.40mm_HandSolder, F.Cu at (167.9, 98.8)
- added R58: 0, Resistor_SMD:R_0603_1608Metric_Pad0.98x0.95mm_HandSolder, F.Cu at (155.7, 115.3)
- added R59: 10m, Resistor_SMD:R_0603_1608Metric_Pad0.98x0.95mm_HandSolder, F.Cu at (112.3, 93.7)
- added R61: 10k, Resistor_SMD:R_0402_1005Metric_Pad0.72x0.64mm_HandSolder, F.Cu at (118.0, 91.2)
- added R63: 10k, Resistor_SMD:R_0603_1608Metric_Pad0.98x0.95mm_HandSolder, F.Cu at (112.3, 96.2)
- added SW10: SKRBAAE010, eec:SKRBAAE010, F.Cu at (219.3, 33.2)
- added SW11: SW_Push, sw:TE_Connectivity-1-1825027-1-0-0-Recommended_Land_Pattern_, F.Cu at (221.4, 25.4)
- added SW12: SW_DIP_x04, dipswitch:CHS04TA1, F.Cu at (237.6, 23.2)
- added SW7: SKRBAAE010, eec:SKRBAAE010, F.Cu at (229.5, 19.0)
- added SW8: SKRBAAE010, eec:SKRBAAE010, F.Cu at (208.1, 54.1)
- added SW9: SW_Push, sw:TE_Connectivity-1-1825027-1-0-0-Recommended_Land_Pattern_, F.Cu at (210.3, 46.3)
- added TP12: MOSI, TestPoint:TestPoint_Pad_1.0x1.0mm, F.Cu at (129.3, 76.2)
- added TP13: +3.3V, TestPoint:TestPoint_Pad_1.0x1.0mm, F.Cu at (153.0, 52.8)
- added TP14: BKL, TestPoint:TestPoint_Pad_1.0x1.0mm, F.Cu at (209.9, 65.0)
- added TP15: SEL, TestPoint:TestPoint_Pad_1.0x1.0mm, F.Cu at (212.6, 59.9)
- added TP16: STR, TestPoint:TestPoint_Pad_1.0x1.0mm, F.Cu at (227.0, 41.9)
- added TP17: L, TestPoint:TestPoint_Pad_1.0x1.0mm, F.Cu at (212.6, 56.9)
- added TP18: R, TestPoint:TestPoint_Pad_1.0x1.0mm, F.Cu at (233.5, 36.0)
- added TP19: +5v Output, TestPoint:TestPoint_Pad_1.0x1.0mm, F.Cu at (229.0, 82.7)
- added TP20: GND, TestPoint:TestPoint_Pad_1.0x1.0mm, F.Cu at (270.8, 26.6)
- added TP21: CEO_N, TestPoint:TestPoint_Pad_1.0x1.0mm, F.Cu at (279.8, 22.8)
- added TP22: SCLK, TestPoint:TestPoint_Pad_1.0x1.0mm, F.Cu at (254.2, 40.5)
- added TP23: MISO, TestPoint:TestPoint_Pad_1.0x1.0mm, F.Cu at (273.9, 26.6)
- added TP24: MOSI, TestPoint:TestPoint_Pad_1.0x1.0mm, F.Cu at (257.2, 37.5)
- added TP25: +3.3V, TestPoint:TestPoint_Pad_1.0x1.0mm, F.Cu at (254.2, 37.5)
- added TP26: BATT+, TestPoint:TestPoint_Pad_1.0x1.0mm, F.Cu at (122.3, 89.2)
- added TP27: AUXR, TestPoint:TestPoint_Pad_1.0x1.0mm, F.Cu at (188.3, 19.8)
- added TP28: AUXL, TestPoint:TestPoint_Pad_1.0x1.0mm, F.Cu at (125.2, 78.7)
- added TP3: CEO_N, TestPoint:TestPoint_Pad_1.0x1.0mm, F.Cu at (120.8, 83.1)
- added TP4: SCLK, TestPoint:TestPoint_Pad_1.0x1.0mm, F.Cu at (125.2, 81.7)
- added TP5: MISO, TestPoint:TestPoint_Pad_1.0x1.0mm, F.Cu at (162.3, 45.3)
- added U3: MP2636GR-P, mp2636:IC_MP2636GR-P, F.Cu at (208.7, 88.8)
- added U4: AP22814AW5, Package_TO_SOT_SMD:SOT-23-5, F.Cu at (112.7, 76.9)
- added U5: BQ27441DRZR-G1B, Package_SON:Texas_S-PDSO-N12, F.Cu at (113.3, 90.1)
- C1, C2, C3, C4, C5, C6: footprint Capacitor_SMD:C_0504_1310Metric_Pad0.83x1.28mm_HandSolder -> Capacitor_SMD:C_0402_1005Metric_Pad0.74x0.62mm_HandSolder
- D2: value 5.1v -> LED; footprint Diode_THT:D_DO-41_SOD81_P7.62mm_Horizontal -> LED_SMD:LED_0805_2012Metric_Pad1.15x1.40mm_HandSolder
- J1: value 1054500101 -> USB_C_Receptacle_USB2.0; footprint MOLEXC:Molex-1054500101-MFG -> Connector_USB:USB_C_Receptacle_JAE_DX07S016JA1R1500
- J2: value 1054500101 -> 52271-0879; footprint MOLEXC:Molex-1054500101-MFG -> MOLEXZIF:Molex-52271-0879-Manufacturer_Recommended
- J3: value 52271-0879 -> Micro_SD_Card; footprint MOLEXZIF:Molex-52271-0879-Manufacturer_Recommended -> sdcard:HRS_DM3CS-SF
- R1, R10, R11, R12, R2, R3, R4, R5, R6, R7, R8, R9: footprint Resistor_SMD:R_0805_2012Metric_Pad1.20x1.40mm_HandSolder -> Resistor_SMD:R_0402_1005Metric_Pad0.72x0.64mm_HandSolder
- R13: footprint Resistor_SMD:R_0805_2012Metric_Pad1.20x1.40mm_HandSolder -> Capacitor_SMD:C_0402_1005Metric_Pad0.74x0.62mm_HandSolder
- R14: value 5.1k -> 270; footprint Resistor_SMD:R_0805_2012Metric_Pad1.20x1.40mm_HandSolder -> Resistor_SMD:R_0603_1608Metric_Pad0.98x0.95mm_HandSolder
- R15: value 5.1k -> 0; footprint Resistor_SMD:R_0805_2012Metric_Pad1.20x1.40mm_HandSolder -> Resistor_SMD:R_0603_1608Metric_Pad0.98x0.95mm_HandSolder
- R16: value 2k -> 56k
- R17: value 1k -> 56k
- R18: value 6.2k -> 150; footprint Resistor_SMD:R_0805_2012Metric_Pad1.20x1.40mm_HandSolder -> Resistor_SMD:R_0603_1608Metric_Pad0.98x0.95mm_HandSolder
- TP1, TP10, TP11, TP2, TP6, TP7, TP8, TP9: footprint TestPoint:TestPoint_Pad_2.0x2.0mm -> TestPoint:TestPoint_Pad_1.0x1.0mm
- moved C3 227.9 mm to (244.1, 25.2)
- moved R12 215.1 mm to (228.2, 31.5)
- moved C2 209.6 mm to (244.1, 21.3)
- moved TP6 207.9 mm to (240.9, 29.6)
- moved TP8 206.3 mm to (230.2, 38.0)
- moved R7 205.2 mm to (228.2, 29.5)
- moved R6 198.1 mm to (223.8, 39.4)
- moved R2 198.0 mm to (231.4, 31.1)
- moved C4 197.9 mm to (244.1, 23.2)
- moved TP11 196.9 mm to (237.8, 31.6)
- moved R5 193.9 mm to (223.8, 33.5)
- moved R11 193.7 mm to (217.0, 47.6)
- moved R1 193.6 mm to (227.1, 35.4)
- moved R3 193.4 mm to (223.8, 37.4)
- moved R10 188.9 mm to (227.1, 33.5)
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Connections:
- C1 pad 1: /Buttons/__DP_L -> GND
- C1 pad 2: GND -> /Buttons/__DP_L
- D2 pad 2: GND -> Net-(D2-Pad2)
- J1 pad A4: Net-(J1-PadA4) -> /+5v
- J1 pad A6: unconnected-(J1-PadA6) -> /Connectors/USB2_D+
- J1 pad A7: unconnected-(J1-PadA7) -> /Connectors/USB2_D-
- J1 pad A9: Net-(J1-PadA4) -> /+5v
- J1 pad B4: Net-(J1-PadA4) -> /+5v
- J1 pad B5: Net-(J1-PadB5) -> Net-(R17-Pad2)
- J1 pad B6: unconnected-(J1-PadB6) -> /Connectors/USB2_D+
- J1 pad B7: unconnected-(J1-PadB7) -> /Connectors/USB2_D-
- J1 pad B9: Net-(J1-PadA4) -> /+5v
- J2 pad 1: GND -> /+3.3v
- J2 pad 2: GND -> /+3.3v
- J2 pad 3: GND -> /CM4/SCREEN_MOSI
- J2 pad 4: GND -> /CM4/SCREEN_MISO
- J3 pad 1: /display board/+3.3v -> /CM4/SD_DAT2
- J3 pad 2: /display board/SPI0_MOSI -> /CM4/SD_DAT3
- J3 pad 3: /display board/SPI_MISO -> /CM4/SD_CMD
- J3 pad 4: unconnected-(J3-Pad4) -> /CM4/SD_PWR
- J3 pad 5: /display board/SPI0_SCLK -> /CM4/SD_CLK
- J3 pad 6: /display board/SPI0_CE0_N -> GND
- J3 pad 7: unconnected-(J3-Pad7) -> /CM4/SD_DAT0
- J3 pad 8: GND -> /CM4/SD_DAT1
- Module0 pad 103: /connectors/USB2_D- -> /Connectors/USB2_D-
- Module0 pad 105: /connectors/USB2_D+ -> /Connectors/USB2_D+
- Module0 pad 151: unconnected-(Module0-Pad151) -> /Connectors/HDMI_CEC
- Module0 pad 153: unconnected-(Module0-Pad153) -> /Connectors/HDMI_HP
- Module0 pad 170: unconnected-(Module0-Pad170) -> /Connectors/TX2_P
- Module0 pad 172: unconnected-(Module0-Pad172) -> /Connectors/TX2_N
- Module0 pad 176: unconnected-(Module0-Pad176) -> /Connectors/TX1_P
- Module0 pad 178: unconnected-(Module0-Pad178) -> /Connectors/TX1_N
- Module0 pad 182: unconnected-(Module0-Pad182) -> /Connectors/TX0_P
- Module0 pad 184: unconnected-(Module0-Pad184) -> /Connectors/TX0_N
- Module0 pad 188: unconnected-(Module0-Pad188) -> /Connectors/CLK_P
- Module0 pad 190: unconnected-(Module0-Pad190) -> /Connectors/CLK_N
- Module0 pad 199: unconnected-(Module0-Pad199) -> /Connectors/HDMI_SDA
- Module0 pad 200: unconnected-(Module0-Pad200) -> /Connectors/HDMI_SCL
- Module0 pad 25: unconnected-(Module0-Pad25) -> /Buttons/SELECT
- Module0 pad 26: unconnected-(Module0-Pad26) -> /CM4/AUX1
- Module0 pad 27: unconnected-(Module0-Pad27) -> /Buttons/BTN_BACKLIGHT
- Module0 pad 28: unconnected-(Module0-Pad28) -> /Buttons/DPAD_LEFT
- Module0 pad 29: unconnected-(Module0-Pad29) -> /Buttons/BTN_B
- Module0 pad 31: unconnected-(Module0-Pad31) -> /Buttons/DPAD_RIGHT
- Module0 pad 38: /CM4/SPI0_SCLK -> /CM4/SCREEN_SCLK
- Module0 pad 39: /CM4/SPI0_CE0_N -> /CM4/SCREEN_CE0_N
- Module0 pad 40: /CM4/SPI_MISO -> /CM4/SCREEN_MISO
- Module0 pad 41: unconnected-(Module0-Pad41) -> /Buttons/BTN_A
- Module0 pad 44: /CM4/SPI0_MOSI -> /CM4/SCREEN_MOSI
- Module0 pad 45: unconnected-(Module0-Pad45) -> /Buttons/START
- Module0 pad 46: unconnected-(Module0-Pad46) -> /Buttons/SHOULDER_L
- Module0 pad 47: unconnected-(Module0-Pad47) -> /Buttons/SHOULDER_R
- Module0 pad 49: unconnected-(Module0-Pad49) -> /CM4/AUX0
- Module0 pad 50: unconnected-(Module0-Pad50) -> /Buttons/DPAD_UP
- Module0 pad 55: unconnected-(Module0-Pad55) -> /Buttons/DPAD_DOWN
- Module0 pad 57: unconnected-(Module0-Pad57) -> /CM4/SD_CLK
- Module0 pad 61: unconnected-(Module0-Pad61) -> /CM4/SD_DAT3
- Module0 pad 62: unconnected-(Module0-Pad62) -> /CM4/SD_CMD
- Module0 pad 63: unconnected-(Module0-Pad63) -> /CM4/SD_DAT0
- Module0 pad 67: unconnected-(Module0-Pad67) -> /CM4/SD_DAT1
- Module0 pad 69: unconnected-(Module0-Pad69) -> /CM4/SD_DAT2
- Module0 pad 75: unconnected-(Module0-Pad75) -> /CM4/SD_PWR_ON
- Module0 pad 76: unconnected-(Module0-Pad76) -> /CM4/Reserved
- Module0 pad 80: unconnected-(Module0-Pad80) -> /Battery/FUEL_SCL
- Module0 pad 82: unconnected-(Module0-Pad82) -> /Battery/FUEL_SDA
- Module0 pad 99: unconnected-(Module0-Pad99) -> /Buttons/GLOBAL_EN
- R1 pad 1: Net-(R1-Pad1) -> Net-(SW1-Pad1)
- R14 pad 1: Net-(J1-PadA5) -> /CM4/AUX1
- R14 pad 2: GND -> Net-(C7-Pad2)
- R15 pad 1: Net-(J1-PadB5) -> Net-(J1-PadS1)
- R16 pad 1: Net-(J1-PadA4) -> /+5v
- R16 pad 2: Net-(D2-Pad1) -> Net-(J1-PadA5)
- R17 pad 1: Net-(D2-Pad1) -> /+5v
- R17 pad 2: Net-(Q1-Pad2) -> Net-(R17-Pad2)
- R18 pad 1: GND -> Net-(C7-Pad2)
- R18 pad 2: Net-(Q1-Pad3) -> GND
- R19 pad 1: /display board/+3.3v -> /Display board (SNAP OFF BOARD)/+3.3v
- R3 pad 1: Net-(R3-Pad1) -> Net-(SW2-Pad1)
- R4 pad 1: Net-(R4-Pad1) -> Net-(SW3-Pad1)
- R5 pad 1: unconnected-(R5-Pad1) -> /+3.3v
- R7 pad 1: Net-(R7-Pad1) -> Net-(SW4-Pad1)
- R9 pad 1: Net-(R9-Pad1) -> Net-(SW5-Pad1)
- SW1 pad 1: unconnected-(SW1-Pad1) -> Net-(SW1-Pad1)
- SW1 pad 3: Net-(R1-Pad1) -> Net-(SW1-Pad1)
- SW1 pad 4: unconnected-(SW1-Pad4) -> GND
- SW2 pad 1: unconnected-(SW2-Pad1) -> Net-(SW2-Pad1)
- SW2 pad 3: Net-(R3-Pad1) -> Net-(SW2-Pad1)
- SW3 pad 1: unconnected-(SW3-Pad1) -> Net-(SW3-Pad1)
- SW3 pad 3: Net-(R4-Pad1) -> Net-(SW3-Pad1)
- SW3 pad 4: unconnected-(SW3-Pad4) -> GND
- SW4 pad 1: unconnected-(SW4-Pad1) -> Net-(SW4-Pad1)
- SW4 pad 3: Net-(R7-Pad1) -> Net-(SW4-Pad1)
- SW4 pad 4: unconnected-(SW4-Pad4) -> GND
- SW5 pad 1: unconnected-(SW5-Pad1) -> Net-(SW5-Pad1)
- SW5 pad 3: Net-(R9-Pad1) -> Net-(SW5-Pad1)
- SW5 pad 4: unconnected-(SW5-Pad4) -> GND
- SW6 pad 1: unconnected-(SW6-Pad1) -> Net-(R11-Pad1)
- SW6 pad 4: unconnected-(SW6-Pad4) -> GND
- U2 pad 10: /display board/SPI0_SCLK -> /Display board (SNAP OFF BOARD)/SPI0_SCLK
- U2 pad 13: /display board/SPI_MISO -> /Display board (SNAP OFF BOARD)/SPI_MISO
- U2 pad 14: /display board/SPI0_MOSI -> /Display board (SNAP OFF BOARD)/SPI0_MOSI
- U2 pad 39: /display board/+3.3v -> /Display board (SNAP OFF BOARD)/+3.3v
- U2 pad 40: /display board/+3.3v -> /Display board (SNAP OFF BOARD)/+3.3v
- U2 pad 6: /display board/+3.3v -> /Display board (SNAP OFF BOARD)/+3.3v
- U2 pad 7: /display board/+3.3v -> /Display board (SNAP OFF BOARD)/+3.3v
- U2 pad 9: /display board/SPI0_CE0_N -> /Display board (SNAP OFF BOARD)/SPI0_CE0_N

Commit message: enough for now
Parts:
- Module0: moved to B.Cu
- moved U1 306.1 mm to (-85.3, 105.2)
- moved C14 303.0 mm to (-65.2, 117.1)
- moved C6 303.0 mm to (-65.2, 119.0)
- moved R31 303.0 mm to (-85.5, 144.2)
- moved TP6 303.0 mm to (-51.4, 109.3)
- moved C10 303.0 mm to (-75.3, 129.2)
- moved C11 303.0 mm to (-45.0, 98.9)
- moved C12 303.0 mm to (-72.1, 129.2)
- moved C13 303.0 mm to (-45.0, 100.9)
- moved C5 303.0 mm to (-62.0, 115.1)
- moved R10 303.0 mm to (-65.2, 113.1)
- moved R11 303.0 mm to (-75.3, 127.3)
- moved R12 303.0 mm to (-64.1, 111.1)
- moved R26 303.0 mm to (-75.3, 125.3)
- moved R27 303.0 mm to (-68.5, 121.1)
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Connections:
- J2 pad 3: /CM4/SCREEN_MOSI -> /CM4/SCREEN_CE0_N
- J2 pad 4: /CM4/SCREEN_MISO -> /CM4/SCREEN_SCLK
- J2 pad 5: /CM4/SCREEN_SCLK -> /CM4/SCREEN_MISO
- J2 pad 6: /CM4/SCREEN_CE0_N -> /CM4/SCREEN_MOSI
- J6 pad 3: /Display board (SNAP OFF BOARD)/SPI0_MOSI -> /Display board (SNAP OFF BOARD)/SPI0_CE0_N
- J6 pad 4: /Display board (SNAP OFF BOARD)/SPI_MISO -> /Display board (SNAP OFF BOARD)/SPI0_SCLK
- J6 pad 5: /Display board (SNAP OFF BOARD)/SPI0_SCLK -> /Display board (SNAP OFF BOARD)/SPI_MISO
- J6 pad 6: /Display board (SNAP OFF BOARD)/SPI0_CE0_N -> /Display board (SNAP OFF BOARD)/SPI0_MOSI
- J6 pad 7: GND -> GND1
- J6 pad 8: GND -> GND1
- J6 pad MP1: GND -> GND1
- J6 pad MP2: GND -> GND1
- TP20 pad 1: GND -> GND1
- U2 pad 16: GND -> GND1
- U2 pad 34: GND -> GND1
- U2 pad 35: GND -> GND1
- U2 pad 36: GND -> GND1
- U2 pad 37: GND -> GND1
- U2 pad 38: GND -> GND1
- U2 pad 5: GND -> GND1
Other:
- board size 77.2 x 77.3 mm -> 77.2 x 105 mm

Commit message: a
Parts:
- R47: footprint Resistor_SMD:R_0603_1608Metric_Pad0.98x0.95mm_HandSolder -> Resistor_SMD:R_1210_3225Metric_Pad1.30x2.65mm_HandSolder
- moved R9 162.0 mm to (86.0, 107.8), turned to 90 degrees
- moved TP14 159.1 mm to (66.7, 89.0)
- moved C5 156.2 mm to (94.2, 113.2), turned to -90 degrees
- moved R11 149.2 mm to (73.1, 111.9), turned to 90 degrees
- moved R10 149.1 mm to (83.9, 113.1), turned to 90 degrees
- moved C6 146.5 mm to (81.3, 117.1), turned to -90 degrees
- moved SW10 146.3 mm to (69.6, 145.4)
- moved R33 138.6 mm to (65.4, 151.0), turned to 90 degrees
- moved TP16 136.7 mm to (69.7, 143.0)
- moved C10 136.0 mm to (58.8, 151.8), turned to -90 degrees
- moved R12 135.3 mm to (71.0, 117.1), turned to 90 degrees
- moved TP15 135.1 mm to (55.4, 143.0)
- moved U1 131.7 mm to (46.0, 94.7), turned to -90 degrees
- moved R26 130.7 mm to (53.5, 147.8), turned to 90 degrees
- moved R32 130.7 mm to (67.7, 147.7), turned to 90 degrees
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Connections:
- SW2 pad 4: unconnected-(SW2-Pad4) -> GND
- SW7 pad 4: unconnected-(SW7-Pad4) -> GND

Commit message: aa
Parts:
- C15, C18, C19, C20, C25, C26: footprint Capacitor_SMD:C_01005_0402Metric_Pad0.57x0.30mm_HandSolder -> Capacitor_SMD:C_2225_5664Metric_Pad1.80x6.60mm_HandSolder
- C22: footprint Capacitor_SMD:C_0603_1608Metric_Pad1.08x0.95mm_HandSolder -> Capacitor_SMD:C_1210_3225Metric_Pad1.33x2.70mm_HandSolder
- R13: footprint Capacitor_SMD:C_0402_1005Metric_Pad0.74x0.62mm_HandSolder -> Resistor_SMD:R_0402_1005Metric_Pad0.72x0.64mm_HandSolder
- R42, R46, R48, R49, R50, R51, R52, R53, R54: footprint Resistor_SMD:R_0603_1608Metric_Pad0.98x0.95mm_HandSolder -> Resistor_SMD:R_0402_1005Metric_Pad0.72x0.64mm_HandSolder
- R47: footprint Resistor_SMD:R_1210_3225Metric_Pad1.30x2.65mm_HandSolder -> Resistor_SMD:R_0402_1005Metric_Pad0.72x0.64mm_HandSolder
- R55, R58: footprint Resistor_SMD:R_0603_1608Metric_Pad0.98x0.95mm_HandSolder -> Resistor_SMD:R_1210_3225Metric_Pad1.30x2.65mm_HandSolder
- R59: footprint Resistor_SMD:R_0603_1608Metric_Pad0.98x0.95mm_HandSolder -> Resistor_SMD:R_2816_7142Metric_Pad3.20x4.45mm_HandSolder
- U1: footprint TI74HC14N:Texas_Instruments-R_R-PDIP-T14-0-0-0 -> Package_SO:SO-14_3.9x8.65mm_P1.27mm
- moved C9 209.4 mm to (324.5, 29.0)
- moved TP28 209.3 mm to (328.0, 27.0)
- moved R18 202.3 mm to (308.2, 33.0), turned to -90 degrees
- moved D5 201.8 mm to (314.8, 33.0), turned to 90 degrees
- moved C7 201.6 mm to (318.8, 30.5)
- moved C24 200.8 mm to (311.2, 29.0)
- moved SW12 187.7 mm to (125.0, 185.2), turned to -90 degrees
- moved D4 174.4 mm to (328.0, 33.0), turned to 90 degrees
- moved R24 168.9 mm to (321.8, 33.0), turned to -90 degrees
- moved J7 161.9 mm to (317.1, 9.89), turned to -90 degrees
- moved R14 148.7 mm to (318.8, 27.5)
- moved R23 148.6 mm to (305.2, 27.5)
- moved C23 147.2 mm to (305.2, 30.5)
- moved J4 144.4 mm to (82.7, 166.0)
- moved TP27 126.9 mm to (315.0, 27.0)
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Connections:
- U1 pad 3: /Buttons/__DP_D -> /Buttons/__DP_R
- U1 pad 4: /Buttons/DPAD_DOWN -> /Buttons/DPAD_RIGHT
- U1 pad 5: /Buttons/__DP_L -> /Buttons/__DP_D
- U1 pad 6: /Buttons/DPAD_LEFT -> /Buttons/DPAD_DOWN
- U1 pad 8: /Buttons/DPAD_RIGHT -> /Buttons/DPAD_LEFT
- U1 pad 9: /Buttons/__DP_R -> /Buttons/__DP_L
Other:
- board text added: "JLCJLCJLCJLC"

Commit message: revise board
Parts:
- moved Module0 101.4 mm to (256.8, 113.8)
- moved D6 94.8 mm to (91.8, 39.2), turned to 180 degrees
- moved R19 77.4 mm to (9.94, 133.2)
- moved TP20 77.4 mm to (11.2, 128.2)
- moved TP21 77.4 mm to (11.2, 115.0)
- moved TP22 77.4 mm to (11.2, 118.2)
- moved TP23 77.4 mm to (11.2, 121.5)
- moved TP24 77.4 mm to (11.2, 124.8)
- moved TP25 77.4 mm to (11.2, 111.8)
- moved U2 77.4 mm to (19.5, 123.0)
- moved J6 77.1 mm to (5.19, 122.5)
- moved R59 35.4 mm to (147.8, 95.2), turned to -90 degrees
- moved C19 20.4 mm to (170.5, 70.2), turned to -90 degrees
- moved TP8 18.7 mm to (72.8, 128.0)
- moved TP6 18.7 mm to (74.2, 126.5)
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Other:
- board size 77.2 x 105 mm -> 103.3 x 77.2 mm

Commit message: aaa
Parts:
- added REF**: MountingHole_2.1mm, MountingHole:MountingHole_2.1mm, F.Cu at (62.5, 113.2)
- moved R55 18.0 mm to (70.0, 165.0)
- moved TP10 0.72 mm to (57.2, 119.0)
- moved U1 0.72 mm to (62.5, 120.2)
- moved C1 0.39 mm to (36.2, 110.0)
- moved TP11 0.33 mm to (57.2, 121.1)
Other:
- outline, holes or cut-outs redrawn
