File: sch/carrier/carrier.kicad_pcb (KiCad board)
At the start: 2 copper layers, 103.3 x 77.2 mm, 147 parts, among them J1 USB_C_Receptacle_USB2.0, J2 52271-0879, J3 Micro_SD_Card, J4 HDMI_D_1.4, J5 USB_C_Receptacle_USB2.0, J6 52271-0879, J7 AudioJack3_Switch, SW1 SKRRACE010, SW10 SKRBAAE010, SW11 SW_Push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

Commit message: aaaaaaaaaaaaaaaaaaaaaaaaa
Parts:
- C18, C19, C20, C25, C26: footprint Capacitor_SMD:C_2225_5664Metric_Pad1.80x6.60mm_HandSolder -> Capacitor_SMD:C_1206_3216Metric_Pad1.33x1.80mm_HandSolder
- R47: footprint Resistor_SMD:R_0402_1005Metric_Pad0.72x0.64mm_HandSolder -> Resistor_SMD:R_1210_3225Metric_Pad1.30x2.65mm_HandSolder
- moved C14 124.4 mm to (13.8, 31.1)
- moved R29 124.4 mm to (-0.60, 48.1)
- moved R31 124.4 mm to (29.3, 40.5)
- moved R34 124.4 mm to (6.96, 37.3)
- moved R35 124.4 mm to (52.1, 36.9)
- moved SW11 124.4 mm to (41.8, 45.5)
- moved SW9 124.4 mm to (58.8, 46.2)
- moved TP17 124.4 mm to (24.8, 43.3)
- moved TP18 124.4 mm to (20.2, 29.7)
- moved C12 124.4 mm to (-5.95, 30.9)
- moved L1 71.8 mm to (258.2, 81.2)
- moved R47 70.3 mm to (265.8, 74.0), turned to 90 degrees
- moved R49 69.6 mm to (250.8, 75.5)
- moved R46 55.1 mm to (242.8, 99.0), turned to 90 degrees
- moved U3 53.9 mm to (240.5, 91.8)
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Connections:
- R46 pad 1: Net-(R46-Pad1) -> GND
- R46 pad 2: GND -> Net-(R46-Pad2)
- U3 pad 13: Net-(R46-Pad1) -> Net-(R46-Pad2)
Other:
- copper layers 2 -> 4
- board text added: "BOOST | CHARGE"
