File: sch/carrier/_autosave-power.kicad_sch (KiCad schematic)
At the start: 32 parts, among them J4 USB_C_Receptacle_USB2.0, U3 MP2636GR-P

Commit message: still alive :)
Parts:
- added R? (x4): 10.5k, symbol Device:R
- added R?: R, symbol Device:R
Connections:
- net GNDA: now also R?.2
- net _CHIP_VCC: now also R?.1, R?.1, R?.1
- net at U3.16 (VB): now also R?.1, R?.2
- net at U3.24 (MODE): now also R?.2
- net at U3.25 (EN): now also R?.2
- net at U3.6 (ILIM): now also R?.1
Other:
- note added: "some figures so dont need to keep hunting for f(sw)=600khz"
- moved on the sheet: C?
