File: sch/carrier/connectors.kicad_sch (KiCad schematic)
At the start: 4 parts

Commit message: AASKHUQAWFHIU
Parts:
- J2: renamed from J?; footprint Molex-1054500101-* -> MOLEXC:Molex-1054500101-MFG
- Module0: renamed from Module?; value ComputeModule4 -> ComputeModule4-CM4
Connections:
- net GND: now also Module0.101 (USB_OTG_ID), Module0.102 (PCIe_CLK_nREQ), Module0.110 (PCIe_CLK_P), Module0.112 (PCIe_CLK_N), Module0.116 (PCIe_RX_P), Module0.118 (PCIe_RX_N), Module0.122 (PCIe_TX_P), Module0.124 (PCIe_TX_N), Module0.128 (CAM0_D0_N), Module0.130 (CAM0_D0_P), Module0.134 (CAM0_D1_N), Module0.136 (CAM0_D1_P), Module0.140 (CAM0_C_N), Module0.142 (CAM0_C_P), Module0.146 (HDMI1_TX2_P), Module0.148 (HDMI1_TX2_N), Module0.152 (HDMI1_TX1_P), Module0.154 (HDMI1_TX1_N), Module0.157 (DSI0_D0_N), Module0.158 (HDMI1_TX0_P), Module0.159 (DSI0_D0_P), Module0.160 (HDMI1_TX0_N), Module0.163 (DSI0_D1_N), Module0.164 (HDMI1_CLK_P), Module0.165 (DSI0_D1_P), Module0.166 (HDMI1_CLK_N), Module0.169 (DSI0_C_N), Module0.171 (DSI0_C_P), Module0.175 (DSI1_D0_N), Module0.177 (DSI1_D0_P), Module0.181 (DSI1_D1_N), Module0.183 (DSI1_D1_P), Module0.187 (DSI1_C_N), Module0.189 (DSI1_C_P), Module0.193 (DSI1_D2_N), Module0.194 (DSI1_D3_N), Module0.195 (DSI1_D2_P), Module0.196 (DSI1_D3_P)
- no-connect marks 0 -> 2

Commit message: goodnight
Other:
- title: (none) -> Port data connectors
Changed lines of the file:
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@@
 (kicad_sch (version 20210621) (generator eeschema)
   (paper "A4")
+  (title_block
+    (title "Port data connectors")
+  )
   (junction (at 18.415 33.02) (diameter 0.9144) (color 0 0 0 0))
   (junction (at 18.415 35.56) (diameter 0.9144) (color 0 0 0 0))

Commit message: hhhhhhhhhhhhhhhhh
Connections:
- net GND: now also Module0.147 (HDMI1_SCL)
Changed lines of the file:
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@@
   (junction (at 94.615 63.5) (diameter 0.9144) (color 0 0 0 0))
   (junction (at 94.615 71.12) (diameter 0.9144) (color 0 0 0 0))
+  (junction (at 94.615 83.82) (diameter 0.9144) (color 0 0 0 0))
   (junction (at 94.615 93.98) (diameter 0.9144) (color 0 0 0 0))
   (junction (at 94.615 96.52) (diameter 0.9144) (color 0 0 0 0))
@@
     (stroke (width 0) (type solid) (color 0 0 0 0))
   )
+  (wire (pts (xy 86.995 83.82) (xy 94.615 83.82))
+    (stroke (width 0) (type solid) (color 0 0 0 0))
+  )
   (wire (pts (xy 86.995 93.98) (xy 94.615 93.98))
     (stroke (width 0) (type solid) (color 0 0 0 0))
@@
     (stroke (width 0) (type solid) (color 0 0 0 0))
   )
-  (wire (pts (xy 94.615 71.12) (xy 94.615 93.98))
-    (stroke (width 0) (type solid) (color 0 0 0 0))
-  )
+  (wire (pts (xy 94.615 71.12) (xy 94.615 83.82))
+    (stroke (width 0) (type solid) (color 0 0 0 0))
+  )
+  (wire (pts (xy 94.615 83.82) (xy 94.615 93.98))
+    (stroke (width 0) (type solid) (color 0 0 0 0))
+  )

Commit message: a
Parts:
- removed J2: 1054500101, MOLEXC:Molex-1054500101-MFG, symbol MOLEXC:1054500101
- added J?: USB_C_Receptacle_USB2.0, Connector_USB:USB_C_Receptacle_JAE_DX07S016JA1R1500, symbol Connector:USB_C_Receptacle_USB2.0
- added R? (x2): 5.1k, Resistor_SMD:R_0805_2012Metric_Pad1.20x1.40mm_HandSolder, symbol Device:R
- added R?: 0, symbol Device:R
Connections:
- net GND: now also J?.A1 (GND), J?.A12 (GND), J?.B1 (GND), J?.B12 (GND), R?.2, R?.2, R?.2
- new net: J?.A5 (CC1), R?.1
- new net: J?.S1 (SHIELD), R?.1
- new net: J?.B5 (CC2), R?.1
- new net VBUS: J?.A4 (VBUS), J?.A9 (VBUS), J?.B4 (VBUS), J?.B9 (VBUS)
Other:
- note added: "TODO: add HDMI connections"
- note added: "Too many people on stack overflow/exchange seem to be unable to agree on this! Leaving this unconnected with a 0 ohm so we can if we choose to - but grounding it could apparently cause a ground loop thingy (which would probably happen since we do not have a true ground in batterys i guess?)"
- note added: "also todo: look up how to do differential pairs in kicad since apparently it needs differential pairs on hdmi (note to sefl: differential pair is 2 wires with the same info but routed in such a way that the resulting signal is 'skewed', which is a bit like what an op amp does to the signal it seems)"

Commit message: oh yeah
Parts:
- gave numbers to parts that had none: 4
Changed lines of the file:
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@@
     (title "Port data connectors")
     (rev "indev")
-    (comment 1 "https://github.com/cinnamondev/gamepithing")
   )
   (junction (at 18.415 33.02) (diameter 0.9144) (color 0 0 0 0))
@@
   (symbol (lib_id "power:GND") (at 224.155 66.675 0) (unit 1)
     (in_bom yes) (on_board yes) (fields_autoplaced)
-    (property "Reference" "#PWR?" (id 0) (at 224.155 73.025 0)
+    (property "Reference" "#PWR08" (id 0) (at 224.155 73.025 0)
       (effects (font (size 1.27 1.27)) hide)
     )
@@
   (symbol (lib_id "power:GND") (at 259.08 28.575 0) (unit 1)
     (in_bom yes) (on_board yes) (fields_autoplaced)
-    (property "Reference" "#PWR?" (id 0) (at 259.08 34.925 0)
+    (property "Reference" "#PWR09" (id 0) (at 259.08 34.925 0)
       (effects (font (size 1.27 1.27)) hide)
     )
@@
   (symbol (lib_id "Device:R") (at 216.535 62.865 0) (unit 1)
     (in_bom yes) (on_board yes)
-    (property "Reference" "R?" (id 0) (at 218.44 61.5949 0)
+    (property "Reference" "R15" (id 0) (at 218.44 61.5949 0)
       (effects (font (size 1.27 1.27)) (justify left))
     )
@@
   (symbol (lib_id "Device:R") (at 248.285 26.035 90) (unit 1)
     (in_bom yes) (on_board yes)
-    (property "Reference" "R?" (id 0) (at 248.285 24.13 90))
+    (property "Reference" "R16" (id 0) (at 248.285 24.13 90))
     (property "Value" "5.1k" (id 1) (at 248.285 26.035 90))
     (property "Footprint" "Resistor_SMD:R_0805_2012Metric_Pad1.20x1.40mm_HandSolder" (id 2) (at 248.285 27.813 90)
@@
   (symbol (lib_id "Device:R") (at 248.285 28.575 90) (unit 1)
     (in_bom yes) (on_board yes)
-    (property "Reference" "R?" (id 0) (at 248.285 31.115 90))
+    (property "Reference" "R17" (id 0) (at 248.285 31.115 90))
     (property "Value" "5.1k" (id 1) (at 248.285 28.575 90))
     (property "Footprint" "Resistor_SMD:R_0805_2012Metric_Pad1.20x1.40mm_HandSolder" (id 2) (at 248.285 30.353 90)
@@
   (symbol (lib_id "Connector:USB_C_Receptacle_USB2.0") (at 224.155 36.195 0) (unit 1)
     (in_bom yes) (on_board yes) (fields_autoplaced)
-    (property "Reference" "J?" (id 0) (at 226.822 12.7 0))
+    (property "Reference" "J1" (id 0) (at 226.822 12.7 0))
     (property "Value" "USB_C_Receptacle_USB2.0" (id 1) (at 226.822 15.24 0))
     (property "Footprint" "Connector_USB:USB_C_Receptacle_JAE_DX07S016JA1R1500" (id 2) (at 227.965 36.195 0)
