File: sch/carrier/connectors.kicad_sch (KiCad schematic)
At the start: 5 parts, among them J1 USB_C_Receptacle_USB2.0

Commit message: get git committed
Parts:
- added J?: USB_C_Receptacle_USB2.0, Connector_USB:USB_C_Receptacle_JAE_DX07S016JA1R1500, symbol Connector:USB_C_Receptacle_USB2.0
- added R? (x2): 5.1k, Resistor_SMD:R_0805_2012Metric_Pad1.20x1.40mm_HandSolder, symbol Device:R
- added R?: 0, symbol Device:R
Connections:
- net GND: now also J?.A1 (GND), J?.A12 (GND), J?.B1 (GND), J?.B12 (GND), R?.2, R?.2, R?.2
- new net: J?.A5 (CC1), R?.1
- new net: J?.B5 (CC2), R?.1
- new net: J?.S1 (SHIELD), R?.1
- new net VBUS_CHARGE: J?.A4 (VBUS), J?.A9 (VBUS), J?.B4 (VBUS), J?.B9 (VBUS)
- no-connect marks 2 -> 8
Other:
- note added: "No data"
- note added: "Too many people on stack overflow/exchange seem to be unable to agree on this! Leaving this unconnected with a 0 ohm so we can if we choose to."
- note added: "per USBC spec - deliver 5V3A"
Changed lines of the file:
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@@
   (junction (at 94.615 144.78) (diameter 0.9144) (color 0 0 0 0))
   (junction (at 94.615 147.32) (diameter 0.9144) (color 0 0 0 0))
+  (junction (at 210.82 126.365) (diameter 0.9144) (color 0 0 0 0))
   (junction (at 224.155 66.675) (diameter 0.9144) (color 0 0 0 0))
+  (junction (at 239.395 160.02) (diameter 0.9144) (color 0 0 0 0))
   (junction (at 259.08 28.575) (diameter 0.9144) (color 0 0 0 0))
   (no_connect (at 26.035 27.94))
   (no_connect (at 26.035 30.48))
+  (no_connect (at 206.375 137.16))
+  (no_connect (at 208.915 137.16))
+  (no_connect (at 211.455 137.16))
+  (no_connect (at 213.995 137.16))
+  (no_connect (at 221.615 137.16))
+  (no_connect (at 224.155 137.16))
   (wire (pts (xy 18.415 25.4) (xy 18.415 33.02))
     (stroke (width 0) (type solid) (color 0 0 0 0))
@@
     (stroke (width 0) (type solid) (color 0 0 0 0))
   )
+  (wire (pts (xy 193.675 137.16) (xy 193.675 132.08))
+    (stroke (width 0) (type solid) (color 0 0 0 0))
+  )
+  (wire (pts (xy 198.755 122.555) (xy 198.755 137.16))
+    (stroke (width 0) (type solid) (color 0 0 0 0))
+  )
+  (wire (pts (xy 198.755 122.555) (xy 203.2 122.555))
+    (stroke (width 0) (type solid) (color 0 0 0 0))
+  )
+  (wire (pts (xy 201.295 126.365) (xy 201.295 137.16))
+    (stroke (width 0) (type solid) (color 0 0 0 0))
+  )
+  (wire (pts (xy 203.2 126.365) (xy 201.295 126.365))
+    (stroke (width 0) (type solid) (color 0 0 0 0))
+  )
+  (wire (pts (xy 210.82 122.555) (xy 210.82 126.365))
+    (stroke (width 0) (type solid) (color 0 0 0 0))
+  )
+  (wire (pts (xy 210.82 126.365) (xy 210.82 128.27))
+    (stroke (width 0) (type solid) (color 0 0 0 0))
+  )
   (wire (pts (xy 216.535 66.675) (xy 224.155 66.675))
     (stroke (width 0) (type solid) (color 0 0 0 0))
@@
     (stroke (width 0) (type solid) (color 0 0 0 0))
   )
+  (wire (pts (xy 231.775 152.4) (xy 239.395 152.4))
+    (stroke (width 0) (type solid) (color 0 0 0 0))
+  )
   (wire (pts (xy 239.395 20.955) (xy 244.475 20.955))
     (stroke (width 0) (type solid) (color 0 0 0 0))
@@
   )
   (wire (pts (xy 239.395 28.575) (xy 244.475 28.575))
+    (stroke (width 0) (type solid) (color 0 0 0 0))
+  )
+  (wire (pts (xy 239.395 160.02) (xy 239.395 152.4))
+    (stroke (width 0) (type solid) (color 0 0 0 0))
+  )
+  (wire (pts (xy 239.395 160.02) (xy 239.395 161.925))
     (stroke (width 0) (type solid) (color 0 0 0 0))
   )
@@
     (effects (font (size 1.27 1.27)) (justify left bottom))
   )
+  (text "No data\n" (at 213.995 136.525 180)
+    (effects (font (size 1.27 1.27)) (justify right bottom))
+  )
+  (text "per USBC spec - deliver 5V3A" (at 215.265 136.525 90)
+    (effects (font (size 1.016 1.016)) (justify left bottom))
+  )
+  (text "Too many people on stack overflow/exchange\nseem to be unable to agree on this! Leaving\nthis unconnected with a 0 ohm so we can if we \nchoose to."
+    (at 241.935 160.02 0)
+    (effects (font (size 1.016 1.016)) (justify left bottom))
+  )
   (label "USB2_D-" (at 107.95 27.94 180)
     (effects (font (size 1.27 1.27)) (justify right bottom))
@@
   (label "VBUS" (at 244.475 20.955 180)
     (effects (font (size 1.27 1.27)) (justify right bottom))
+  )
+  (hierarchical_label "VBUS_CHARGE" (shape output) (at 193.675 132.08 90)
+    (effects (font (size 1.27 1.27)) (justify left))
   )
   (symbol (lib_id "power:GND") (at 18.415 161.29 0) (unit 1)
@@
     (pin "1")
   )
+  (symbol (lib_id "power:GND") (at 210.82 128.27 0) (unit 1)
+    (in_bom yes) (on_board yes) (fields_autoplaced)
+    (property "Reference" "#PWR?" (id 0) (at 210.82 134.62 0)
+      (effects (font (size 1.27 1.27)) hide)
+    )
+    (property "Value" "GND" (id 1) (at 210.82 132.715 0))
+    (property "Footprint" "" (id 2) (at 210.82 128.27 0)
+      (effects (font (size 1.27 1.27)) hide)
+    )
+    (property "Datasheet" "" (id 3) (at 210.82 128.27 0)
+      (effects (font (size 1.27 1.27)) hide)
+    )
+    (pin "1")
+  )
   (symbol (lib_id "power:GND") (at 224.155 66.675 0) (unit 1)
     (in_bom yes) (on_board yes) (fields_autoplaced)
@@
     (pin "1")
   )
+  (symbol (lib_id "power:GND") (at 239.395 161.925 0) (unit 1)
+    (in_bom yes) (on_board yes)
+    (property "Reference" "#PWR?" (id 0) (at 239.395 168.275 0)
+      (effects (font (size 1.27 1.27)) hide)
+    )
+    (property "Value" "GND" (id 1) (at 239.395 165.735 0))
+    (property "Footprint" "" (id 2) (at 239.395 161.925 0)
+      (effects (font (size 1.27 1.27)) hide)
+    )
+    (property "Datasheet" "" (id 3) (at 239.395 161.925 0)
+      (effects (font (size 1.27 1.27)) hide)
+    )
+    (pin "1")
+  )
   (symbol (lib_id "power:GND") (at 259.08 28.575 0) (unit 1)
     (in_bom yes) (on_board yes) (fields_autoplaced)
@@
     )
     (pin "1")
+  )
+  (symbol (lib_id "Device:R") (at 207.01 122.555 90) (unit 1)
+    (in_bom yes) (on_board yes)
+    (property "Reference" "R?" (id 0) (at 207.01 120.65 90))
+    (property "Value" "5.1k" (id 1) (at 207.01 122.555 90))
+    (property "Footprint" "Resistor_SMD:R_0805_2012Metric_Pad1.20x1.40mm_HandSolder" (id 2) (at 207.01 124.333 90)
+      (effects (font (size 1.27 1.27)) hide)
+    )
+    (property "Datasheet" "~" (id 3) (at 207.01 122.555 0)
+      (effects (font (size 1.27 1.27)) hide)
+    )
+    (pin "1")
+    (pin "2")
+  )
+  (symbol (lib_id "Device:R") (at 207.01 126.365 90) (unit 1)
+    (in_bom yes) (on_board yes)
+    (property "Reference" "R?" (id 0) (at 207.01 124.46 90))
+    (property "Value" "5.1k" (id 1) (at 207.01 126.365 90))
+    (property "Footprint" "Resistor_SMD:R_0805_2012Metric_Pad1.20x1.40mm_HandSolder" (id 2) (at 207.01 128.143 90)
+      (effects (font (size 1.27 1.27)) hide)
+    )
+    (property "Datasheet" "~" (id 3) (at 207.01 126.365 0)
+      (effects (font (size 1.27 1.27)) hide)
+    )
+    (pin "1")
+    (pin "2")
   )
   (symbol (lib_id "Device:R") (at 216.535 62.865 0) (unit 1)
@@
     )
     (property "Datasheet" "~" (id 3) (at 216.535 62.865 0)
+      (effects (font (size 1.27 1.27)) hide)
+    )
+    (pin "1")
+    (pin "2")
+  )
+  (symbol (lib_id "Device:R") (at 235.585 160.02 90) (unit 1)
+    (in_bom yes) (on_board yes)
+    (property "Reference" "R?" (id 0) (at 237.4899 158.115 90)
+      (effects (font (size 1.27 1.27)) (justify left))
+    )
+    (property "Value" "0" (id 1) (at 236.2199 160.02 90)
+      (effects (font (size 1.27 1.27)) (justify left))
+    )
+    (property "Footprint" "" (id 2) (at 235.585 161.798 90)
+      (effects (font (size 1.27 1.27)) hide)
+    )
+    (property "Datasheet" "~" (id 3) (at 235.585 160.02 0)
       (effects (font (size 1.27 1.27)) hide)
     )
@@
     (pin "2")
   )
+  (symbol (lib_id "Connector:USB_C_Receptacle_USB2.0") (at 208.915 152.4 90) (unit 1)
+    (in_bom yes) (on_board yes) (fields_autoplaced)
+    (property "Reference" "J?" (id 0) (at 185.42 149.733 0))
+    (property "Value" "USB_C_Receptacle_USB2.0" (id 1) (at 187.96 149.733 0))
+    (property "Footprint" "Connector_USB:USB_C_Receptacle_JAE_DX07S016JA1R1500" (id 2) (at 208.915 148.59 0)
+      (effects (font (size 1.27 1.27)) hide)
+    )
+    (property "Datasheet" "https://www.usb.org/sites/default/files/documents/usb_type-c.zip" (id 3) (at 208.915 148.59 0)
+      (effects (font (size 1.27 1.27)) hide)
+    )
+    (pin "A1")
+    (pin "A12")
+    (pin "A4")
+    (pin "A5")
+    (pin "A6")
+    (pin "A7")
+    (pin "A8")
+    (pin "A9")
+    (pin "B1")
+    (pin "B12")
+    (pin "B4")
+    (pin "B5")
+    (pin "B6")
+    (pin "B7")
+    (pin "B8")
+    (pin "B9")
+    (pin "S1")
+  )
   (symbol (lib_id "Connector:USB_C_Receptacle_USB2.0") (at 224.155 36.195 0) (unit 1)

Commit message: aaaaaaaaaaaaaaaa
Parts:
- removed J?: USB_C_Receptacle_USB2.0, Connector_USB:USB_C_Receptacle_JAE_DX07S016JA1R1500, symbol Connector:USB_C_Receptacle_USB2.0
- removed R? (x2): 5.1k, Resistor_SMD:R_0805_2012Metric_Pad1.20x1.40mm_HandSolder, symbol Device:R
- removed R?: 0, symbol Device:R
- added J?: HDMI_D_1.4, symbol Connector:HDMI_D_1.4
- added J?: USB_C_Receptacle_USB2.0, Connector_USB:USB_C_Receptacle_JAE_DX07S016JA1R1500, symbol Connector:USB_C_Receptacle_USB2.0
- added R? (x2): 5.1k, Resistor_SMD:R_0805_2012Metric_Pad1.20x1.40mm_HandSolder, symbol Device:R
- added R? (x2): 0, symbol Device:R
Connections:
- net GND: now also R16.1, R17.1, J?.16 (GND), J?.A1 (GND), J?.A12 (GND), J?.B1 (GND), J?.B12 (GND), R?.1, R?.1, R?.2, R?.2; no longer R16.2, R17.2
- net USB2_D+: now also J1.A6 (D+), J1.B6 (D+)
- net USB2_D-: now also J1.A7 (D-), J1.B7 (D-)
- net VBUS_CHARGE: now also J?.A4 (VBUS), J?.A9 (VBUS), J?.B4 (VBUS), J?.B9 (VBUS)
- net at J1.A5 (CC1): now also R16.2; no longer R16.1
- net HDMI_CEC: now reaches Module0.151 (HDMI0_CEC)
- net HDMI_CEC: now also J?.15 (CEC)
- net TX2_P: now reaches Module0.170 (HDMI0_TX2_P)
- net TX2_P: now also J?.3 (D2+)
- net TX2_N: now reaches Module0.172 (HDMI0_TX2_N)
- net TX2_N: now also J?.5 (D2-)
- net TX1_P: now reaches Module0.176 (HDMI0_TX1_P)
- net TX1_P: now also J?.6 (D1+)
- net TX1_N: now reaches Module0.178 (HDMI0_TX1_N)
- net TX1_N: now also J?.8 (D1-)
- net TX0_P: now reaches Module0.182 (HDMI0_TX0_P)
- net TX0_P: now also J?.9 (D0+)
- net TX0_N: now reaches Module0.184 (HDMI0_TX0_N)
- net TX0_N: now also J?.11 (D0-)
- net CLK_P: now reaches Module0.188 (HDMI0_CLK_P)
- net CLK_P: now also J?.12 (CK+)
- net CLK_N: now reaches Module0.190 (HDMI0_CLK_N)
- net CLK_N: now also J?.14 (CK-)
- net HDMI_SDA: now reaches Module0.199 (HDMI0_SDA)
- net HDMI_SDA: now also J?.18 (SDA)
- net HDMI_SCL: now reaches Module0.200 (HDMI0_SCL)
- net HDMI_SCL: now also J?.17 (SCL)
- net at J1.B5 (CC2): now also R17.2; no longer R17.1
- new net: J?.B5 (CC2), R?.2
- new net: J?.SH, R?.1
- new net: J?.S1 (SHIELD), R?.1
- new net: J?.A5 (CC1), R?.2
- no-connect marks 8 -> 6
Other:
- note added: "HDMI 1.4 Type-D Port"
- note added: "USB 2.0 Type-C Port (DATA only)"
- note added: "USB 2.0 Type-C Port (POWER only)"
- note removed: "No data"
- note removed: "Too many people on stack overflow/exchange seem to be unable to agree on this! Leaving this unconnected with a 0 ohm so we can if we choose to."
- note removed: "USB-C 2.0 OTG PORT (No power in)"
- note removed: "per USBC spec - deliver 5V3A"
- moved on the sheet: J1, Module0B, R15, R16, R17

Commit message: changes and carrier backups
Connections:
- net VBUS is gone; now on net +5v: J1.A4 (VBUS), J1.A9 (VBUS), J1.B4 (VBUS), J1.B9 (VBUS)
- net GND: now also J?.10 (D0S), J?.13 (CKS), J?.4 (D2S), J?.7 (D1S)
- net HDMI_HP: now reaches J?.1 (HPD/HEAC-)
- net HDMI_HP: now also Module0.153 (HDMI0_HOTPLUG)
- net +5v: now reaches J?.19 (+5V)
- no-connect marks 6 -> 7
Other:
- note added: "NO DATA!"
- note added: "TODO: Find out how to do 'differential pairs' in KiCad"
- note removed: "also todo: look up how to do differential pairs in kicad since apparently it needs differential pairs on hdmi (note to sefl: differential pair is 2 wires with the same info but routed in such a way that the resulting signal is 'skewed', which is a bit like what an op amp does to the signal it seems)"
- moved on the sheet: J?, R?

Commit message: add speaker and charger
Parts:
- J?: footprint (none) -> Connector_HDMI:HDMI_Micro-D_Molex_46765-1x01
Other:
- note removed: "TODO: add HDMI connections"

Commit message: git pushed
Other:
- note added: "We don't need like, 99% of the pins on this one No PCIe No 2nd HDMI No Camera No DSI/MIPI (For now)"
Changed lines of the file:
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@@
     (title "Port data connectors")
     (rev "indev")
-    (comment 1 "https://www.github.com/cinnamondev/gamepithing")
   )
   (junction (at 29.21 33.655) (diameter 0.9144) (color 0 0 0 0))
@@
     (stroke (width 0) (type dash) (color 0 0 0 0))
   )
+  (text "We don't need like, 99% of the pins on this one\nNo PCIe\nNo 2nd HDMI\nNo Camera\nNo DSI/MIPI (For now)"
+    (at 142.875 121.285 0)
+    (effects (font (size 1.27 1.27)) (justify left bottom))
+  )
   (text "TODO: Find out how to do\n'differential pairs' in \nKiCad"

Commit message: ersfdxcv
Parts:
- gave numbers to parts that had none: 6
Changed lines of the file:
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@@
   (symbol (lib_id "power:GND") (at 195.58 83.185 0) (unit 1)
     (in_bom yes) (on_board yes)
-    (property "Reference" "#PWR?" (id 0) (at 195.58 89.535 0)
+    (property "Reference" "#PWR044" (id 0) (at 195.58 89.535 0)
       (effects (font (size 1.27 1.27)) hide)
     )
@@
   (symbol (lib_id "power:GND") (at 271.145 95.25 0) (unit 1)
     (in_bom yes) (on_board yes) (fields_autoplaced)
-    (property "Reference" "#PWR?" (id 0) (at 271.145 101.6 0)
+    (property "Reference" "#PWR045" (id 0) (at 271.145 101.6 0)
       (effects (font (size 1.27 1.27)) hide)
     )
@@
   (symbol (lib_id "power:GND") (at 281.94 120.65 0) (unit 1)
     (in_bom yes) (on_board yes) (fields_autoplaced)
-    (property "Reference" "#PWR?" (id 0) (at 281.94 127 0)
+    (property "Reference" "#PWR046" (id 0) (at 281.94 127 0)
       (effects (font (size 1.27 1.27)) hide)
     )
@@
   (symbol (lib_id "Device:R") (at 198.12 78.74 0) (unit 1)
     (in_bom yes) (on_board yes)
-    (property "Reference" "R?" (id 0) (at 199.39 78.7399 0)
+    (property "Reference" "R55" (id 0) (at 199.39 78.7399 0)
       (effects (font (size 1.27 1.27)) (justify left))
     )
@@
   (symbol (lib_id "Device:R") (at 250.825 87.63 270) (unit 1)
     (in_bom yes) (on_board yes)
-    (property "Reference" "R?" (id 0) (at 250.825 85.725 90))
+    (property "Reference" "R56" (id 0) (at 250.825 85.725 90))
     (property "Value" "5.1k" (id 1) (at 250.825 87.63 90))
     (property "Footprint" "Resistor_SMD:R_0805_2012Metric_Pad1.20x1.40mm_HandSolder" (id 2) (at 250.825 85.852 90)
@@
   (symbol (lib_id "Device:R") (at 250.825 92.075 270) (unit 1)
     (in_bom yes) (on_board yes)
-    (property "Reference" "R?" (id 0) (at 250.825 90.17 90))
+    (property "Reference" "R57" (id 0) (at 250.825 90.17 90))
     (property "Value" "5.1k" (id 1) (at 250.825 92.075 90))
     (property "Footprint" "Resistor_SMD:R_0805_2012Metric_Pad1.20x1.40mm_HandSolder" (id 2) (at 250.825 90.297 90)
@@
   (symbol (lib_id "Device:R") (at 275.59 119.38 90) (unit 1)
     (in_bom yes) (on_board yes)
-    (property "Reference" "R?" (id 0) (at 275.5899 116.84 90)
+    (property "Reference" "R58" (id 0) (at 275.5899 116.84 90)
       (effects (font (size 1.27 1.27)) (justify left))
     )
@@
   (symbol (lib_id "Connector:USB_C_Receptacle_USB2.0") (at 248.92 111.76 90) (unit 1)
     (in_bom yes) (on_board yes)
-    (property "Reference" "J?" (id 0) (at 229.235 111.633 90))
+    (property "Reference" "J5" (id 0) (at 229.235 111.633 90))
     (property "Value" "USB_C_Receptacle_USB2.0" (id 1) (at 227.965 109.093 0)
       (effects (font (size 1.27 1.27)) hide)
@@
   (symbol (lib_id "Connector:HDMI_D_1.4") (at 190.5 46.99 0) (unit 1)
     (in_bom yes) (on_board yes)
-    (property "Reference" "J?" (id 0) (at 201.295 46.9899 0)
-      (effects (font (size 1.27 1.27)) (justify left))
-    )
+    (property "Reference" "J4" (id 0) (at 201.295 46.9899 0)
+      (effects (font (size 1.27 1.27)) (justify left))
+    )

Commit message: a
Parts:
- R15, R55, R58: footprint (none) -> Resistor_SMD:R_0603_1608Metric_Pad0.98x0.95mm_HandSolder
Changed lines of the file:
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@@
       (effects (font (size 1.27 1.27)) (justify left))
     )
-    (property "Footprint" "" (id 2) (at 196.342 78.74 90)
+    (property "Footprint" "Resistor_SMD:R_0603_1608Metric_Pad0.98x0.95mm_HandSolder" (id 2) (at 196.342 78.74 90)
       (effects (font (size 1.27 1.27)) hide)
     )
@@
       (effects (font (size 1.27 1.27)) (justify left))
     )
-    (property "Footprint" "" (id 2) (at 275.59 58.293 90)
+    (property "Footprint" "Resistor_SMD:R_0603_1608Metric_Pad0.98x0.95mm_HandSolder" (id 2) (at 275.59 58.293 90)
       (effects (font (size 1.27 1.27)) hide)
     )
@@
       (effects (font (size 1.27 1.27)) (justify left))
     )
-    (property "Footprint" "" (id 2) (at 275.59 121.158 90)
+    (property "Footprint" "Resistor_SMD:R_0603_1608Metric_Pad0.98x0.95mm_HandSolder" (id 2) (at 275.59 121.158 90)
       (effects (font (size 1.27 1.27)) hide)
     )

Commit message: fds
Parts:
- R16, R17: value 5.1k -> 56k
Other:
- note added: "USB 2.0 Type-C Port (Small peripherals)"
- note added: "apparently resistance determines if host or device 56k upp down"
- note added: "todo: USB protection (tvs diode or something)"
- note removed: "USB 2.0 Type-C Port (DATA only)"
Changed lines of the file:
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@@
+    (effects (font (size 1.27 1.27)) (justify left bottom))
+  )
+  (text "apparently resistance determines if host or device\n56k upp down"
+    (at 219.71 9.525 0)
+    (effects (font (size 1.27 1.27)) (justify left bottom))
+  )
+  (text "todo: USB protection (tvs diode or something)" (at 227.965 11.43 0)
     (effects (font (size 1.27 1.27)) (justify left bottom))
   )
@@
     (effects (font (size 0.508 0.508)) (justify right bottom))
   )
-  (text "USB 2.0 Type-C Port (DATA only)\n" (at 282.575 72.39 180)
+  (text "USB 2.0 Type-C Port (Small peripherals)\n" (at 282.575 72.39 180)
     (effects (font (size 1.27 1.27)) (justify right bottom))
   )
@@
     (in_bom yes) (on_board yes)
     (property "Reference" "R16" (id 0) (at 250.825 13.97 90))
-    (property "Value" "5.1k" (id 1) (at 250.825 15.875 90))
+    (property "Value" "56k" (id 1) (at 250.825 15.875 90))
     (property "Footprint" "Resistor_SMD:R_0805_2012Metric_Pad1.20x1.40mm_HandSolder" (id 2) (at 250.825 14.097 90)
       (effects (font (size 1.27 1.27)) hide)
@@
     (in_bom yes) (on_board yes)
     (property "Reference" "R17" (id 0) (at 250.825 20.32 90))
-    (property "Value" "5.1k" (id 1) (at 250.825 22.225 90))
+    (property "Value" "56k" (id 1) (at 250.825 22.225 90))
     (property "Footprint" "Resistor_SMD:R_0805_2012Metric_Pad1.20x1.40mm_HandSolder" (id 2) (at 250.825 20.447 90)
       (effects (font (size 1.27 1.27)) hide)
