File: sch/carrier/gamepad.kicad_sch (KiCad schematic)
At the start: 25 parts, among them SW1 SKRRACE010, SW2 SKRRACE010, SW3 SKRRACE010, SW4 SKRRACE010, SW5 SKRRACE010, SW6 SKRRACE010, U1 SN74HC14N

Commit message: put some stuff on the pcb - it is going to kill me trying to get all on
Parts:
- added TP10: A, TestPoint:TestPoint_Pad_2.0x2.0mm, symbol Connector:TestPoint
- added TP11: B, TestPoint:TestPoint_Pad_2.0x2.0mm, symbol Connector:TestPoint
- added TP6: UP, TestPoint:TestPoint_Pad_2.0x2.0mm, symbol Connector:TestPoint
- added TP7: DOWN, TestPoint:TestPoint_Pad_2.0x2.0mm, symbol Connector:TestPoint
- added TP8: LEFT, TestPoint:TestPoint_Pad_2.0x2.0mm, symbol Connector:TestPoint
- added TP9: RIGHT, TestPoint:TestPoint_Pad_2.0x2.0mm, symbol Connector:TestPoint
Connections:
- net +3.3v: no longer R5.1
- net BTN_A: now also TP10.1
- net BTN_B: now also TP11.1
- net DPAD_DOWN: now also TP7.1
- net DPAD_LEFT: now also TP8.1
- net DPAD_RIGHT: now also TP9.1
- net DPAD_UP: now also TP6.1
- net GND: now also C1.1; no longer C1.2
- net __DP_L: now also C1.2; no longer C1.1
Other:
- moved on the sheet: C1, U1

Commit message: a
Connections:
- net +3.3v: now also R5.1
Other:
- note added: "TODO: consider getting rid of this?? we already have a RC network to help with debounce do we really need this"
- moved on the sheet: U1

Commit message: oh yeah
Parts:
- added C? (x3): 0.1uF, Capacitor_SMD:C_0504_1310Metric_Pad0.83x1.28mm_HandSolder, symbol Device:C
- added R? (x3): 10k, Resistor_SMD:R_0805_2012Metric_Pad1.20x1.40mm_HandSolder, symbol Device:R
- added R? (x3): 1k, Resistor_SMD:R_0805_2012Metric_Pad1.20x1.40mm_HandSolder, symbol Device:R
- added SW7, SW? (x2): SKRBAAE010, eec:SKRBAAE010, symbol EECBTN:SKRBAAE010
Connections:
- net +3.3v: now also R?.1, R?.1, R?.1
- net GND: now also C?.2, C?.2, C?.2, SW7.2, SW?.2, SW?.2
- new net: R?.1, SW7.3
- new net: R?.1, SW?.3 (x2)
- new net BTN_BACKLIGHT: C?.1, R?.2, R?.2
- new net BTN_SELECT: C?.1, R?.2, R?.2
- new net BTN_START: C?.1, R?.2, R?.2
Other:
- moved on the sheet: C1, C2, C3, C4, C5, C6, R1, R10, R11, R12, R2, R3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

Commit message: push updates
Parts:
- added SW?: DTSM31NV, symbol Switch:SW_Push
Other:
- note added: "Pi reset pin/global_en"
Changed lines of the file:
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@@
+    (effects (font (size 1.27 1.27)) (justify left bottom))
+  )
+  (text "Pi reset pin/global_en" (at 256.54 20.32 0)
     (effects (font (size 1.27 1.27)) (justify left bottom))
   )
@@
       (effects (font (size 1.27 1.27)) hide)
     )
+    (pin "1")
+    (pin "2")
+  )
+  (symbol (lib_id "Switch:SW_Push") (at 250.825 22.86 0) (unit 1)
+    (in_bom yes) (on_board yes) (fields_autoplaced)
+    (property "Reference" "SW?" (id 0) (at 250.825 15.24 0))
+    (property "Value" "DTSM31NV" (id 1) (at 250.825 17.78 0))
+    (property "Footprint" "" (id 2) (at 250.825 17.78 0)
+      (effects (font (size 1.27 1.27)) hide)
+    )
+    (property "Datasheet" "~" (id 3) (at 250.825 17.78 0)
+      (effects (font (size 1.27 1.27)) hide)
+    )

Commit message: adsasdas
Parts:
- removed SW?: DTSM31NV, symbol Switch:SW_Push
- added SW?: SW_DIP_x04, symbol Switch:SW_DIP_x04
- added TP?: STR, TestPoint:TestPoint_Pad_2.0x2.0mm, symbol Connector:TestPoint
- added TP?: SEL, TestPoint:TestPoint_Pad_2.0x2.0mm, symbol Connector:TestPoint
- added TP?: BKL, TestPoint:TestPoint_Pad_2.0x2.0mm, symbol Connector:TestPoint
Connections:
- net BTN_BACKLIGHT: now also TP?.1
- net GND: now also SW?.8
- new net GLOBAL_EN: SW?.1
Other:
- note added: "Global_EN when pulled to GND causes pi to 'turn off'"
Changed lines of the file:
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@@
     (stroke (width 0) (type solid) (color 0 0 0 0))
   )
-  (wire (pts (xy 146.685 139.7) (xy 147.955 139.7))
+  (wire (pts (xy 146.685 139.7) (xy 148.59 139.7))
     (stroke (width 0) (type solid) (color 0 0 0 0))
   )
@@
     (stroke (width 0) (type solid) (color 0 0 0 0))
   )
+  (wire (pts (xy 148.59 130.81) (xy 148.59 139.7))
+    (stroke (width 0) (type solid) (color 0 0 0 0))
+  )
+  (wire (pts (xy 148.59 130.81) (xy 154.94 130.81))
+    (stroke (width 0) (type solid) (color 0 0 0 0))
+  )
   (wire (pts (xy 149.86 60.452) (xy 159.385 60.452))
     (stroke (width 0) (type solid) (color 0 0 0 0))
@@
     (stroke (width 0) (type solid) (color 0 0 0 0))
   )
-  (wire (pts (xy 159.385 59.055) (xy 161.925 59.055))
+  (wire (pts (xy 159.385 59.055) (xy 176.53 59.055))
     (stroke (width 0) (type solid) (color 0 0 0 0))
   )
@@
     (stroke (width 0) (type solid) (color 0 0 0 0))
   )
-  (wire (pts (xy 182.245 139.7) (xy 184.15 139.7))
+  (wire (pts (xy 182.245 139.7) (xy 186.69 139.7))
     (stroke (width 0) (type solid) (color 0 0 0 0))
   )
@@
     (stroke (width 0) (type solid) (color 0 0 0 0))
   )
+  (wire (pts (xy 186.69 130.81) (xy 186.69 139.7))
+    (stroke (width 0) (type solid) (color 0 0 0 0))
+  )
+  (wire (pts (xy 186.69 130.81) (xy 194.945 130.81))
+    (stroke (width 0) (type solid) (color 0 0 0 0))
+  )
   (wire (pts (xy 203.835 40.64) (xy 207.645 40.64))
     (stroke (width 0) (type solid) (color 0 0 0 0))
@@
     (stroke (width 0) (type solid) (color 0 0 0 0))
   )
+  (wire (pts (xy 203.835 70.485) (xy 207.645 70.485))
+    (stroke (width 0) (type solid) (color 0 0 0 0))
+  )
   (wire (pts (xy 208.915 114.3) (xy 208.915 115.57))
     (stroke (width 0) (type solid) (color 0 0 0 0))
@@
   )
   (wire (pts (xy 271.78 76.835) (xy 264.16 76.835))
+    (stroke (width 0) (type solid) (color 0 0 0 0))
+  )
+  (wire (pts (xy 272.415 44.45) (xy 262.255 44.45))
+    (stroke (width 0) (type solid) (color 0 0 0 0))
+  )
+  (wire (pts (xy 272.415 54.61) (xy 272.415 44.45))
     (stroke (width 0) (type solid) (color 0 0 0 0))
   )
@@
     (effects (font (size 1.27 1.27)) (justify left bottom))
   )
+  (text "Global_EN when pulled to GND causes pi to 'turn off'"
+    (at 229.235 43.18 0)
+    (effects (font (size 0.508 0.508)) (justify left bottom))
+  )
   (text "Pi reset pin/global_en" (at 256.54 20.32 0)
     (effects (font (size 1.27 1.27)) (justify left bottom))
@@
     (effects (font (size 1.27 1.27)) (justify right bottom))
   )
+  (label "SELECT" (at 148.59 130.81 0)
+    (effects (font (size 1.27 1.27)) (justify left bottom))
+  )
   (label "+3.3v" (at 151.13 56.007 180)
     (effects (font (size 1.27 1.27)) (justify right bottom))
   )
+  (label "BTN_BACKLIGHT" (at 160.02 59.055 0)
+    (effects (font (size 1.27 1.27)) (justify left bottom))
+  )
   (label "+3.3v" (at 173.99 137.16 180)
     (effects (font (size 1.27 1.27)) (justify right bottom))
   )
+  (label "START" (at 186.69 130.81 0)
+    (effects (font (size 1.27 1.27)) (justify left bottom))
+  )
   (label "DPAD_UP" (at 203.835 40.64 180)
     (effects (font (size 1.27 1.27)) (justify right bottom))
@@
   )
   (label "BTN_B" (at 203.835 66.04 180)
+    (effects (font (size 1.27 1.27)) (justify right bottom))
+  )
+  (label "BTN_BACKLIGHT" (at 203.835 70.485 180)
+    (effects (font (size 1.27 1.27)) (justify right bottom))
+  )
+  (label "SELECT" (at 203.835 74.93 180)
+    (effects (font (size 1.27 1.27)) (justify right bottom))
+  )
+  (label "START" (at 203.835 80.645 180)
     (effects (font (size 1.27 1.27)) (justify right bottom))
   )
@@
     (effects (font (size 1.27 1.27)) (justify left))
   )
-  (hierarchical_label "BTN_SELECT" (shape output) (at 147.955 139.7 0)
+  (hierarchical_label "BTN_SELECT" (shape output) (at 154.94 130.81 0)
     (effects (font (size 1.27 1.27)) (justify left))
   )
-  (hierarchical_label "BTN_BACKLIGHT" (shape output) (at 161.925 59.055 0)
+  (hierarchical_label "BTN_BACKLIGHT" (shape output) (at 176.53 59.055 0)
     (effects (font (size 1.27 1.27)) (justify left))
   )
-  (hierarchical_label "BTN_START" (shape output) (at 184.15 139.7 0)
+  (hierarchical_label "BTN_START" (shape output) (at 194.945 130.81 0)
     (effects (font (size 1.27 1.27)) (justify left))
   )
+  (hierarchical_label "GLOBAL_EN" (shape input) (at 247.015 44.45 180)
+    (effects (font (size 1.27 1.27)) (justify right))
+  )
   (symbol (lib_id "Connector:TestPoint") (at 207.645 40.64 270) (unit 1)
     (in_bom yes) (on_board yes)
@@
     )
     (property "Datasheet" "~" (id 3) (at 207.645 71.12 0)
+      (effects (font (size 1.27 1.27)) hide)
+    )
+    (pin "1")
+  )
+  (symbol (lib_id "Connector:TestPoint") (at 207.645 70.485 270) (unit 1)
+    (in_bom yes) (on_board yes)
+    (property "Reference" "TP?" (id 0) (at 208.28 68.5799 90)
+      (effects (font (size 1.27 1.27)) (justify left))
+    )
+    (property "Value" "BKL" (id 1) (at 212.09 70.4849 90)
+      (effects (font (size 1.27 1.27)) (justify left))
+    )
+    (property "Footprint" "TestPoint:TestPoint_Pad_2.0x2.0mm" (id 2) (at 207.645 75.565 0)
+      (effects (font (size 1.27 1.27)) hide)
+    )
+    (property "Datasheet" "~" (id 3) (at 207.645 75.565 0)
+      (effects (font (size 1.27 1.27)) hide)
+    )
+    (pin "1")
+  )
+  (symbol (lib_id "Connector:TestPoint") (at 207.645 74.93 270) (unit 1)
+    (in_bom yes) (on_board yes)
+    (property "Reference" "TP?" (id 0) (at 208.28 73.0249 90)
+      (effects (font (size 1.27 1.27)) (justify left))
+    )
+    (property "Value" "SEL" (id 1) (at 212.09 74.9299 90)
+      (effects (font (size 1.27 1.27)) (justify left))
+    )
+    (property "Footprint" "TestPoint:TestPoint_Pad_2.0x2.0mm" (id 2) (at 207.645 80.01 0)
+      (effects (font (size 1.27 1.27)) hide)
+    )
+    (property "Datasheet" "~" (id 3) (at 207.645 80.01 0)
+      (effects (font (size 1.27 1.27)) hide)
+    )
+    (pin "1")
+  )
+  (symbol (lib_id "Connector:TestPoint") (at 207.645 80.645 270) (unit 1)
+    (in_bom yes) (on_board yes)
+    (property "Reference" "TP?" (id 0) (at 208.28 78.7399 90)
+      (effects (font (size 1.27 1.27)) (justify left))
+    )
+    (property "Value" "STR" (id 1) (at 212.09 80.6449 90)
+      (effects (font (size 1.27 1.27)) (justify left))
+    )
+    (property "Footprint" "TestPoint:TestPoint_Pad_2.0x2.0mm" (id 2) (at 207.645 85.725 0)
+      (effects (font (size 1.27 1.27)) hide)
+    )
+    (property "Datasheet" "~" (id 3) (at 207.645 85.725 0)
       (effects (font (size 1.27 1.27)) hide)
     )
@@
     )
     (property "Datasheet" "" (id 3) (at 254.635 95.885 0)
+      (effects (font (size 1.27 1.27)) hide)
+    )
+    (pin "1")
+  )
+  (symbol (lib_id "power:GND") (at 272.415 54.61 0) (unit 1)
+    (in_bom yes) (on_board yes) (fields_autoplaced)
+    (property "Reference" "#PWR?" (id 0) (at 272.415 60.96 0)
+      (effects (font (size 1.27 1.27)) hide)
+    )
+    (property "Value" "GND" (id 1) (at 272.415 59.055 0))
+    (property "Footprint" "" (id 2) (at 272.415 54.61 0)
+      (effects (font (size 1.27 1.27)) hide)
+    )
+    (property "Datasheet" "" (id 3) (at 272.415 54.61 0)
       (effects (font (size 1.27 1.27)) hide)
     )
@@
     (pin "2")
   )
-  (symbol (lib_id "Switch:SW_Push") (at 250.825 22.86 0) (unit 1)
-    (in_bom yes) (on_board yes) (fields_autoplaced)
-    (property "Reference" "SW?" (id 0) (at 250.825 15.24 0))
-    (property "Value" "DTSM31NV" (id 1) (at 250.825 17.78 0))
-    (property "Footprint" "" (id 2) (at 250.825 17.78 0)
-      (effects (font (size 1.27 1.27)) hide)
-    )
-    (property "Datasheet" "~" (id 3) (at 250.825 17.78 0)
-      (effects (font (size 1.27 1.27)) hide)
-    )
-    (pin "1")
-    (pin "2")
-  )
   (symbol (lib_id "EECBTN:SKRRACE010") (at 24.765 129.54 90) (unit 1)
     (in_bom yes) (on_board yes) (fields_autoplaced)
@@
     (pin "4")
   )
+  (symbol (lib_id "Switch:SW_DIP_x04") (at 254.635 49.53 0) (unit 1)
+    (in_bom yes) (on_board yes) (fields_autoplaced)
+    (property "Reference" "SW?" (id 0) (at 254.635 36.195 0))
+    (property "Value" "SW_DIP_x04" (id 1) (at 254.635 38.735 0))
+    (property "Footprint" "" (id 2) (at 254.635 49.53 0)
+      (effects (font (size 1.27 1.27)) hide)
+    )
+    (property "Datasheet" "~" (id 3) (at 254.635 49.53 0)
+      (effects (font (size 1.27 1.27)) hide)
+    )
+    (pin "1")
+    (pin "2")
+    (pin "3")
+    (pin "4")
+    (pin "5")
+    (pin "6")
+    (pin "7")
+    (pin "8")
+  )
   (symbol (lib_id "TI74HC14N:SN74HC14N") (at 34.29 22.86 0) (unit 1)

Commit message: git pushed
Other:
- note added: "Global_EN when pulled to GND causes pi to 'turn off' - all loads source from pi so there should be no load"
- note added: "This button will be used for GPIO halt / fake sleep mode When device is not in use GLOBAL_EN should still be pulled low"
- note added: "We will use a dip switch for this because lazy, can position it so its hidden under that battery tray"
- note added: "chs-04ta"
- note removed: "Global_EN when pulled to GND causes pi to 'turn off'"
Changed lines of the file:
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@@
     (title "Gamepad buttons")
     (rev "indev")
-    (comment 1 "https://www.github.com/cinnamondev/gamepithing")
   )
   (junction (at 24.765 129.54) (diameter 0.9144) (color 0 0 0 0))
@@
     (effects (font (size 1.27 1.27)) (justify left bottom))
   )
-  (text "Global_EN when pulled to GND causes pi to 'turn off'"
-    (at 229.235 43.18 0)
+  (text "This button will be used for GPIO halt / fake sleep mode\nWhen device is not in use GLOBAL_EN should still be pulled low"
+    (at 132.08 88.9 0)
+    (effects (font (size 1.27 1.27)) (justify left bottom))
+  )
+  (text "We will use a dip switch for this because lazy, can position it so its hidden under that battery tray"
+    (at 186.69 15.24 0)
+    (effects (font (size 1.27 1.27)) (justify left bottom))
+  )
+  (text "Global_EN when pulled to GND causes pi to 'turn off' - all \nloads source from pi so there should be no load"
+    (at 227.33 42.545 0)
     (effects (font (size 0.508 0.508)) (justify left bottom))
   )
-  (text "Pi reset pin/global_en" (at 256.54 20.32 0)
-    (effects (font (size 1.27 1.27)) (justify left bottom))
-  )
+  (text "Pi reset pin/global_en" (at 243.205 34.29 0)
+    (effects (font (size 1.27 1.27)) (justify left bottom))
+  )
+  (text "chs-04ta\n" (at 262.255 41.275 0)
+    (effects (font (size 1.27 1.27)) (justify left bottom))
+  )
