File: sch/carrier/gamepad.kicad_sch (KiCad schematic)
At the start: 47 parts, among them SW1 SKRRACE010, SW2 SKRRACE010, SW3 SKRRACE010, SW4 SKRRACE010, SW5 SKRRACE010, SW6 SKRRACE010, SW7 SKRBAAE010, U1 SN74HC14N

Commit message: aaaaaaaaaaaaaa
Parts:
- added C? (x2): 0.1uF, Capacitor_SMD:C_0504_1310Metric_Pad0.83x1.28mm_HandSolder, symbol Device:C
- added R? (x2): 10k, Resistor_SMD:R_0805_2012Metric_Pad1.20x1.40mm_HandSolder, symbol Device:R
- added R? (x2): 1k, Resistor_SMD:R_0805_2012Metric_Pad1.20x1.40mm_HandSolder, symbol Device:R
- added SW? (x2): SW_Push, sw:TE_Connectivity-1-1825027-1-0-0-Recommended_Land_Pattern_, symbol Switch:SW_Push
- added TP?: R, TestPoint:TestPoint_Pad_2.0x2.0mm, symbol Connector:TestPoint
- added TP?: L, TestPoint:TestPoint_Pad_2.0x2.0mm, symbol Connector:TestPoint
Connections:
- net +3.3v: now also R?.1, R?.1
- net BTN_SELECT: now also TP?.1
- net BTN_START: now also TP?.1
- net GND: now also C?.2, C?.2, SW?.1, SW?.1
- new net: R?.1, SW?.2 (x2)
- new net SHOULDER_L: C?.1, R?.2, R?.2, TP?.1
- new net SHOULDER_R: C?.1, R?.2, R?.2, TP?.1
Other:
- moved on the sheet: SW?, TP10, TP11, TP6, TP7, TP8, TP9, TP?

Commit message: ersfdxcv
Parts:
- TP10, TP11, TP6, TP7, TP8, TP9: footprint TestPoint:TestPoint_Pad_2.0x2.0mm -> TestPoint:TestPoint_Pad_1.0x1.0mm
- TP14, TP15, TP16, TP17, TP18: renamed from TP?; footprint TestPoint:TestPoint_Pad_2.0x2.0mm -> TestPoint:TestPoint_Pad_1.0x1.0mm
- gave numbers to parts that had none: 20

Commit message: footprint assignmnt
Parts:
- C1, C10, C2, C3, C4, C5, C6: footprint Capacitor_SMD:C_0504_1310Metric_Pad0.83x1.28mm_HandSolder -> Capacitor_SMD:C_0402_1005Metric_Pad0.74x0.62mm_HandSolder
- R1, R10, R11, R12, R2, R26, R27, R28, R29, R3, R30, R31, R32, R33, R34, R35, R4, R5, R6, R7, R8, R9: footprint Resistor_SMD:R_0805_2012Metric_Pad1.20x1.40mm_HandSolder -> Resistor_SMD:R_0402_1005Metric_Pad0.72x0.64mm_HandSolder
Other:
- note added: "0.0025"

Commit message: a
Changed lines of the file:
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@@
   )
   (text "0.0025" (at 26.035 102.87 180)
-    (effects (font (size 1.27 1.27)))
+    (effects (font (size 1.27 1.27)) (justify right bottom))
   )
   (text "This button will be used for GPIO halt / fake sleep mode\nWhen device is not in use GLOBAL_EN should still be pulled low"

Commit message: aaaaaaaaaaaaaaaaaaaaaaaaaaaaaaaa
Parts:
- SW12: footprint (none) -> dipswitch:CHS04TA1
Connections:
- net GND: now also SW1.4, SW10.4, SW3.4, SW4.4, SW5.4, SW6.4, SW8.4
- net at R9.1, SW5.3: now also SW5.1
- net at SW6.1: now also R11.1, SW6.3
- net at R26.1, SW7.3: now also SW7.1
- net at SW1.1: now also R1.1, SW1.3
- net at SW10.1: now also R32.1, SW10.3
- net at R4.1, SW3.3: now also SW3.1
- net at SW2.1: now also R3.1, SW2.3
- net at SW4.1: now also R7.1, SW4.3
- net at SW8.1: now also R28.1, SW8.3
Other:
- note added: "chs-04ta1"
- note removed: "chs-04ta"
- moved on the sheet: C11, SW8

Commit message: pcb time?
Parts:
- C11, C12, C13, C14: footprint Capacitor_SMD:C_0504_1310Metric_Pad0.83x1.28mm_HandSolder -> Capacitor_SMD:C_0402_1005Metric_Pad0.74x0.62mm_HandSolder
Changed lines of the file:
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@@
       (effects (font (size 1.27 1.27)) (justify left))
     )
-    (property "Footprint" "Capacitor_SMD:C_0504_1310Metric_Pad0.83x1.28mm_HandSolder" (id 2) (at 160.3502 73.025 0)
+    (property "Footprint" "Capacitor_SMD:C_0402_1005Metric_Pad0.74x0.62mm_HandSolder" (id 2) (at 160.3502 73.025 0)
       (effects (font (size 1.27 1.27)) hide)
     )
@@
       (effects (font (size 1.27 1.27)) (justify left))
     )
-    (property "Footprint" "Capacitor_SMD:C_0504_1310Metric_Pad0.83x1.28mm_HandSolder" (id 2) (at 161.6202 44.45 0)
+    (property "Footprint" "Capacitor_SMD:C_0402_1005Metric_Pad0.74x0.62mm_HandSolder" (id 2) (at 161.6202 44.45 0)
       (effects (font (size 1.27 1.27)) hide)
     )
@@
       (effects (font (size 1.27 1.27)) (justify left))
     )
-    (property "Footprint" "Capacitor_SMD:C_0504_1310Metric_Pad0.83x1.28mm_HandSolder" (id 2) (at 183.2102 153.67 0)
+    (property "Footprint" "Capacitor_SMD:C_0402_1005Metric_Pad0.74x0.62mm_HandSolder" (id 2) (at 183.2102 153.67 0)
       (effects (font (size 1.27 1.27)) hide)
     )
@@
       (effects (font (size 1.27 1.27)) (justify left))
     )
-    (property "Footprint" "Capacitor_SMD:C_0504_1310Metric_Pad0.83x1.28mm_HandSolder" (id 2) (at 234.0102 61.595 0)
+    (property "Footprint" "Capacitor_SMD:C_0402_1005Metric_Pad0.74x0.62mm_HandSolder" (id 2) (at 234.0102 61.595 0)
       (effects (font (size 1.27 1.27)) hide)
     )

Commit message: a
Connections:
- net GND: now also SW2.4, SW7.4
Changed lines of the file:
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@@
   (junction (at 46.99 155.575) (diameter 0.9144) (color 0 0 0 0))
   (junction (at 51.435 78.74) (diameter 0.9144) (color 0 0 0 0))
+  (junction (at 51.435 98.425) (diameter 0.9144) (color 0 0 0 0))
   (junction (at 52.07 138.43) (diameter 0.9144) (color 0 0 0 0))
   (junction (at 52.07 155.575) (diameter 0.9144) (color 0 0 0 0))
@@
   (junction (at 124.46 158.75) (diameter 0.9144) (color 0 0 0 0))
   (junction (at 129.54 141.605) (diameter 0.9144) (color 0 0 0 0))
+  (junction (at 129.54 158.75) (diameter 0.9144) (color 0 0 0 0))
   (junction (at 133.35 49.53) (diameter 0.9144) (color 0 0 0 0))
   (junction (at 136.525 78.74) (diameter 0.9144) (color 0 0 0 0))
@@
     (stroke (width 0) (type solid) (color 0 0 0 0))
   )
-  (wire (pts (xy 46.355 98.425) (xy 68.58 98.425))
+  (wire (pts (xy 46.355 98.425) (xy 51.435 98.425))
     (stroke (width 0) (type solid) (color 0 0 0 0))
   )
@@
     (stroke (width 0) (type solid) (color 0 0 0 0))
   )
+  (wire (pts (xy 51.435 93.98) (xy 51.435 98.425))
+    (stroke (width 0) (type solid) (color 0 0 0 0))
+  )
+  (wire (pts (xy 51.435 98.425) (xy 68.58 98.425))
+    (stroke (width 0) (type solid) (color 0 0 0 0))
+  )
   (wire (pts (xy 52.07 153.67) (xy 52.07 155.575))
     (stroke (width 0) (type solid) (color 0 0 0 0))
@@
     (stroke (width 0) (type solid) (color 0 0 0 0))
   )
+  (wire (pts (xy 129.54 156.845) (xy 129.54 158.75))
+    (stroke (width 0) (type solid) (color 0 0 0 0))
+  )
+  (wire (pts (xy 129.54 158.75) (xy 124.46 158.75))
+    (stroke (width 0) (type solid) (color 0 0 0 0))
+  )
   (wire (pts (xy 133.35 32.385) (xy 133.35 49.53))
     (stroke (width 0) (type solid) (color 0 0 0 0))
@@
     (stroke (width 0) (type solid) (color 0 0 0 0))
   )
-  (wire (pts (xy 146.685 158.75) (xy 124.46 158.75))
+  (wire (pts (xy 146.685 158.75) (xy 129.54 158.75))
     (stroke (width 0) (type solid) (color 0 0 0 0))
   )
@@
     (in_bom yes) (on_board yes)
     (property "Reference" "R12" (id 0) (at 259.715 71.755 90))
-    (property "Value" "10k" (id 1) (at 259.715 74.93 90))
+    (property "Value" "10k" (id 1) (at 259.715 74.93 0))
     (property "Footprint" "Resistor_SMD:R_0402_1005Metric_Pad0.72x0.64mm_HandSolder" (id 2) (at 259.715 76.708 90)
       (effects (font (size 1.27 1.27)) hide)

Commit message: aa
Parts:
- U1: footprint TI74HC14N:Texas_Instruments-R_R-PDIP-T14-0-0-0 -> Package_SO:SO-14_3.9x8.65mm_P1.27mm
Connections:
- net DPAD_DOWN: now also U1.6 (3Y); no longer U1.4 (2Y)
- net DPAD_LEFT: now also U1.8 (4Y); no longer U1.6 (3Y)
- net DPAD_RIGHT: now also U1.4 (2Y); no longer U1.8 (4Y)
- net __DP_D: now also U1.5 (3A); no longer U1.3 (2A)
- net __DP_L: now also U1.9 (4A); no longer U1.5 (3A)
- net __DP_R: now also U1.3 (2A); no longer U1.9 (4A)
Changed lines of the file:
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@@
   )
   (text "TODO: consider getting rid of this?? we already have a RC network to help with debounce do we really need this\n"
-    (at 17.145 47.625 0)
+    (at 17.145 48.26 0)
     (effects (font (size 1.27 1.27)) (justify left bottom))
   )
@@
     (effects (font (size 1.27 1.27)) (justify left bottom))
   )
-  (label "__DP_D" (at 29.21 30.48 0)
+  (label "__DP_R" (at 29.21 30.48 0)
     (effects (font (size 1.27 1.27)) (justify left bottom))
   )
-  (label "__DP_L" (at 29.21 33.02 0)
+  (label "__DP_D" (at 29.21 33.02 0)
     (effects (font (size 1.27 1.27)) (justify left bottom))
   )
-  (label "__DP_R" (at 29.21 35.56 0)
+  (label "__DP_L" (at 29.21 35.56 0)
     (effects (font (size 1.27 1.27)) (justify left bottom))
   )
@@
     (effects (font (size 1.27 1.27)) (justify right bottom))
   )
-  (label "DPAD_DOWN" (at 70.485 25.4 180)
-    (effects (font (size 1.27 1.27)) (justify right bottom))
-  )
-  (label "DPAD_LEFT" (at 70.485 27.94 180)
-    (effects (font (size 1.27 1.27)) (justify right bottom))
-  )
-  (label "DPAD_RIGHT" (at 70.485 30.48 180)
+  (label "DPAD_RIGHT" (at 70.485 25.4 180)
+    (effects (font (size 1.27 1.27)) (justify right bottom))
+  )
+  (label "DPAD_DOWN" (at 70.485 27.94 180)
+    (effects (font (size 1.27 1.27)) (justify right bottom))
+  )
+  (label "DPAD_LEFT" (at 70.485 30.48 180)
     (effects (font (size 1.27 1.27)) (justify right bottom))
   )
@@
     (effects (font (size 1.27 1.27)) (justify left))
   )
-  (hierarchical_label "DPAD_DOWN" (shape output) (at 70.485 25.4 0)
+  (hierarchical_label "DPAD_RIGHT" (shape output) (at 70.485 25.4 0)
     (effects (font (size 1.27 1.27)) (justify left))
   )
-  (hierarchical_label "DPAD_LEFT" (shape output) (at 70.485 27.94 0)
+  (hierarchical_label "DPAD_DOWN" (shape output) (at 70.485 27.94 0)
     (effects (font (size 1.27 1.27)) (justify left))
   )
-  (hierarchical_label "DPAD_RIGHT" (shape output) (at 70.485 30.48 0)
+  (hierarchical_label "DPAD_LEFT" (shape output) (at 70.485 30.48 0)
     (effects (font (size 1.27 1.27)) (justify left))
   )
@@
     (property "Reference" "U1" (id 0) (at 48.26 14.605 0))
     (property "Value" "SN74HC14N" (id 1) (at 48.26 17.145 0))
-    (property "Footprint" "TI74HC14N:Texas_Instruments-R_R-PDIP-T14-0-0-0" (id 2) (at 34.29 12.7 0)
-      (effects (font (size 1.27 1.27)) (justify left) hide)
-    )
+    (property "Footprint" "Package_SO:SO-14_3.9x8.65mm_P1.27mm" (id 2) (at 34.29 12.7 0)
+      (effects (font (size 1.27 1.27)) (justify left) hide)
+    )
