File: sch/carrier/stmcontrol.kicad_sch (KiCad schematic)
At the start: 0 parts

Commit message: a
Other:
- note added: "IGNORE THIS SHEET"
Changed lines of the file:
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@@
     (title "STM32 control subsystem")
   )
+  (text "IGNORE THIS SHEET" (at 104.775 99.695 0)
+    (effects (font (size 5.08 5.08)) (justify left bottom))
+  )
 )
