File: sch/carrier/power.kicad_sch (KiCad schematic)
At the start: 32 parts, among them J4 USB_C_Receptacle_USB2.0, U3 MP2636GR-P

Commit message: :)
Parts:
- removed C?: C, symbol Device:C
- removed R? (x2): R, symbol Device:R
- removed TH?: Thermistor_NTC, symbol Device:Thermistor_NTC
- added R? (x6): 10.5k, symbol Device:R
- L?: value L -> 6.8uH
- NT?: value NetTie_2 -> NetTie; footprint (none) -> NetTie:NetTie-2_SMD_Pad0.5mm
- R?: value R -> 10k
- R?: value R -> 55.2k
- R?: value R -> 3k
Connections:
- net 5v: now also R?.1
- net GND: now also C?.2, C?.2
- net GNDA: now also R?.2, R?.2
- net _CHIP_VCC: now also R?.1, R?.1, R?.1
- net at U3.12 (NTC): now also R?.1, R?.2
- net at U3.16 (VB): now also R?.1, R?.2
- net at U3.24 (MODE): now also R?.2
- net at U3.25 (EN): now also R?.2
- net at U3.6 (ILIM): now also R?.1
Other:
- note added: "(nice)"
- note added: "For further understanding, Chip VCC is the INTERNAL supply!"
- note added: "Keeps within the NTC window. CBA"
- note added: "some figures so dont need to keep hunting for f(sw)=600khz"
- moved on the sheet: C?, NT?

Commit message: get git committed
Parts:
- removed J4: USB_C_Receptacle_USB2.0, Connector_USB:USB_C_Receptacle_JAE_DX07S016JA1R1500, symbol Connector:USB_C_Receptacle_USB2.0
- removed R14: 0, symbol Device:R
- removed R20, R21: 5.1k, Resistor_SMD:R_0805_2012Metric_Pad1.20x1.40mm_HandSolder, symbol Device:R
- added C?: 0.47uF, symbol Device:C
- added U?: BQ27441DRZR-G1B, Package_SON:Texas_S-PDSO-N12, symbol Battery_Management:BQ27441DRZR-G1B
Connections:
- net FUEL_SCL: now also U?.2 (SCL)
- net FUEL_SDA: now also U?.1 (SDA)
- net GND: now also R?.2, C?.2
- net BATT+ renamed VBATT+
- new net: C?.1, U?.3 (VSS), U?.5 (VDD)
- no-connect marks 7 -> 1
Other:
- note added: "BATT will be a 3000mAh 3.7v nomimal LiPo battery (if we can get larger will do) (reckon we can squeeze a 4200mAh in with some modifications (gut out the battery cage, min)"
- note added: "I'm not sure if we actually need this layout but apparently you should (GNDA is analogue ground)"
- note added: "chip VCC is the INTERNAL supply!"
- note added: "revise later??"
- note added: "worth noting our battery bank is to have its own protection circuitry so it can be omitted"
- note removed: "(nice)"
- note removed: "BATT will be a 3000mAh 3.7v nomimal LiPo battery (if we can get larger will do) (reckon we can squeeze a 4200mAh in with some modifications (gut out the battery cage)"
- note removed: "For further understanding, Chip VCC is the INTERNAL supply!"
- note removed: "No data"
- note removed: "This version of the battery sheet used the MP2636 IC - will be WAY better."
- note removed: "Too many people on stack overflow/exchange seem to be unable to agree on this! Leaving this unconnected with a 0 ohm so we can if we choose to."
- note removed: "revise later"
- moved on the sheet: R?

Commit message: aaaaaaaaaaaaaaaa
Parts:
- removed C?: 0.47uF, symbol Device:C
- removed U?: BQ27441DRZR-G1B, Package_SON:Texas_S-PDSO-N12, symbol Battery_Management:BQ27441DRZR-G1B
Connections:
- net VBATT+ renamed BATT
- net VBUS renamed CHRG
Other:
- note removed: "worth noting our battery bank is to have its own protection circuitry so it can be omitted"
Changed lines of the file:
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@@
   (junction (at 147.955 36.83) (diameter 0.9144) (color 0 0 0 0))
   (junction (at 150.495 101.6) (diameter 0.9144) (color 0 0 0 0))
-  (junction (at 151.13 166.37) (diameter 0.9144) (color 0 0 0 0))
   (junction (at 156.845 36.83) (diameter 0.9144) (color 0 0 0 0))
   (junction (at 175.895 55.88) (diameter 0.9144) (color 0 0 0 0))
@@
     (stroke (width 0) (type solid) (color 0 0 0 0))
   )
-  (wire (pts (xy 128.27 166.37) (xy 151.13 166.37))
-    (stroke (width 0) (type solid) (color 0 0 0 0))
-  )
   (wire (pts (xy 137.795 26.035) (xy 137.795 36.83))
     (stroke (width 0) (type solid) (color 0 0 0 0))
@@
     (stroke (width 0) (type solid) (color 0 0 0 0))
   )
-  (wire (pts (xy 143.51 143.51) (xy 151.13 143.51))
-    (stroke (width 0) (type solid) (color 0 0 0 0))
-  )
   (wire (pts (xy 147.955 36.83) (xy 147.32 36.83))
     (stroke (width 0) (type solid) (color 0 0 0 0))
@@
   )
   (wire (pts (xy 150.495 101.6) (xy 152.4 101.6))
-    (stroke (width 0) (type solid) (color 0 0 0 0))
-  )
-  (wire (pts (xy 151.13 143.51) (xy 151.13 166.37))
-    (stroke (width 0) (type solid) (color 0 0 0 0))
-  )
-  (wire (pts (xy 151.13 166.37) (xy 151.13 169.545))
     (stroke (width 0) (type solid) (color 0 0 0 0))
   )
@@
     (effects (font (size 0.635 0.635)) (justify left bottom))
   )
-  (text "worth noting our battery bank is to have its own\nprotection circuitry so it can be omitted"
-    (at 69.85 175.895 0)
-    (effects (font (size 1.27 1.27)) (justify left bottom))
-  )
   (text "Based of the MP2636 datasheet." (at 78.105 40.005 0)
     (effects (font (size 1.905 1.905)) (justify left bottom))
@@
     (effects (font (size 1.27 1.27)) (justify left bottom))
   )
-  (label "VSYS" (at 69.85 140.97 180)
-    (effects (font (size 1.27 1.27)) (justify right bottom))
-  )
   (label "VSYS" (at 201.93 26.035 180)
     (effects (font (size 1.27 1.27)) (justify right bottom))
@@
     (effects (font (size 1.27 1.27)) (justify right bottom))
   )
-  (label "VBATT+" (at 268.605 55.88 180)
-    (effects (font (size 1.27 1.27)) (justify right bottom))
-  )
   (label "BATT-" (at 270.51 73.025 180)
     (effects (font (size 1.27 1.27)) (justify right bottom))
   )
-  (hierarchical_label "VBUS" (shape input) (at 24.765 55.88 180)
-    (effects (font (size 1.27 1.27)) (justify right))
-  )
-  (hierarchical_label "FUEL_SDA" (shape bidirectional) (at 113.03 146.05 180)
-    (effects (font (size 1.27 1.27)) (justify right))
-  )
-  (hierarchical_label "FUEL_SCL" (shape input) (at 113.03 148.59 180)
+  (hierarchical_label "CHRG" (shape input) (at 24.765 55.88 180)
     (effects (font (size 1.27 1.27)) (justify right))
   )
@@
     (effects (font (size 1.27 1.27)) (justify left))
   )
+  (hierarchical_label "BATT" (shape bidirectional) (at 268.605 55.88 0)
+    (effects (font (size 1.27 1.27)) (justify left))
+  )
   (symbol (lib_id "Device:NetTie_2") (at 146.685 118.745 90) (unit 1)
     (in_bom yes) (on_board yes) (fields_autoplaced)
@@
     )
     (property "Datasheet" "" (id 3) (at 146.685 121.285 0)
-      (effects (font (size 1.27 1.27)) hide)
-    )
-    (pin "1")
-  )
-  (symbol (lib_id "power:GND") (at 151.13 177.165 0) (unit 1)
-    (in_bom yes) (on_board yes) (fields_autoplaced)
-    (property "Reference" "#PWR?" (id 0) (at 151.13 183.515 0)
-      (effects (font (size 1.27 1.27)) hide)
-    )
-    (property "Value" "GND" (id 1) (at 151.13 181.61 0))
-    (property "Footprint" "" (id 2) (at 151.13 177.165 0)
-      (effects (font (size 1.27 1.27)) hide)
-    )
-    (property "Datasheet" "" (id 3) (at 151.13 177.165 0)
       (effects (font (size 1.27 1.27)) hide)
     )
@@
     (pin "2")
   )
-  (symbol (lib_id "Device:C") (at 151.13 173.355 0) (unit 1)
-    (in_bom yes) (on_board yes) (fields_autoplaced)
-    (property "Reference" "C?" (id 0) (at 154.94 172.0849 0)
-      (effects (font (size 1.27 1.27)) (justify left))
-    )
-    (property "Value" "0.47uF" (id 1) (at 154.94 174.6249 0)
-      (effects (font (size 1.27 1.27)) (justify left))
-    )
-    (property "Footprint" "" (id 2) (at 152.0952 177.165 0)
-      (effects (font (size 1.27 1.27)) hide)
-    )
-    (property "Datasheet" "~" (id 3) (at 151.13 173.355 0)
-      (effects (font (size 1.27 1.27)) hide)
-    )
-    (pin "1")
-    (pin "2")
-  )
   (symbol (lib_id "Device:C") (at 175.895 97.155 0) (unit 1)
     (in_bom yes) (on_board yes) (fields_autoplaced)
@@
     (pin "2")
   )
-  (symbol (lib_id "Battery_Management:BQ27441DRZR-G1B") (at 128.27 151.13 0) (unit 1)
-    (in_bom yes) (on_board yes) (fields_autoplaced)
-    (property "Reference" "U?" (id 0) (at 128.27 133.35 0))
-    (property "Value" "BQ27441DRZR-G1B" (id 1) (at 128.27 135.89 0))
-    (property "Footprint" "Package_SON:Texas_S-PDSO-N12" (id 2) (at 134.62 165.1 0)
-      (effects (font (size 1.27 1.27)) (justify left) hide)
-    )
-    (property "Datasheet" "http://www.ti.com/lit/ds/symlink/bq27441-g1.pdf" (id 3) (at 133.35 146.05 0)
-      (effects (font (size 1.27 1.27)) hide)
-    )
-    (pin "1")
-    (pin "10")
-    (pin "11")
-    (pin "12")
-    (pin "13")
-    (pin "2")
-    (pin "3")
-    (pin "4")
-    (pin "5")
-    (pin "6")
-    (pin "7")
-    (pin "8")
-    (pin "9")
-  )
   (symbol (lib_id "mp2636:MP2636GR-P") (at 146.685 81.28 0) (unit 1)

Commit message: add speaker and charger
Parts:
- added TP?: +5v Output, symbol Connector:TestPoint
Changed lines of the file:
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@@
     (effects (font (size 1.27 1.27)) (justify left))
   )
-  (hierarchical_label "BATT" (shape bidirectional) (at 268.605 55.88 0)
+  (hierarchical_label "BATT" (shape input) (at 268.605 55.88 0)
     (effects (font (size 1.27 1.27)) (justify left))
   )
@@
     (pin "1")
     (pin "2")
+  )
+  (symbol (lib_id "Connector:TestPoint") (at 203.835 26.035 180) (unit 1)
+    (in_bom yes) (on_board yes)
+    (property "Reference" "TP?" (id 0) (at 200.025 27.8764 0)
+      (effects (font (size 1.27 1.27)) (justify right))
+    )
+    (property "Value" "+5v Output" (id 1) (at 199.39 31.0514 0)
+      (effects (font (size 1.27 1.27)) (justify right))
+    )
+    (property "Footprint" "" (id 2) (at 198.755 26.035 0)
+      (effects (font (size 1.27 1.27)) hide)
+    )
+    (property "Datasheet" "~" (id 3) (at 198.755 26.035 0)
+      (effects (font (size 1.27 1.27)) hide)
+    )
+    (pin "1")
   )
   (symbol (lib_id "power:GND") (at 30.48 76.835 0) (unit 1)
@@
       (effects (font (size 1.27 1.27)) hide)
     )
-    (pin "1")
-  )
-  (symbol (lib_id "power:GND") (at 215.265 132.715 0) (unit 1)
-    (in_bom yes) (on_board yes) (fields_autoplaced)
-    (property "Reference" "#PWR?" (id 0) (at 215.265 139.065 0)
-      (effects (font (size 1.27 1.27)) hide)
-    )
-    (property "Value" "GND" (id 1) (at 215.265 137.16 0))
-    (property "Footprint" "" (id 2) (at 215.265 132.715 0)
-      (effects (font (size 1.27 1.27)) hide)
-    )
-    (property "Datasheet" "" (id 3) (at 215.265 132.715 0)
-      (effects (font (size 1.27 1.27)) hide)
-    )

Commit message: git pushed
Changed lines of the file:
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@@
     (title "Power and battery")
     (rev "indev")
-    (comment 1 "https://www.github.com/cinnamondev/gamepithing")
   )
   (junction (at 30.48 55.88) (diameter 0.9144) (color 0 0 0 0))
@@
     (effects (font (size 1.27 1.27)) (justify left))
   )
-  (hierarchical_label "BATT" (shape input) (at 268.605 55.88 0)
+  (hierarchical_label "BATT" (shape bidirectional) (at 268.605 55.88 0)
     (effects (font (size 1.27 1.27)) (justify left))
   )

Commit message: ersfdxcv
Parts:
- D2, D3: renamed from D?; footprint (none) -> LED_SMD:LED_0805_2012Metric_Pad1.15x1.40mm_HandSolder
- L1: renamed from L?; footprint (none) -> Inductor_SMD:L_Wuerth_WE-PD-Typ-M-Typ-S_Handsoldering
- TP19: renamed from TP?; footprint (none) -> TestPoint:TestPoint_Pad_1.0x1.0mm
- U3: footprint IC_MP2636GR-P -> mp2636:IC_MP2636GR-P
- gave numbers to parts that had none: 26

Commit message: a
Parts:
- R36, R37, R38, R39: footprint (none) -> Resistor_SMD:R_0402_1005Metric_Pad0.72x0.64mm_HandSolder
- R40, R41, R42, R43, R44, R45, R46, R47, R48, R49, R50, R51, R52, R53, R54: footprint (none) -> Resistor_SMD:R_0603_1608Metric_Pad0.98x0.95mm_HandSolder
Changed lines of the file:
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@@
       (effects (font (size 1.27 1.27)) (justify left))
     )
-    (property "Footprint" "" (id 2) (at 42.672 59.69 90)
+    (property "Footprint" "Resistor_SMD:R_0402_1005Metric_Pad0.72x0.64mm_HandSolder" (id 2) (at 42.672 59.69 90)
       (effects (font (size 1.27 1.27)) hide)
     )
@@
       (effects (font (size 1.27 1.27)) (justify left))
     )
-    (property "Footprint" "" (id 2) (at 42.672 73.025 90)
+    (property "Footprint" "Resistor_SMD:R_0402_1005Metric_Pad0.72x0.64mm_HandSolder" (id 2) (at 42.672 73.025 90)
       (effects (font (size 1.27 1.27)) hide)
     )
@@
       (effects (font (size 1.27 1.27)) (justify left))
     )
-    (property "Footprint" "" (id 2) (at 52.832 59.69 90)
+    (property "Footprint" "Resistor_SMD:R_0402_1005Metric_Pad0.72x0.64mm_HandSolder" (id 2) (at 52.832 59.69 90)
       (effects (font (size 1.27 1.27)) hide)
     )
@@
       (effects (font (size 1.27 1.27)) (justify left))
     )
-    (property "Footprint" "" (id 2) (at 52.832 73.025 90)
+    (property "Footprint" "Resistor_SMD:R_0402_1005Metric_Pad0.72x0.64mm_HandSolder" (id 2) (at 52.832 73.025 90)
       (effects (font (size 1.27 1.27)) hide)
     )
@@
     (property "Reference" "R40" (id 0) (at 93.98 78.105 90))
     (property "Value" "10.5k" (id 1) (at 93.98 80.01 90))
-    (property "Footprint" "" (id 2) (at 93.98 81.788 90)
+    (property "Footprint" "Resistor_SMD:R_0603_1608Metric_Pad0.98x0.95mm_HandSolder" (id 2) (at 93.98 81.788 90)
       (effects (font (size 1.27 1.27)) hide)
     )
@@
     (property "Reference" "R41" (id 0) (at 93.98 83.82 90))
     (property "Value" "10.5k" (id 1) (at 93.98 85.725 90))
-    (property "Footprint" "" (id 2) (at 93.98 87.503 90)
+    (property "Footprint" "Resistor_SMD:R_0603_1608Metric_Pad0.98x0.95mm_HandSolder" (id 2) (at 93.98 87.503 90)
       (effects (font (size 1.27 1.27)) hide)
     )
@@
       (effects (font (size 1.27 1.27)) (justify left))
     )
-    (property "Footprint" "" (id 2) (at 114.427 88.9 90)
+    (property "Footprint" "Resistor_SMD:R_0603_1608Metric_Pad0.98x0.95mm_HandSolder" (id 2) (at 114.427 88.9 90)
       (effects (font (size 1.27 1.27)) hide)
     )
@@
     (property "Reference" "R43" (id 0) (at 143.51 34.29 90))
     (property "Value" "10k" (id 1) (at 143.51 36.83 90))
-    (property "Footprint" "" (id 2) (at 143.51 35.052 90)
+    (property "Footprint" "Resistor_SMD:R_0603_1608Metric_Pad0.98x0.95mm_HandSolder" (id 2) (at 143.51 35.052 90)
       (effects (font (size 1.27 1.27)) hide)
     )
@@
     (property "Reference" "R44" (id 0) (at 152.4 34.29 90))
     (property "Value" "3k" (id 1) (at 152.4 36.83 90))
-    (property "Footprint" "" (id 2) (at 152.4 38.608 90)
+    (property "Footprint" "Resistor_SMD:R_0603_1608Metric_Pad0.98x0.95mm_HandSolder" (id 2) (at 152.4 38.608 90)
       (effects (font (size 1.27 1.27)) hide)
     )
@@
       (effects (font (size 1.27 1.27)) (justify right))
     )
-    (property "Footprint" "" (id 2) (at 166.243 41.91 90)
+    (property "Footprint" "Resistor_SMD:R_0603_1608Metric_Pad0.98x0.95mm_HandSolder" (id 2) (at 166.243 41.91 90)
       (effects (font (size 1.27 1.27)) hide)
     )
@@
       (effects (font (size 1.27 1.27)) (justify left))
     )
-    (property "Footprint" "" (id 2) (at 184.277 97.155 90)
+    (property "Footprint" "Resistor_SMD:R_0603_1608Metric_Pad0.98x0.95mm_HandSolder" (id 2) (at 184.277 97.155 90)
       (effects (font (size 1.27 1.27)) hide)
     )
@@
     (property "Reference" "R47" (id 0) (at 192.405 53.34 90))
     (property "Value" "20m" (id 1) (at 192.405 55.88 90))
-    (property "Footprint" "" (id 2) (at 192.405 57.658 90)
+    (property "Footprint" "Resistor_SMD:R_0603_1608Metric_Pad0.98x0.95mm_HandSolder" (id 2) (at 192.405 57.658 90)
       (effects (font (size 1.27 1.27)) hide)
     )
@@
       (effects (font (size 1.27 1.27)) (justify left))
     )
-    (property "Footprint" "" (id 2) (at 196.977 97.79 90)
+    (property "Footprint" "Resistor_SMD:R_0603_1608Metric_Pad0.98x0.95mm_HandSolder" (id 2) (at 196.977 97.79 90)
       (effects (font (size 1.27 1.27)) hide)
     )
@@
       (effects (font (size 1.27 1.27)) (justify left))
     )
-    (property "Footprint" "" (id 2) (at 207.772 97.79 90)
+    (property "Footprint" "Resistor_SMD:R_0603_1608Metric_Pad0.98x0.95mm_HandSolder" (id 2) (at 207.772 97.79 90)
       (effects (font (size 1.27 1.27)) hide)
     )
@@
       (effects (font (size 1.27 1.27)) (justify left))
     )
-    (property "Footprint" "" (id 2) (at 219.202 97.79 90)
+    (property "Footprint" "Resistor_SMD:R_0603_1608Metric_Pad0.98x0.95mm_HandSolder" (id 2) (at 219.202 97.79 90)
       (effects (font (size 1.27 1.27)) hide)
     )
@@
       (effects (font (size 1.27 1.27)) (justify left))
     )
-    (property "Footprint" "" (id 2) (at 231.902 90.17 90)
+    (property "Footprint" "Resistor_SMD:R_0603_1608Metric_Pad0.98x0.95mm_HandSolder" (id 2) (at 231.902 90.17 90)
       (effects (font (size 1.27 1.27)) hide)
     )
@@
       (effects (font (size 1.27 1.27)) (justify left))
     )
-    (property "Footprint" "" (id 2) (at 231.902 97.79 90)
+    (property "Footprint" "Resistor_SMD:R_0603_1608Metric_Pad0.98x0.95mm_HandSolder" (id 2) (at 231.902 97.79 90)
       (effects (font (size 1.27 1.27)) hide)
     )
@@
       (effects (font (size 1.27 1.27)) (justify left))
     )
-    (property "Footprint" "" (id 2) (at 250.952 90.17 90)
+    (property "Footprint" "Resistor_SMD:R_0603_1608Metric_Pad0.98x0.95mm_HandSolder" (id 2) (at 250.952 90.17 90)
       (effects (font (size 1.27 1.27)) hide)
     )
@@
       (effects (font (size 1.27 1.27)) (justify left))
     )
-    (property "Footprint" "" (id 2) (at 250.952 97.79 90)
-      (effects (font (size 1.27 1.27)) hide)
-    )
+    (property "Footprint" "Resistor_SMD:R_0603_1608Metric_Pad0.98x0.95mm_HandSolder" (id 2) (at 250.952 97.79 90)
+      (effects (font (size 1.27 1.27)) hide)
+    )

Commit message: aaaaaaaaaaaaaaaaaaaaaaaaaaaaaaaa
Other:
- note added: "selected for worst case"
Changed lines of the file:
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@@
+    (effects (font (size 1.27 1.27)) (justify left bottom))
+  )
+  (text "selected for worst case\n" (at 184.15 49.53 0)
     (effects (font (size 1.27 1.27)) (justify left bottom))
   )
