File: sch/carrier/battery.kicad_sch (KiCad schematic)
At the start: 9 parts, among them U5 BQ27441DRZR-G1B

Commit message: aaaaaaaaaaaaaaaaaaaaaaaaaaaaaaaa
Parts:
- C21, C22: footprint (none) -> Capacitor_SMD:C_0603_1608Metric_Pad1.08x0.95mm_HandSolder
Changed lines of the file:
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@@
   )
   (text "(Current) sense resistors are low value low tolerance resistors \nhttps://blog.ttelectronics.com/current-sense-resistors\n"
-    (at 33.02 92.075 0)
+    (at 36.195 56.515 0)
     (effects (font (size 1.27 1.27)) (justify left bottom))
   )
@@
       (effects (font (size 1.27 1.27)) (justify left))
     )
-    (property "Footprint" "" (id 2) (at 96.8502 80.01 0)
+    (property "Footprint" "Capacitor_SMD:C_0603_1608Metric_Pad1.08x0.95mm_HandSolder" (id 2) (at 96.8502 80.01 0)
       (effects (font (size 1.27 1.27)) hide)
     )
@@
       (effects (font (size 1.27 1.27)) (justify left))
     )
-    (property "Footprint" "" (id 2) (at 171.7802 82.55 0)
-      (effects (font (size 1.27 1.27)) hide)
-    )
+    (property "Footprint" "Capacitor_SMD:C_0603_1608Metric_Pad1.08x0.95mm_HandSolder" (id 2) (at 171.7802 82.55 0)
+      (effects (font (size 1.27 1.27)) hide)
+    )

Commit message: pcb time?
Parts:
- removed R60, R62: 5.1k, Resistor_SMD:R_0402_1005Metric_Pad0.72x0.64mm_HandSolder, symbol Device:R
Changed lines of the file:
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@@
   (junction (at 110.49 85.09) (diameter 0.9144) (color 0 0 0 0))
   (junction (at 110.49 92.71) (diameter 0.9144) (color 0 0 0 0))
-  (junction (at 116.84 77.47) (diameter 0.9144) (color 0 0 0 0))
-  (junction (at 120.65 55.88) (diameter 0.9144) (color 0 0 0 0))
-  (junction (at 125.095 80.01) (diameter 0.9144) (color 0 0 0 0))
   (junction (at 141.605 97.79) (diameter 0.9144) (color 0 0 0 0))
   (junction (at 158.75 74.93) (diameter 0.9144) (color 0 0 0 0))
@@
     (stroke (width 0) (type solid) (color 0 0 0 0))
   )
-  (wire (pts (xy 114.935 77.47) (xy 116.84 77.47))
+  (wire (pts (xy 114.935 77.47) (xy 126.365 77.47))
     (stroke (width 0) (type solid) (color 0 0 0 0))
   )
-  (wire (pts (xy 114.935 80.01) (xy 125.095 80.01))
-    (stroke (width 0) (type solid) (color 0 0 0 0))
-  )
-  (wire (pts (xy 116.84 55.88) (xy 120.65 55.88))
-    (stroke (width 0) (type solid) (color 0 0 0 0))
-  )
-  (wire (pts (xy 116.84 57.15) (xy 116.84 55.88))
-    (stroke (width 0) (type solid) (color 0 0 0 0))
-  )
-  (wire (pts (xy 116.84 64.77) (xy 116.84 77.47))
-    (stroke (width 0) (type solid) (color 0 0 0 0))
-  )
-  (wire (pts (xy 116.84 77.47) (xy 126.365 77.47))
+  (wire (pts (xy 114.935 80.01) (xy 126.365 80.01))
     (stroke (width 0) (type solid) (color 0 0 0 0))
   )
@@
     (stroke (width 0) (type solid) (color 0 0 0 0))
   )
-  (wire (pts (xy 120.65 53.34) (xy 120.65 55.88))
-    (stroke (width 0) (type solid) (color 0 0 0 0))
-  )
-  (wire (pts (xy 120.65 55.88) (xy 125.095 55.88))
-    (stroke (width 0) (type solid) (color 0 0 0 0))
-  )
   (wire (pts (xy 122.555 92.71) (xy 126.365 92.71))
     (stroke (width 0) (type solid) (color 0 0 0 0))
@@
     (stroke (width 0) (type solid) (color 0 0 0 0))
   )
-  (wire (pts (xy 125.095 55.88) (xy 125.095 57.15))
-    (stroke (width 0) (type solid) (color 0 0 0 0))
-  )
-  (wire (pts (xy 125.095 64.77) (xy 125.095 80.01))
-    (stroke (width 0) (type solid) (color 0 0 0 0))
-  )
-  (wire (pts (xy 125.095 80.01) (xy 126.365 80.01))
-    (stroke (width 0) (type solid) (color 0 0 0 0))
-  )
   (wire (pts (xy 126.365 87.63) (xy 118.745 87.63))
-    (stroke (width 0) (type solid) (color 0 0 0 0))
-  )
-  (wire (pts (xy 127 53.34) (xy 120.65 53.34))
     (stroke (width 0) (type solid) (color 0 0 0 0))
   )
@@
   (hierarchical_label "FUEL_SCL" (shape input) (at 114.935 80.01 180)
     (effects (font (size 1.27 1.27)) (justify right))
-  )
-  (hierarchical_label "+3.3v" (shape input) (at 127 53.34 0)
-    (effects (font (size 1.27 1.27)) (justify left))
   )
   (symbol (lib_id "Connector:TestPoint") (at 92.075 72.39 0) (unit 1)
@@
     (pin "2")
   )
-  (symbol (lib_id "Device:R") (at 116.84 60.96 0) (unit 1)
-    (in_bom yes) (on_board yes) (fields_autoplaced)
-    (property "Reference" "R60" (id 0) (at 119.38 59.6899 0)
-      (effects (font (size 1.27 1.27)) (justify left))
-    )
-    (property "Value" "5.1k" (id 1) (at 119.38 62.2299 0)
-      (effects (font (size 1.27 1.27)) (justify left))
-    )
-    (property "Footprint" "Resistor_SMD:R_0402_1005Metric_Pad0.72x0.64mm_HandSolder" (id 2) (at 115.062 60.96 90)
-      (effects (font (size 1.27 1.27)) hide)
-    )
-    (property "Datasheet" "~" (id 3) (at 116.84 60.96 0)
-      (effects (font (size 1.27 1.27)) hide)
-    )
-    (pin "1")
-    (pin "2")
-  )
   (symbol (lib_id "Device:R") (at 122.555 100.33 180) (unit 1)
     (in_bom yes) (on_board yes)
@@
       (effects (font (size 1.27 1.27)) hide)
     )
-    (pin "1")
-    (pin "2")
-  )
-  (symbol (lib_id "Device:R") (at 125.095 60.96 0) (unit 1)
-    (in_bom yes) (on_board yes) (fields_autoplaced)
-    (property "Reference" "R62" (id 0) (at 127.635 59.6899 0)
-      (effects (font (size 1.27 1.27)) (justify left))
-    )
-    (property "Value" "5.1k" (id 1) (at 127.635 62.2299 0)
-      (effects (font (size 1.27 1.27)) (justify left))
-    )
-    (property "Footprint" "Resistor_SMD:R_0402_1005Metric_Pad0.72x0.64mm_HandSolder" (id 2) (at 123.317 60.96 90)
-      (effects (font (size 1.27 1.27)) hide)
-    )
-    (property "Datasheet" "~" (id 3) (at 125.095 60.96 0)
-      (effects (font (size 1.27 1.27)) hide)
-    )
