File: sch/carrier/display_board.kicad_sch (KiCad schematic)
At the start: 3 parts, among them J3 52271-0879, U2 ER-CON40HT-1

Commit message: put some stuff on the pcb - it is going to kill me trying to get all on
Parts:
- added R19: 33, Resistor_SMD:R_0805_2012Metric_Pad1.20x1.40mm_HandSolder, symbol Device:R
Connections:
- net +3.3v: now also R19.1; no longer U2.33 (LEDA)
- new net: R19.2, U2.33 (LEDA)
Changed lines of the file:
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@@
+    (stroke (width 0) (type solid) (color 0 0 0 0))
+  )
+  (wire (pts (xy 124.46 96.52) (xy 130.81 96.52))
     (stroke (width 0) (type solid) (color 0 0 0 0))
   )
@@
     (effects (font (size 1.27 1.27)) (justify right bottom))
   )
+  (label "+3.3v" (at 124.46 96.52 0)
+    (effects (font (size 1.27 1.27)) (justify left bottom))
+  )
   (label "SPI0_CE0_N" (at 131.445 49.53 0)
     (effects (font (size 1.27 1.27)) (justify left bottom))
@@
   )
   (label "+3.3v" (at 137.795 43.815 0)
-    (effects (font (size 1.27 1.27)) (justify left bottom))
-  )
-  (label "+3.3v" (at 138.43 96.52 0)
     (effects (font (size 1.27 1.27)) (justify left bottom))
   )
@@
     (pin "1")
   )
+  (symbol (lib_id "Device:R") (at 134.62 96.52 90) (unit 1)
+    (in_bom yes) (on_board yes)
+    (property "Reference" "R19" (id 0) (at 134.62 94.615 90))
+    (property "Value" "33" (id 1) (at 134.62 96.52 90))
+    (property "Footprint" "Resistor_SMD:R_0805_2012Metric_Pad1.20x1.40mm_HandSolder" (id 2) (at 134.62 98.298 90)
+      (effects (font (size 1.27 1.27)) hide)
+    )
+    (property "Datasheet" "~" (id 3) (at 134.62 96.52 0)
+      (effects (font (size 1.27 1.27)) hide)
+    )
+    (pin "1")
+    (pin "2")
+  )
   (symbol (lib_id "MOLEXZIF:52271-0879") (at 106.68 70.485 90) (unit 1)

Commit message: holy shit i hate chargers
Connections:
- net +3.3v: now also J3.2
- net GND: now also J3.7
- net SPI0_MOSI: now also J3.3; no longer J3.2
- net SPI_MISO: now also J3.4; no longer J3.3
Changed lines of the file:
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@@
   (junction (at 104.14 47.625) (diameter 0.9144) (color 0 0 0 0))
   (junction (at 104.14 52.705) (diameter 0.9144) (color 0 0 0 0))
+  (junction (at 104.14 70.485) (diameter 0.9144) (color 0 0 0 0))
   (junction (at 143.51 43.815) (diameter 0.9144) (color 0 0 0 0))
   (junction (at 144.145 109.855) (diameter 0.9144) (color 0 0 0 0))
@@
     (stroke (width 0) (type solid) (color 0 0 0 0))
   )
+  (wire (pts (xy 104.14 52.705) (xy 104.14 55.245))
+    (stroke (width 0) (type solid) (color 0 0 0 0))
+  )
   (wire (pts (xy 104.14 57.785) (xy 115.57 57.785))
     (stroke (width 0) (type solid) (color 0 0 0 0))
@@
     (stroke (width 0) (type solid) (color 0 0 0 0))
   )
+  (wire (pts (xy 104.14 62.865) (xy 115.57 62.865))
+    (stroke (width 0) (type solid) (color 0 0 0 0))
+  )
   (wire (pts (xy 104.14 65.405) (xy 115.57 65.405))
     (stroke (width 0) (type solid) (color 0 0 0 0))
   )
-  (wire (pts (xy 104.14 67.945) (xy 115.57 67.945))
+  (wire (pts (xy 104.14 67.945) (xy 104.14 70.485))
     (stroke (width 0) (type solid) (color 0 0 0 0))
   )
@@
     (effects (font (size 1.27 1.27)) (justify right bottom))
   )
-  (label "SPI_MISO" (at 115.57 65.405 180)
+  (label "SPI_MISO" (at 115.57 62.865 180)
     (effects (font (size 1.27 1.27)) (justify right bottom))
   )
-  (label "SPI0_MOSI" (at 115.57 67.945 180)
+  (label "SPI0_MOSI" (at 115.57 65.405 180)
     (effects (font (size 1.27 1.27)) (justify right bottom))
   )

Commit message: push
Other:
- note added: "connector to our board (replicate on another point, but make sure this is on its own snap board)"
- note removed: "connector to our board"
Changed lines of the file:
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@@
   (title_block
     (title "Display connector board (not part of mainboard)")
+    (rev "indev")
+    (comment 1 "https://github.com/cinnamondev/gamepithing")
   )
   (junction (at 104.14 45.085) (diameter 0.9144) (color 0 0 0 0))
@@
     (stroke (width 0) (type solid) (color 0 0 0 0))
   )
-  (text "connector to our board\n" (at 95.885 57.15 180)
+  (text "connector to our board \n(replicate on another point, \nbut make sure this is on its \nown snap board)\n"
+    (at 95.885 57.15 0)
     (effects (font (size 1.27 1.27)) (justify right bottom))
   )
@@
     (effects (font (size 1.27 1.27)) (justify right bottom))
   )
-  (text "This is the display connector\n" (at 197.485 48.26 180)
+  (text "This is the display connector\n" (at 198.755 52.705 180)
     (effects (font (size 1.27 1.27)) (justify right bottom))
   )

Commit message: oh yeah
Parts:
- removed J3: 52271-0879, MOLEXZIF:Molex-52271-0879-Manufacturer_Recommended, symbol MOLEXZIF:52271-0879
- removed TP1: GND, TestPoint:TestPoint_Pad_2.0x2.0mm, symbol Connector:TestPoint
- added J?: 52271-0879, MOLEXZIF:Molex-52271-0879-Manufacturer_Recommended, symbol MOLEXZIF:52271-0879
- added TP?: GND, TestPoint:TestPoint_Pad_2.0x2.0mm, symbol Connector:TestPoint
- added TP?: +3.3V, symbol Connector:TestPoint
- added TP?: CEO_N, symbol Connector:TestPoint
- added TP?: MOSI, symbol Connector:TestPoint
- added TP?: SCLK, symbol Connector:TestPoint
- added TP?: MISO, symbol Connector:TestPoint
Connections:
- net +3.3v: now also J?.1, J?.2, TP?.1
- net GND: now also J?.7, J?.8, J?.MP1, J?.MP2, TP?.1
- net SPI0_CE0_N: now also J?.6, TP?.1
- net SPI0_MOSI: now also J?.3, TP?.1
- net SPI0_SCLK: now also J?.5, TP?.1
- net SPI_MISO: now also J?.4, TP?.1

Commit message: ersfdxcv
Parts:
- TP20: renamed from TP?; footprint TestPoint:TestPoint_Pad_2.0x2.0mm -> TestPoint:TestPoint_Pad_1.0x1.0mm
- TP21, TP22, TP23, TP24, TP25: renamed from TP?; footprint (none) -> TestPoint:TestPoint_Pad_1.0x1.0mm
- gave numbers to parts that had none: 1
Changed lines of the file:
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@@
   (symbol (lib_id "Connector:TestPoint") (at 90.805 46.355 270) (unit 1)
     (in_bom yes) (on_board yes)
-    (property "Reference" "TP?" (id 0) (at 95.885 45.0849 90)
+    (property "Reference" "TP20" (id 0) (at 95.885 45.0849 90)
       (effects (font (size 1.27 1.27)) (justify left))
     )
@@
       (effects (font (size 1.27 1.27)) (justify left))
     )
-    (property "Footprint" "TestPoint:TestPoint_Pad_2.0x2.0mm" (id 2) (at 90.805 51.435 0)
+    (property "Footprint" "TestPoint:TestPoint_Pad_1.0x1.0mm" (id 2) (at 90.805 51.435 0)
       (effects (font (size 1.27 1.27)) hide)
     )
@@
   (symbol (lib_id "Connector:TestPoint") (at 90.805 51.435 270) (unit 1)
     (in_bom yes) (on_board yes) (fields_autoplaced)
-    (property "Reference" "TP?" (id 0) (at 95.885 50.1649 90)
+    (property "Reference" "TP21" (id 0) (at 95.885 50.1649 90)
       (effects (font (size 1.27 1.27)) (justify left))
     )
@@
       (effects (font (size 1.27 1.27)) (justify left))
     )
-    (property "Footprint" "" (id 2) (at 90.805 56.515 0)
+    (property "Footprint" "TestPoint:TestPoint_Pad_1.0x1.0mm" (id 2) (at 90.805 56.515 0)
       (effects (font (size 1.27 1.27)) hide)
     )
@@
   (symbol (lib_id "Connector:TestPoint") (at 90.805 55.88 270) (unit 1)
     (in_bom yes) (on_board yes) (fields_autoplaced)
-    (property "Reference" "TP?" (id 0) (at 95.885 54.6099 90)
+    (property "Reference" "TP22" (id 0) (at 95.885 54.6099 90)
       (effects (font (size 1.27 1.27)) (justify left))
     )
@@
       (effects (font (size 1.27 1.27)) (justify left))
     )
-    (property "Footprint" "" (id 2) (at 90.805 60.96 0)
+    (property "Footprint" "TestPoint:TestPoint_Pad_1.0x1.0mm" (id 2) (at 90.805 60.96 0)
       (effects (font (size 1.27 1.27)) hide)
     )
@@
   (symbol (lib_id "Connector:TestPoint") (at 90.805 60.96 270) (unit 1)
     (in_bom yes) (on_board yes) (fields_autoplaced)
-    (property "Reference" "TP?" (id 0) (at 95.885 59.6899 90)
+    (property "Reference" "TP23" (id 0) (at 95.885 59.6899 90)
       (effects (font (size 1.27 1.27)) (justify left))
     )
@@
       (effects (font (size 1.27 1.27)) (justify left))
     )
-    (property "Footprint" "" (id 2) (at 90.805 66.04 0)
+    (property "Footprint" "TestPoint:TestPoint_Pad_1.0x1.0mm" (id 2) (at 90.805 66.04 0)
       (effects (font (size 1.27 1.27)) hide)
     )
@@
   (symbol (lib_id "Connector:TestPoint") (at 90.805 66.04 270) (unit 1)
     (in_bom yes) (on_board yes) (fields_autoplaced)
-    (property "Reference" "TP?" (id 0) (at 95.885 64.7699 90)
+    (property "Reference" "TP24" (id 0) (at 95.885 64.7699 90)
       (effects (font (size 1.27 1.27)) (justify left))
     )
@@
       (effects (font (size 1.27 1.27)) (justify left))
     )
-    (property "Footprint" "" (id 2) (at 90.805 71.12 0)
+    (property "Footprint" "TestPoint:TestPoint_Pad_1.0x1.0mm" (id 2) (at 90.805 71.12 0)
       (effects (font (size 1.27 1.27)) hide)
     )
@@
   (symbol (lib_id "Connector:TestPoint") (at 90.805 71.12 270) (unit 1)
     (in_bom yes) (on_board yes) (fields_autoplaced)
-    (property "Reference" "TP?" (id 0) (at 95.885 69.8499 90)
+    (property "Reference" "TP25" (id 0) (at 95.885 69.8499 90)
       (effects (font (size 1.27 1.27)) (justify left))
     )
@@
       (effects (font (size 1.27 1.27)) (justify left))
     )
-    (property "Footprint" "" (id 2) (at 90.805 76.2 0)
+    (property "Footprint" "TestPoint:TestPoint_Pad_1.0x1.0mm" (id 2) (at 90.805 76.2 0)
       (effects (font (size 1.27 1.27)) hide)
     )
@@
   (symbol (lib_id "power:GND") (at 64.77 48.26 90) (unit 1)
     (in_bom yes) (on_board yes)
-    (property "Reference" "#PWR?" (id 0) (at 71.12 48.26 0)
+    (property "Reference" "#PWR047" (id 0) (at 71.12 48.26 0)
       (effects (font (size 1.27 1.27)) hide)
     )
@@
   (symbol (lib_id "MOLEXZIF:52271-0879") (at 67.31 66.04 90) (unit 1)
     (in_bom yes) (on_board yes) (fields_autoplaced)
-    (property "Reference" "J?" (id 0) (at 61.1505 32.385 90))
+    (property "Reference" "J6" (id 0) (at 61.1505 32.385 90))
     (property "Value" "52271-0879" (id 1) (at 61.1505 34.925 90))
     (property "Footprint" "MOLEXZIF:Molex-52271-0879-Manufacturer_Recommended" (id 2) (at 49.53 66.04 0)

Commit message: enough for now
Connections:
- net SPI0_CE0_N: now also J6.3; no longer J6.6
- net SPI0_MOSI: now also J6.6; no longer J6.3
- net SPI0_SCLK: now also J6.4; no longer J6.5
- net SPI_MISO: now also J6.5; no longer J6.4
- net GND renamed GND1
Other:
- moved on the sheet: TP21, TP22, TP23, TP24
Changed lines of the file:
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@@
     (rev "indev")
   )
+  (junction (at 64.77 41.91) (diameter 0.9144) (color 0 0 0 0))
   (junction (at 64.77 43.18) (diameter 0.9144) (color 0 0 0 0))
   (junction (at 64.77 46.355) (diameter 0.9144) (color 0 0 0 0))
@@
   (no_connect (at 149.225 92.71))
   (no_connect (at 149.225 94.615))
-  (wire (pts (xy 64.77 40.64) (xy 64.77 43.18))
+  (wire (pts (xy 64.77 40.64) (xy 64.77 41.91))
+    (stroke (width 0) (type solid) (color 0 0 0 0))
+  )
+  (wire (pts (xy 64.77 41.91) (xy 64.77 43.18))
     (stroke (width 0) (type solid) (color 0 0 0 0))
   )
@@
     (effects (font (size 1.27 1.27)) (justify right bottom))
   )
-  (label "SPI0_CE0_N" (at 77.47 53.34 180)
-    (effects (font (size 1.27 1.27)) (justify right bottom))
-  )
-  (label "SPI0_SCLK" (at 77.47 55.88 180)
-    (effects (font (size 1.27 1.27)) (justify right bottom))
-  )
-  (label "SPI_MISO" (at 77.47 58.42 180)
-    (effects (font (size 1.27 1.27)) (justify right bottom))
-  )
-  (label "SPI0_MOSI" (at 77.47 60.96 180)
+  (label "SPI0_CE0_N" (at 76.835 60.96 180)
+    (effects (font (size 1.27 1.27)) (justify right bottom))
+  )
+  (label "SPI0_MOSI" (at 77.47 53.34 180)
+    (effects (font (size 1.27 1.27)) (justify right bottom))
+  )
+  (label "SPI_MISO" (at 77.47 55.88 180)
+    (effects (font (size 1.27 1.27)) (justify right bottom))
+  )
+  (label "SPI0_SCLK" (at 77.47 58.42 180)
     (effects (font (size 1.27 1.27)) (justify right bottom))
   )
@@
   (symbol (lib_id "Connector:TestPoint") (at 90.805 51.435 270) (unit 1)
     (in_bom yes) (on_board yes) (fields_autoplaced)
-    (property "Reference" "TP21" (id 0) (at 95.885 50.1649 90)
-      (effects (font (size 1.27 1.27)) (justify left))
-    )
-    (property "Value" "CEO_N" (id 1) (at 95.885 52.7049 90)
+    (property "Reference" "TP24" (id 0) (at 95.885 50.1649 90)
+      (effects (font (size 1.27 1.27)) (justify left))
+    )
+    (property "Value" "MOSI" (id 1) (at 95.885 52.7049 90)
       (effects (font (size 1.27 1.27)) (justify left))
     )
@@
   (symbol (lib_id "Connector:TestPoint") (at 90.805 55.88 270) (unit 1)
     (in_bom yes) (on_board yes) (fields_autoplaced)
-    (property "Reference" "TP22" (id 0) (at 95.885 54.6099 90)
-      (effects (font (size 1.27 1.27)) (justify left))
-    )
-    (property "Value" "SCLK" (id 1) (at 95.885 57.1499 90)
+    (property "Reference" "TP23" (id 0) (at 95.885 54.6099 90)
+      (effects (font (size 1.27 1.27)) (justify left))
+    )
+    (property "Value" "MISO" (id 1) (at 95.885 57.1499 90)
       (effects (font (size 1.27 1.27)) (justify left))
     )
@@
   (symbol (lib_id "Connector:TestPoint") (at 90.805 60.96 270) (unit 1)
     (in_bom yes) (on_board yes) (fields_autoplaced)
-    (property "Reference" "TP23" (id 0) (at 95.885 59.6899 90)
-      (effects (font (size 1.27 1.27)) (justify left))
-    )
-    (property "Value" "MISO" (id 1) (at 95.885 62.2299 90)
+    (property "Reference" "TP22" (id 0) (at 95.885 59.6899 90)
+      (effects (font (size 1.27 1.27)) (justify left))
+    )
+    (property "Value" "SCLK" (id 1) (at 95.885 62.2299 90)
       (effects (font (size 1.27 1.27)) (justify left))
     )
@@
   (symbol (lib_id "Connector:TestPoint") (at 90.805 66.04 270) (unit 1)
     (in_bom yes) (on_board yes) (fields_autoplaced)
-    (property "Reference" "TP24" (id 0) (at 95.885 64.7699 90)
-      (effects (font (size 1.27 1.27)) (justify left))
-    )
-    (property "Value" "MOSI" (id 1) (at 95.885 67.3099 90)
+    (property "Reference" "TP21" (id 0) (at 95.885 64.7699 90)
+      (effects (font (size 1.27 1.27)) (justify left))
+    )
+    (property "Value" "CEO_N" (id 1) (at 95.885 67.3099 90)
       (effects (font (size 1.27 1.27)) (justify left))
     )
@@
     (pin "1")
   )
-  (symbol (lib_id "power:GND") (at 64.77 48.26 90) (unit 1)
-    (in_bom yes) (on_board yes)
-    (property "Reference" "#PWR047" (id 0) (at 71.12 48.26 0)
-      (effects (font (size 1.27 1.27)) hide)
-    )
-    (property "Value" "GND" (id 1) (at 67.945 48.2599 90)
+  (symbol (lib_id "power:GND1") (at 64.77 41.91 90) (unit 1)
+    (in_bom yes) (on_board yes) (fields_autoplaced)
+    (property "Reference" "#PWR?" (id 0) (at 71.12 41.91 0)
+      (effects (font (size 1.27 1.27)) hide)
+    )
+    (property "Value" "GND1" (id 1) (at 68.58 41.9099 90)
       (effects (font (size 1.27 1.27)) (justify right))
     )
-    (property "Footprint" "" (id 2) (at 64.77 48.26 0)
-      (effects (font (size 1.27 1.27)) hide)
-    )
-    (property "Datasheet" "" (id 3) (at 64.77 48.26 0)
-      (effects (font (size 1.27 1.27)) hide)
-    )
-    (pin "1")
-  )
-  (symbol (lib_id "power:GND") (at 145.415 111.125 0) (unit 1)
-    (in_bom yes) (on_board yes) (fields_autoplaced)
-    (property "Reference" "#PWR017" (id 0) (at 145.415 117.475 0)
-      (effects (font (size 1.27 1.27)) hide)
-    )
-    (property "Value" "GND" (id 1) (at 145.415 115.57 0))
+    (property "Footprint" "" (id 2) (at 64.77 41.91 0)
+      (effects (font (size 1.27 1.27)) hide)
+    )
+    (property "Datasheet" "" (id 3) (at 64.77 41.91 0)
+      (effects (font (size 1.27 1.27)) hide)
+    )
+    (pin "1")
+  )
+  (symbol (lib_id "power:GND1") (at 145.415 111.125 0) (unit 1)
+    (in_bom yes) (on_board yes) (fields_autoplaced)
+    (property "Reference" "#PWR?" (id 0) (at 145.415 117.475 0)
+      (effects (font (size 1.27 1.27)) hide)
+    )
+    (property "Value" "GND1" (id 1) (at 148.59 112.2044 0)
+      (effects (font (size 1.27 1.27)) (justify left))
+    )
     (property "Footprint" "" (id 2) (at 145.415 111.125 0)
       (effects (font (size 1.27 1.27)) hide)
