File: sch/carrier/CM4.kicad_sch (KiCad schematic)
At the start: 26 parts, among them J2 52271-0879, J3 Micro_SD_Card_Det, Q1 Q_NPN_BCE, U4 AP22814AW5

Commit message: asd
Parts:
- R25: footprint (none) -> Resistor_SMD:R_0603_1608Metric_Pad0.98x0.95mm_HandSolder
Changed lines of the file:
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@@
     (property "Reference" "R25" (id 0) (at 277.495 92.075 90))
     (property "Value" "0" (id 1) (at 277.495 90.17 90))
-    (property "Footprint" "" (id 2) (at 277.495 88.392 90)
+    (property "Footprint" "Resistor_SMD:R_0603_1608Metric_Pad0.98x0.95mm_HandSolder" (id 2) (at 277.495 88.392 90)
       (effects (font (size 1.27 1.27)) hide)
     )

Commit message: randomtexttofillthecommittext
Parts:
- removed C7: 33uF, symbol Device:C
- removed C9: 10uF, symbol Device:C
- removed LS1: Speaker, symbol Device:Speaker
- removed Q1: Q_NPN_BCE, symbol Device:Q_NPN_BCE
- removed R14: 270, Resistor_SMD:R_0603_1608Metric_Pad0.98x0.95mm_HandSolder, symbol Device:R
- removed R18: 140, Resistor_SMD:R_0603_1608Metric_Pad0.98x0.95mm_HandSolder, symbol Device:R
- removed R23: 15k, Resistor_SMD:R_0603_1608Metric_Pad0.98x0.95mm_HandSolder, symbol Device:R
- removed R24: 8, Resistor_SMD:R_0603_1608Metric_Pad0.98x0.95mm_HandSolder, symbol Device:R
- added C? (x2): 10u, symbol Device:C
- added C? (x2): 33n, symbol Device:C
- added D? (x2): BAV99, Package_TO_SOT_SMD:SOT-23, symbol Diode:BAV99
- added J?: AudioJack3_Ground_Switch, symbol Connector:AudioJack3_Ground_Switch
- added R? (x2): 150, symbol Device:R
- added R?: 0, symbol Device:R
- added R? (x2): 270, symbol Device:R
Connections:
- net +3.3v: now also D?.2 (A), D?.2 (A)
- net BTN_A: now also Module0.41 (GPIO25); no longer Module0.49 (GPIO18)
- net BTN_START: now also Module0.45 (GPIO24); no longer Module0.26 (GPIO19)
- net GND: now also C?.1, C?.1, D?.1 (K), D?.1 (K), J?.T, R?.2, R?.2, R?.2
- new net: C?.2, D?.3 (K), J?.S
- new net: C?.1, C?.2, R?.1, R?.2 (x2)
- new net: C?.2, D?.3 (K), J?.R
- new net: J?.G, R?.1
- new net AUX0: Module0.49 (GPIO18), R?.1
- new net AUX1: Module0.26 (GPIO19), R?.1
Other:
- note added: "Audio - follows https://learn.adafruit.com/introducing-the-raspberry-pi-zero/audio-outputs (pi schematic)"
- note added: "sounds good enough"
- note removed: "Audio - follows https://learn.adafruit.com/introducing-the-raspberry-pi-zero/audio-outputs Adaptations made to drive a small speaker in place of the original"
- note removed: "divider to get 3.3 --> 1.1v"
- note removed: "low pass filter"
- note removed: "npm transistor to drive a speaker"
- note removed: "our signal output is apparently a PWM (digital thingymajigy) will 'trick the speaker'"

Commit message: aaaaaaaaaaaaaaaaaaaaaaaaaaaaaaaa
Parts:
- added TP27: AUXR, TestPoint:TestPoint_Pad_1.0x1.0mm, symbol Connector:TestPoint
- added TP28: AUXL, TestPoint:TestPoint_Pad_1.0x1.0mm, symbol Connector:TestPoint
- C23, C24: renamed from C?; footprint (none) -> Capacitor_SMD:C_0603_1608Metric_Pad1.08x0.95mm_HandSolder
- J7: renamed from J?; footprint (none) -> audio:audio
- R14, R18, R23, R24, R64: renamed from R?; footprint (none) -> Resistor_SMD:R_0603_1608Metric_Pad0.98x0.95mm_HandSolder
- gave numbers to parts that had none: 4
Connections:
- net at C9.2, D4.3 (K), J7.S: now also TP28.1
- net at C24.2, D5.3 (K), J7.R: now also TP27.1

Commit message: pcb time?
Parts:
- removed J3: Micro_SD_Card_Det, sdcard:HRS_DM3CS-SF, symbol Connector:Micro_SD_Card_Det
- removed J7: AudioJack3_Ground_Switch, audio:audio, symbol Connector:AudioJack3_Ground_Switch
- removed R20, R21: nf, Resistor_SMD:R_0402_1005Metric, symbol Device:R
- removed R64: 0, Resistor_SMD:R_0603_1608Metric_Pad0.98x0.95mm_HandSolder, symbol Device:R
- added J3: Micro_SD_Card, sdcard:HRS_DM3CS-SF, symbol Connector:Micro_SD_Card
- added J7: AudioJack3_Switch, audio:audio, symbol Connector:AudioJack3_Switch
- C7, C8, C9: footprint (none) -> Capacitor_SMD:C_0603_1608Metric_Pad1.08x0.95mm_HandSolder
Connections:
- net GND: now also J3.6 (VSS), J7.T
- net SD_CLK: now also J3.5 (CLK)
- net SD_CMD: now also J3.3 (CMD)
- net SD_DAT0: now also J3.7 (DAT0)
- net SD_DAT1: now also J3.8 (DAT1)
- net SD_DAT2: now also J3.1 (DAT2)
- net SD_DAT3: now also J3.2 (DAT3/CD)
- net SD_PWR: now also J3.4 (VDD)
- net at C9.2, D4.3 (K), TP28.1: now also J7.S
- net at C24.2, D5.3 (K), TP27.1: now also J7.R
- net at R25.2: now also J3.9 (SHIELD)
Other:
- note added: "apparently these diodes serve as clamping diodes https://electronics.stackexchange.com/questions/137643/how-does-a-diode-clamping-circuit-protect-against-overvoltage-and-esd"
- note removed: "sounds good enough"
Changed lines of the file:
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@@
-    (stroke (width 0) (type solid) (color 0 0 0 0))
-  )
-  (wire (pts (xy 211.455 87.63) (xy 222.885 87.63))
-    (stroke (width 0) (type solid) (color 0 0 0 0))
-  )
-  (wire (pts (xy 211.455 95.25) (xy 222.885 95.25))
     (stroke (width 0) (type solid) (color 0 0 0 0))
   )
@@
     (stroke (width 0) (type solid) (color 0 0 0 0))
   )
-  (wire (pts (xy 230.505 90.17) (xy 230.505 95.25))
-    (stroke (width 0) (type solid) (color 0 0 0 0))
-  )
   (wire (pts (xy 231.775 106.045) (xy 247.65 106.045))
     (stroke (width 0) (type solid) (color 0 0 0 0))
@@
   )
   (text "Audio - follows https://learn.adafruit.com/introducing-the-raspberry-pi-zero/audio-outputs\n(pi schematic)"
-    (at 109.855 170.18 0)
-    (effects (font (size 1.27 1.27)) (justify left bottom))
+    (at 90.17 172.72 0)
+    (effects (font (size 1.27 1.27)) (justify left bottom))
+  )
+  (text "apparently these diodes serve as clamping diodes\nhttps://electronics.stackexchange.com/questions/137643/how-does-a-diode-clamping-circuit-protect-against-overvoltage-and-esd"
+    (at 105.41 163.83 0)
+    (effects (font (size 0.635 0.635)) (justify left bottom))
   )
   (text "To enable SPI you must enable the SPI alt mode." (at 135.89 19.05 180)
@@
     (effects (font (size 1.27 1.27)) (justify left bottom))
   )
-  (text "sounds good enough\n" (at 219.71 148.59 0)
-    (effects (font (size 1.27 1.27)) (justify left bottom))
-  )
   (text "close relative part to whats on the cm4io's sheet\n"
     (at 234.95 125.095 0)
@@
     (effects (font (size 1.27 1.27)) (justify left bottom))
   )
-  (label "+3.3v" (at 211.455 87.63 0)
-    (effects (font (size 1.27 1.27)) (justify left bottom))
-  )
   (label "SD_PWR" (at 212.09 72.39 0)
     (effects (font (size 1.27 1.27)) (justify left bottom))
-  )
-  (label "Reserved" (at 219.71 95.25 180)
-    (effects (font (size 1.27 1.27)) (justify right bottom))
   )
   (label "SD_DAT2" (at 221.615 67.31 0)
@@
     )
     (property "Datasheet" "" (id 3) (at 210.82 80.01 0)
-      (effects (font (size 1.27 1.27)) hide)
-    )
-    (pin "1")
-  )
-  (symbol (lib_id "power:GND") (at 212.725 154.94 0) (unit 1)
-    (in_bom yes) (on_board yes) (fields_autoplaced)
-    (property "Reference" "#PWR054" (id 0) (at 212.725 161.29 0)
-      (effects (font (size 1.27 1.27)) hide)
-    )
-    (property "Value" "GND" (id 1) (at 212.725 159.385 0))
-    (property "Footprint" "" (id 2) (at 212.725 154.94 0)
-      (effects (font (size 1.27 1.27)) hide)
-    )
-    (property "Datasheet" "" (id 3) (at 212.725 154.94 0)
       (effects (font (size 1.27 1.27)) hide)
     )
@@
     )
     (property "Datasheet" "~" (id 3) (at 166.37 128.27 0)
-      (effects (font (size 1.27 1.27)) hide)
-    )
-    (pin "1")
-    (pin "2")
-  )
-  (symbol (lib_id "Device:R") (at 212.725 151.13 0) (unit 1)
-    (in_bom yes) (on_board yes)
-    (property "Reference" "R64" (id 0) (at 213.995 151.1299 0)
-      (effects (font (size 1.27 1.27)) (justify left))
-    )
-    (property "Value" "0" (id 1) (at 212.09 151.1299 0)
-      (effects (font (size 1.27 1.27)) (justify left))
-    )
-    (property "Footprint" "Resistor_SMD:R_0603_1608Metric_Pad0.98x0.95mm_HandSolder" (id 2) (at 210.947 151.13 90)
-      (effects (font (size 1.27 1.27)) hide)
-    )
-    (property "Datasheet" "~" (id 3) (at 212.725 151.13 0)
-      (effects (font (size 1.27 1.27)) hide)
-    )
-    (pin "1")
-    (pin "2")
-  )
-  (symbol (lib_id "Device:R") (at 226.695 87.63 90) (unit 1)
-    (in_bom yes) (on_board yes)
-    (property "Reference" "R20" (id 0) (at 225.425 90.17 90)
-      (effects (font (size 1.27 1.27)) (justify left))
-    )
-    (property "Value" "nf" (id 1) (at 229.235 90.17 90)
-      (effects (font (size 1.27 1.27)) (justify left))
-    )
-    (property "Footprint" "Resistor_SMD:R_0402_1005Metric" (id 2) (at 226.695 89.408 90)
-      (effects (font (size 1.27 1.27)) hide)
-    )
-    (property "Datasheet" "https://fscdn.rohm.com/en/products/databook/datasheet/passive/resistor/chip_resistor/mcr-e.pdf" (id 3) (at 226.695 87.63 0)
-      (effects (font (size 1.27 1.27)) hide)
-    )
-    (property "Field4" "Farnell" (id 4) (at 226.695 87.63 0)
-      (effects (font (size 1.27 1.27)) hide)
-    )
-    (property "Field5" "9239235" (id 5) (at 226.695 87.63 0)
-      (effects (font (size 1.27 1.27)) hide)
-    )
-    (property "Field7" "KOA EUROPE GMBH" (id 6) (at 226.695 87.63 0)
-      (effects (font (size 1.27 1.27)) hide)
-    )
-    (property "Field6" "RK73H1ETTP1001F" (id 7) (at 226.695 87.63 0)
-      (effects (font (size 1.27 1.27)) hide)
-    )
-    (property "Part Description" "Resistor 1K M1005 1% 63mW" (id 8) (at 226.695 87.63 0)
-      (effects (font (size 1.27 1.27)) hide)
-    )
-    (property "Field8" "125049511" (id 9) (at 226.695 87.63 0)
-      (effects (font (size 1.27 1.27)) hide)
-    )
-    (pin "1")
-    (pin "2")
-  )
-  (symbol (lib_id "Device:R") (at 226.695 95.25 90) (unit 1)
-    (in_bom yes) (on_board yes)
-    (property "Reference" "R21" (id 0) (at 225.1456 97.6376 90)
-      (effects (font (size 1.27 1.27)) (justify left))
-    )
-    (property "Value" "nf" (id 1) (at 229.1588 97.5868 90)
-      (effects (font (size 1.27 1.27)) (justify left))
-    )
-    (property "Footprint" "Resistor_SMD:R_0402_1005Metric" (id 2) (at 226.695 97.028 90)
-      (effects (font (size 1.27 1.27)) hide)
-    )
-    (property "Datasheet" "https://fscdn.rohm.com/en/products/databook/datasheet/passive/resistor/chip_resistor/mcr-e.pdf" (id 3) (at 226.695 95.25 0)
-      (effects (font (size 1.27 1.27)) hide)
-    )
-    (property "Field4" "Farnell" (id 4) (at 226.695 95.25 0)
-      (effects (font (size 1.27 1.27)) hide)
-    )
-    (property "Field5" "9239235" (id 5) (at 226.695 95.25 0)
-      (effects (font (size 1.27 1.27)) hide)
-    )
-    (property "Field7" "KOA EUROPE GMBH" (id 6) (at 226.695 95.25 0)
-      (effects (font (size 1.27 1.27)) hide)
-    )
-    (property "Field6" "RK73H1ETTP1001F" (id 7) (at 226.695 95.25 0)
-      (effects (font (size 1.27 1.27)) hide)
-    )
-    (property "Part Description" "Resistor 1K M1005 1% 63mW" (id 8) (at 226.695 95.25 0)
-      (effects (font (size 1.27 1.27)) hide)
-    )
-    (property "Field8" "125049511" (id 9) (at 226.695 95.25 0)
       (effects (font (size 1.27 1.27)) hide)
     )
@@
     (property "Reference" "C7" (id 0) (at 127 139.065 90))
     (property "Value" "33n" (id 1) (at 132.715 139.065 90))
-    (property "Footprint" "" (id 2) (at 133.35 140.0048 0)
+    (property "Footprint" "Capacitor_SMD:C_0603_1608Metric_Pad1.08x0.95mm_HandSolder" (id 2) (at 133.35 140.0048 0)
       (effects (font (size 1.27 1.27)) hide)
     )
@@
     (property "Reference" "C9" (id 0) (at 149.86 131.445 90))
     (property "Value" "10u" (id 1) (at 149.86 133.985 90))
-    (property "Footprint" "" (id 2) (at 153.67 138.0998 0)
+    (property "Footprint" "Capacitor_SMD:C_0603_1608Metric_Pad1.08x0.95mm_HandSolder" (id 2) (at 153.67 138.0998 0)
       (effects (font (size 1.27 1.27)) hide)
     )
@@
       (effects (font (size 1.27 1.27)) (justify left))
     )
-    (property "Footprint" "" (id 2) (at 211.7852 80.01 0)
+    (property "Footprint" "Capacitor_SMD:C_0603_1608Metric_Pad1.08x0.95mm_HandSolder" (id 2) (at 211.7852 80.01 0)
       (effects (font (size 1.27 1.27)) hide)
     )
@@
     (pin "3")
   )
-  (symbol (lib_id "Connector:AudioJack3_Ground_Switch") (at 212.725 134.62 0) (mirror y) (unit 1)
-    (in_bom yes) (on_board yes) (fields_autoplaced)
-    (property "Reference" "J7" (id 0) (at 220.98 136.6519 0)
+  (symbol (lib_id "Connector:AudioJack3_Switch") (at 212.725 134.62 0) (mirror y) (unit 1)
+    (in_bom yes) (on_board yes) (fields_autoplaced)
+    (property "Reference" "J7" (id 0) (at 220.345 134.6199 0)
       (effects (font (size 1.27 1.27)) (justify right))
     )
-    (property "Value" "AudioJack3_Ground_Switch" (id 1) (at 220.98 139.1919 0)
+    (property "Value" "AudioJack3_Switch" (id 1) (at 220.345 137.1599 0)
       (effects (font (size 1.27 1.27)) (justify right))
     )
@@
       (effects (font (size 1.27 1.27)) hide)
     )
-    (pin "G")
     (pin "R")
     (pin "RN")
@@
     (pin "5")
   )
-  (symbol (lib_id "Connector:Micro_SD_Card_Det") (at 253.365 77.47 0) (unit 1)
-    (in_bom yes) (on_board yes) (fields_autoplaced)
-    (property "Reference" "J3" (id 0) (at 252.095 55.245 0))
-    (property "Value" "Micro_SD_Card_Det" (id 1) (at 252.095 57.785 0))
-    (property "Footprint" "sdcard:HRS_DM3CS-SF" (id 2) (at 305.435 59.69 0)
-      (effects (font (size 1.27 1.27)) hide)
-    )
-    (property "Datasheet" "https://www.hirose.com/product/en/download_file/key_name/DM3/category/Catalog/doc_file_id/49662/?file_category_id=4&item_id=195&is_series=1" (id 3) (at 253.365 74.93 0)
-      (effects (font (size 1.27 1.27)) hide)
-    )
-    (pin "1")
-    (pin "10")
-    (pin "11")
+  (symbol (lib_id "Connector:Micro_SD_Card") (at 253.365 74.93 0) (unit 1)
+    (in_bom yes) (on_board yes) (fields_autoplaced)
+    (property "Reference" "J3" (id 0) (at 252.095 55.88 0))
+    (property "Value" "Micro_SD_Card" (id 1) (at 252.095 58.42 0))
+    (property "Footprint" "sdcard:HRS_DM3CS-SF" (id 2) (at 282.575 67.31 0)
+      (effects (font (size 1.27 1.27)) hide)
+    )
+    (property "Datasheet" "http://katalog.we-online.de/em/datasheet/693072010801.pdf" (id 3) (at 253.365 74.93 0)
+      (effects (font (size 1.27 1.27)) hide)
+    )
+    (pin "1")
     (pin "2")
     (pin "3")

Commit message: enough for now
Connections:
- net SCREEN_CE0_N: now also J2.3; no longer J2.6
- net SCREEN_MISO: now also J2.5; no longer J2.4
- net SCREEN_MOSI: now also J2.6; no longer J2.3
- net SCREEN_SCLK: now also J2.4; no longer J2.5
Other:
- moved on the sheet: TP12, TP3, TP4, TP5
Changed lines of the file:
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@@
-    (effects (font (size 1.27 1.27)) (justify left bottom))
-  )
-  (label "SCREEN_CE0_N" (at 246.38 34.925 0)
-    (effects (font (size 1.27 1.27)) (justify left bottom))
-  )
-  (label "SCREEN_SCLK" (at 246.38 37.465 0)
-    (effects (font (size 1.27 1.27)) (justify left bottom))
-  )
-  (label "SCREEN_MISO" (at 246.38 40.005 0)
-    (effects (font (size 1.27 1.27)) (justify left bottom))
-  )
-  (label "SCREEN_MOSI" (at 246.38 42.545 0)
     (effects (font (size 1.27 1.27)) (justify left bottom))
   )
   (label "+3.3v" (at 247.015 106.045 180)
     (effects (font (size 1.27 1.27)) (justify right bottom))
+  )
+  (label "SCREEN_MOSI" (at 248.285 34.925 0)
+    (effects (font (size 1.27 1.27)) (justify left bottom))
+  )
+  (label "SCREEN_MISO" (at 248.285 37.465 0)
+    (effects (font (size 1.27 1.27)) (justify left bottom))
+  )
+  (label "SCREEN_SCLK" (at 248.285 40.005 0)
+    (effects (font (size 1.27 1.27)) (justify left bottom))
+  )
+  (label "SCREEN_CE0_N" (at 248.285 42.545 0)
+    (effects (font (size 1.27 1.27)) (justify left bottom))
   )
   (label "+3.3v" (at 257.81 47.625 180)
@@
   (symbol (lib_id "Connector:TestPoint") (at 272.415 33.02 270) (unit 1)
     (in_bom yes) (on_board yes) (fields_autoplaced)
-    (property "Reference" "TP3" (id 0) (at 277.495 31.7499 90)
+    (property "Reference" "TP12" (id 0) (at 277.495 31.7499 90)
       (effects (font (size 1.27 1.27)) (justify left))
     )
-    (property "Value" "CEO_N" (id 1) (at 277.495 34.2899 90)
+    (property "Value" "MOSI" (id 1) (at 277.495 34.2899 90)
       (effects (font (size 1.27 1.27)) (justify left))
     )
@@
   (symbol (lib_id "Connector:TestPoint") (at 272.415 37.465 270) (unit 1)
     (in_bom yes) (on_board yes) (fields_autoplaced)
-    (property "Reference" "TP4" (id 0) (at 277.495 36.1949 90)
+    (property "Reference" "TP5" (id 0) (at 277.495 36.1949 90)
       (effects (font (size 1.27 1.27)) (justify left))
     )
-    (property "Value" "SCLK" (id 1) (at 277.495 38.7349 90)
+    (property "Value" "MISO" (id 1) (at 277.495 38.7349 90)
       (effects (font (size 1.27 1.27)) (justify left))
     )
@@
   (symbol (lib_id "Connector:TestPoint") (at 272.415 42.545 270) (unit 1)
     (in_bom yes) (on_board yes) (fields_autoplaced)
-    (property "Reference" "TP5" (id 0) (at 277.495 41.2749 90)
+    (property "Reference" "TP4" (id 0) (at 277.495 41.2749 90)
       (effects (font (size 1.27 1.27)) (justify left))
     )
-    (property "Value" "MISO" (id 1) (at 277.495 43.8149 90)
+    (property "Value" "SCLK" (id 1) (at 277.495 43.8149 90)
       (effects (font (size 1.27 1.27)) (justify left))
     )
@@
   (symbol (lib_id "Connector:TestPoint") (at 272.415 47.625 270) (unit 1)
     (in_bom yes) (on_board yes) (fields_autoplaced)
-    (property "Reference" "TP12" (id 0) (at 277.495 46.3549 90)
+    (property "Reference" "TP3" (id 0) (at 277.495 46.3549 90)
       (effects (font (size 1.27 1.27)) (justify left))
     )
-    (property "Value" "MOSI" (id 1) (at 277.495 48.8949 90)
+    (property "Value" "CEO_N" (id 1) (at 277.495 48.8949 90)
       (effects (font (size 1.27 1.27)) (justify left))
     )

Commit message: aa
Parts:
- R13: footprint Capacitor_SMD:C_0402_1005Metric_Pad0.74x0.62mm_HandSolder -> Resistor_SMD:R_0402_1005Metric_Pad0.72x0.64mm_HandSolder
Changed lines of the file:
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@@
       (effects (font (size 1.27 1.27)) (justify right))
     )
-    (property "Footprint" "Capacitor_SMD:C_0402_1005Metric_Pad0.74x0.62mm_HandSolder" (id 2) (at 114.173 48.26 90)
+    (property "Footprint" "Resistor_SMD:R_0402_1005Metric_Pad0.72x0.64mm_HandSolder" (id 2) (at 114.173 48.26 90)
       (effects (font (size 1.27 1.27)) hide)
     )
