File: carrier/carrier.kicad_pcb (KiCad board)
At the start: 4 copper layers, 103.3 x 77.2 mm, 147 parts, among them J1 USB_C_Receptacle_USB2.0, J2 52271-0879, J3 Micro_SD_Card, J4 HDMI_D_1.4, J5 USB_C_Receptacle_USB2.0, J6 52271-0879, J7 AudioJack3_Switch, SW1 SKRRACE010, SW10 SKRBAAE010, SW11 SW_Push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

Commit message: pcb!?
Parts:
- R47: footprint Resistor_SMD:R_1210_3225Metric_Pad1.30x2.65mm_HandSolder -> Resistor_SMD:R_0402_1005Metric_Pad0.72x0.64mm_HandSolder
- moved C22 433.5 mm to (556.5, 55.0), turned to -90 degrees
- moved C21 430.9 mm to (555.5, 60.2), turned to -90 degrees
- moved R61 423.4 mm to (558.2, 60.2), turned to 90 degrees
- moved R63 414.8 mm to (545.0, 59.0), turned to 180 degrees
- moved U5 414.8 mm to (545.0, 54.0), turned to 180 degrees
- moved TP26 405.0 mm to (526.5, 75.0)
- moved R59 401.3 mm to (548.2, 70.2), turned to 180 degrees
- moved NT1 316.3 mm to (508.2, 79.5)
- moved C12 274.1 mm to (260.8, -32.3)
- moved C14 274.1 mm to (280.5, -32.1)
- moved C15 274.1 mm to (464.2, 15.5)
- moved C16 274.1 mm to (474.3, 24.2)
- moved C17 274.1 mm to (467.1, 34.6)
- moved C18 274.1 mm to (428.8, 7.00)
- moved C19 274.1 mm to (437.2, 7.00)
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Routing:
- net /Display board (SNAP OFF BOARD)/SPI0_CE0_N: track 0.00 -> 16.2 mm
- net /Display board (SNAP OFF BOARD)/SPI0_MOSI: track 0.00 -> 13.8 mm
- net /Display board (SNAP OFF BOARD)/SPI0_SCLK: track 0.00 -> 13.3 mm
- net /Display board (SNAP OFF BOARD)/SPI_MISO: track 0.00 -> 13.0 mm
- net Net-(R19-Pad2): track 0.00 -> 8.59 mm
- net GND1: track 0.00 -> 2.34 mm, vias 0 -> 3
- added copper zone on F.Cu, net /Display board (SNAP OFF BOARD)/+3.3v
- added copper zone on In2.Cu, net GND
- added copper zone on B.Cu, net GND1
- added copper zone on F.Cu, net GND1
Other:
- outline, holes or cut-outs redrawn

Commit message: pcb
Parts:
- removed R58: 0, Resistor_SMD:R_1210_3225Metric_Pad1.30x2.65mm_HandSolder
- removed TP27: AUXR, TestPoint:TestPoint_Pad_1.0x1.0mm
- removed TP28: AUXL, TestPoint:TestPoint_Pad_1.0x1.0mm
- moved D4 565.1 mm to (34.8, 45.5)
- moved C9 562.6 mm to (33.8, 41.0)
- moved C7 560.8 mm to (30.0, 44.0)
- moved R14 560.8 mm to (30.0, 41.0)
- moved J7 550.9 mm to (38.6, 25.1)
- moved R18 550.4 mm to (30.0, 47.0), turned to 180 degrees
- moved R24 546.9 mm to (47.1, 47.0), turned to 0 degrees
- moved D5 544.4 mm to (42.4, 45.5)
- moved C24 539.9 mm to (43.4, 41.0), turned to 180 degrees
- moved C23 530.5 mm to (47.1, 44.0), turned to 180 degrees
- moved R23 530.5 mm to (47.1, 41.0), turned to 180 degrees
- moved TP10 34.0 mm to (160.1, 117.8), turned to 180 degrees
- moved TP11 31.7 mm to (160.1, 115.2), turned to 90 degrees
- moved U1 23.6 mm to (154.4, 116.5), turned to 0 degrees
- moved TP7 16.8 mm to (154.4, 125.9)
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Connections:
- J1 pad S1: Net-(J1-PadS1) -> unconnected-(J1-PadS1)
- J5 pad S1: Net-(J5-PadS1) -> unconnected-(J5-PadS1)
Routing:
- net /Buttons/__DP_L: track 0.00 -> 96.0 mm
- net /Buttons/__DP_U: track 0.00 -> 49.7 mm
- net /Buttons/__DP_R: track 0.00 -> 43.6 mm
- net /Buttons/__DP_D: track 0.00 -> 35.8 mm
- net /Buttons/__B_A: track 0.00 -> 34.4 mm
- net GND: track 0.00 -> 31.3 mm, vias 0 -> 6
- net /Buttons/__B_B: track 0.00 -> 23.3 mm
- net /Buttons/DPAD_RIGHT: track 0.00 -> 17.0 mm, vias 0 -> 1
- net /Buttons/DPAD_DOWN: track 0.00 -> 13.6 mm, vias 0 -> 1
- net Net-(J5-PadA5): track 0.00 -> 13.5 mm
- net Net-(J5-PadB5): track 0.00 -> 10.5 mm
- net /Buttons/DPAD_UP: track 0.00 -> 10.2 mm, vias 0 -> 1
- net Net-(R4-Pad1): track 0.00 -> 8.86 mm
- net Net-(R1-Pad1): track 0.00 -> 8.75 mm
- net Net-(R7-Pad1): track 0.00 -> 8.42 mm
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- added copper zone on F.Cu, net GND
Other:
- outline, holes or cut-outs redrawn

Commit message: aaaa
Parts:
- removed R15: 0, Resistor_SMD:R_0603_1608Metric_Pad0.98x0.95mm_HandSolder
- removed REF**: MountingHole_2.1mm, MountingHole:MountingHole_2.1mm
- added D7: 824011, tvs:SOT95P280X145-5N, B.Cu at (118.9, 71.8)
- D6, J1, J5, R16, R17: moved to B.Cu
- R56, R57: footprint Resistor_SMD:R_0805_2012Metric_Pad1.20x1.40mm_HandSolder -> Resistor_SMD:R_0603_1608Metric_Pad0.98x0.95mm_HandSolder; moved to B.Cu
- moved R16 239.4 mm to (144.8, 72.8)
- moved J1 234.2 mm to (147.9, 65.3), turned to 0 degrees
- moved D6 230.4 mm to (151.5, 77.2), turned to 90 degrees
- moved R17 224.5 mm to (150.8, 72.8)
- moved R25 144.3 mm to (315.9, 119.3)
- moved C17 132.0 mm to (341.4, 75.0)
- moved J4 132.0 mm to (223.8, 143.2)
- moved R42 132.0 mm to (344.3, 62.2)
- moved C15 132.0 mm to (338.6, 56.0)
- moved C16 132.0 mm to (348.7, 64.7)
- moved C18 132.0 mm to (303.1, 47.5)
- moved C19 132.0 mm to (311.6, 47.5)
- moved C20 132.0 mm to (371.6, 103.2)
- moved C21 132.0 mm to (429.9, 100.7)
- moved C22 132.0 mm to (430.9, 95.5)
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Connections:
- J5 pad A7: Net-(J5-PadA6) -> Net-(J5-PadA7)
- J5 pad B7: Net-(J5-PadA6) -> Net-(J5-PadA7)
- R56 pad 1: GND -> Net-(J5-PadB5)
- R56 pad 2: Net-(J5-PadA5) -> GND
- R57 pad 1: GND -> Net-(J5-PadA5)
- R57 pad 2: Net-(J5-PadB5) -> GND
Routing:
- net GND: track 31.3 -> 145.3 mm, vias 6 -> 15
- net GND1: track 2.34 -> 67.0 mm, vias 3 -> 0
- net /Buttons/__DP_L: track 96.0 -> 46.9 mm
- net /Buttons/__DP_R: track 43.6 -> 13.7 mm
- net /Buttons/__DP_U: track 49.7 -> 21.2 mm
- net /+5v: track 0.00 -> 24.6 mm, vias 0 -> 3
- net /Display board (SNAP OFF BOARD)/+3.3v: track 0.00 -> 21.4 mm
- net /Buttons/__DP_D: track 35.8 -> 17.7 mm
- net /Buttons/START: track 0.00 -> 17.1 mm, vias 0 -> 1
- net /Buttons/SELECT: track 0.00 -> 17.0 mm, vias 0 -> 1
- net Net-(J5-PadA7): track 0.00 -> 13.8 mm
- net /+3.3v: track 0.00 -> 13.1 mm, vias 0 -> 3
- net /Buttons/__B_A: track 34.4 -> 47.1 mm
- net Net-(C9-Pad2): track 0.00 -> 11.3 mm
- net Net-(J5-PadA5): track 13.5 -> 2.24 mm
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- removed copper zone on F.Cu, net /Display board (SNAP OFF BOARD)/+3.3v
- removed copper zone on F.Cu, net GND
- removed copper zone on B.Cu, net GND1
- removed copper zone on F.Cu, net GND1

Commit message: a
Parts:
- D1, R13, SW12, TP2: moved to B.Cu
- moved D1 205.1 mm to (101.5, 88.2), turned to 90 degrees
- moved R13 202.2 mm to (101.5, 92.0), turned to 90 degrees
- moved TP2 199.0 mm to (104.8, 90.5), turned to 90 degrees
- moved SW12 108.5 mm to (194.8, 80.8)
- moved TP17 15.1 mm to (246.2, 25.0)
Routing:
- net Net-(D1-Pad1): track 0.00 -> 5.38 mm
- net /+5v: track 24.6 -> 23.8 mm

Commit message: aaaaaa
Parts:
- J4: moved to B.Cu
- moved J4 67.0 mm to (157.2, 135.2), turned to 180 degrees
- moved Module0 58.2 mm to (112.8, 131.5), turned to 90 degrees

Commit message: a
Parts:
- removed R55: 0, Resistor_SMD:R_1210_3225Metric_Pad1.30x2.65mm_HandSolder
Connections:
- J4 pad SH: Net-(J4-PadSH) -> unconnected-(J4-PadSH)

Commit message: aaaa
Parts:
- removed TP2: Activity, TestPoint:TestPoint_Pad_1.0x1.0mm
- C15: footprint Capacitor_SMD:C_2225_5664Metric_Pad1.80x6.60mm_HandSolder -> Capacitor_SMD:C_1206_3216Metric_Pad1.33x1.80mm_HandSolder; moved to B.Cu
- C8, J3, NT1, R22, R25, R36, R37, R38, R39, R43, R44, R51, R52, U3, U4: moved to B.Cu
- moved J3 219.1 mm to (108.4, 84.3), turned to 180 degrees
- moved R25 212.8 mm to (107.8, 75.0), turned to 180 degrees
- moved R22 207.0 mm to (119.8, 80.6)
- moved U4 205.1 mm to (119.8, 83.9), turned to 90 degrees
- moved C8 205.0 mm to (118.0, 88.0), turned to 0 degrees
- moved SW12 100.0 mm to (104.1, 123.0), turned to 180 degrees
- moved C15 87.4 mm to (385.9, 129.4), turned to 90 degrees
- moved D1 65.6 mm to (146.2, 136.2), turned to 0 degrees
- moved R13 60.3 mm to (142.5, 136.2), turned to 0 degrees
- moved R36 26.5 mm to (382.4, 133.1), turned to 180 degrees
- moved U3 20.1 mm to (377.6, 132.1), turned to 180 degrees
- moved NT1 17.6 mm to (375.8, 136.2)
- moved R51 15.7 mm to (375.5, 107.7)
- moved R38 15.4 mm to (378.1, 116.7), turned to 180 degrees
- moved R37 14.8 mm to (383.0, 129.5), turned to 90 degrees
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Connections:
- Module0 pad 25: /Buttons/SELECT -> /Buttons/START
- Module0 pad 45: /Buttons/START -> unconnected-(Module0-Pad45)
- Module0 pad 55: /Buttons/DPAD_DOWN -> /Buttons/SELECT
- R37 pad 2: GNDA -> GND
- R39 pad 2: GNDA -> GND
Routing:
- net /Connectors/USB2_D-: track 0.00 -> 38.9 mm
- net /Connectors/USB2_D+: track 0.00 -> 37.5 mm, vias 1 -> 3
- net /Buttons/GLOBAL_EN: track 0.00 -> 22.7 mm
- net /CM4/SD_PWR: track 0.00 -> 19.2 mm
- net Net-(R51-Pad2): track 0.00 -> 16.4 mm
- net Net-(R38-Pad2): track 0.00 -> 13.8 mm, vias 0 -> 2
- net GND: track 145.3 -> 157.3 mm, vias 15 -> 20
- net /Battery Charger/_CHIP_VCC: track 0.00 -> 6.37 mm
- net Net-(R43-Pad1): track 0.00 -> 5.11 mm
- net /Buttons/START: track 17.1 -> 22.2 mm
- net /Buttons/SELECT: track 17.0 -> 21.1 mm
- net Net-(D1-Pad1): track 5.38 -> 2.13 mm
- net Net-(J3-Pad9): track 0.00 -> 3.07 mm
- net /CM4/SD_PWR_ON: track 0.00 -> 2.26 mm
- net /+3.3v: track 13.1 -> 15.4 mm
- added copper zone on B.Cu, net GND

Commit message: aaaaaaaaaaaaaaaaaaaaaaaaaaaaaaaaaaaaaaaaaaaaaaaaaaaaaaaaaaaaaaaaa
Parts:
- C22: footprint Capacitor_SMD:C_1210_3225Metric_Pad1.33x2.70mm_HandSolder -> Capacitor_SMD:C_0603_1608Metric_Pad1.08x0.95mm_HandSolder
- R45, R46, R49, R53, R54: moved to B.Cu
- R47: footprint Resistor_SMD:R_0402_1005Metric_Pad0.72x0.64mm_HandSolder -> Resistor_SMD:R_2816_7142Metric_Pad3.20x4.45mm_HandSolder
- moved R53 77.5 mm to (363.8, 120.4), turned to 0 degrees
- moved R54 72.9 mm to (363.8, 117.8), turned to 180 degrees
- moved TP19 72.9 mm to (364.0, 130.6)
- moved C18 58.2 mm to (330.5, 98.8)
- moved C19 58.2 mm to (339.0, 98.8)
- moved C25 58.2 mm to (322.0, 98.8)
- moved C16 44.3 mm to (392.7, 69.2)
- moved C17 44.3 mm to (385.5, 79.6)
- moved R42 44.3 mm to (388.4, 66.7)
- moved R47 22.9 mm to (394.4, 94.8)
- moved D2 22.4 mm to (377.9, 92.6)
- moved D3 22.4 mm to (374.4, 92.6)
- moved R59 21.7 mm to (417.6, 89.6), turned to 90 degrees
- moved U3 19.9 mm to (372.2, 113.0)
- moved C15 18.4 mm to (374.2, 143.6)
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Routing:
- net Net-(R63-Pad2): track 0.00 -> 15.4 mm, vias 0 -> 2
- net Net-(R53-Pad2): track 0.00 -> 13.2 mm
- net Net-(R46-Pad2): track 0.00 -> 8.07 mm
- net Net-(R45-Pad1): track 0.00 -> 7.78 mm
- net Net-(C22-Pad1): track 0.00 -> 7.47 mm
- net Net-(R49-Pad1): track 0.00 -> 5.07 mm
- net Net-(R43-Pad1): track 5.11 -> 9.08 mm
- net Net-(R38-Pad2): track 13.8 -> 10.4 mm
- net Net-(R51-Pad2): track 16.4 -> 13.2 mm
- net Net-(R61-Pad2): track 0.00 -> 3.03 mm
- net /Battery Charger/_CHIP_VCC: track 6.37 -> 4.05 mm
- net GND: track 157.3 -> 159.6 mm, vias 20 -> 21
- net Net-(C21-Pad1): track 0.00 -> 2.16 mm
- net GNDA: track 0.00 -> 1.99 mm
- added copper zone on In1.Cu, net /+5v
- removed copper zone on B.Cu, net GND
