File: carrier/carrier.kicad_pcb (KiCad board)
At the start: 4 copper layers, 103.3 x 77.2 mm, 142 parts, among them J1 USB_C_Receptacle_USB2.0, J2 52271-0879, J3 Micro_SD_Card, J4 HDMI_D_1.4, J5 USB_C_Receptacle_USB2.0, J6 52271-0879, J7 AudioJack3_Switch, SW1 SKRRACE010, SW10 SKRBAAE010, SW11 SW_Push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

Commit message: jjjjj
Parts:
- removed the D6 at (151.5, 77.2)
- moved C8 97.2 mm to (37.5, 33.5)
- moved J3 97.2 mm to (27.9, 29.8)
- moved R22 97.2 mm to (39.3, 26.1)
- moved R25 97.2 mm to (27.2, 20.5)
- moved U4 97.2 mm to (39.3, 29.4)
- moved Module0 49.4 mm to (120.5, 82.8), turned to 0 degrees
- moved D7 27.2 mm to (151.5, 77.0), turned to 180 degrees
- moved TP1 14.1 mm to (148.2, 72.2)
Routing:
- net /Connectors/USB2_D-: track 38.9 -> 52.9 mm
- net /Connectors/USB2_D+: track 37.5 -> 49.0 mm, vias 3 -> 1
- net /Battery Charger/CHRG: track 4.30 -> 5.69 mm, vias 4 -> 3
- net /+5v: track 23.7 -> 22.4 mm
- net GND: track 155.4 -> 154.1 mm, vias 23 -> 24
- net /+3.3v: vias 3 -> 5
- removed copper zone on B.Cu, net /Battery Charger/CHRG

Commit message: getting back into the swing of this
aded some stuff for the resistors, moved some stuff about, removed the schmitt inverter (software is the solution for all our problems, forever)
Parts:
- removed U1: SN74HC14N, Package_SO:SO-14_3.9x8.65mm_P1.27mm
- C17, C21, C22, C23, C24, C7, C9, D4, D5, J7, R14, R18, R23, R24, R40, R41, R59, R61, R63, U5: moved to B.Cu
- moved R18 83.4 mm to (113.6, 98.0), turned to 90 degrees
- moved C7 79.2 mm to (110.6, 98.0), turned to -90 degrees
- moved R14 75.0 mm to (107.6, 98.0), turned to -90 degrees
- moved D4 74.8 mm to (112.1, 102.7), turned to 180 degrees
- moved TP18 74.3 mm to (284.0, -30.5)
- moved C12 74.3 mm to (257.9, -29.3)
- moved R29 74.3 mm to (263.2, -12.1)
- moved R34 74.3 mm to (270.8, -22.8)
- moved C14 74.3 mm to (277.6, -29.1)
- moved C9 69.7 mm to (107.6, 101.8), turned to -90 degrees
- moved R24 64.3 mm to (114.3, 108.0)
- moved D5 62.5 mm to (109.7, 109.5), turned to -90 degrees
- moved C23 60.8 mm to (114.3, 111.0)
- moved R31 59.9 mm to (272.2, -19.1)
- moved R35 59.9 mm to (295.1, -22.8)
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Connections:
- Module0 pad 24: unconnected-(Module0-Pad24) -> /Buttons/__DP_L
- Module0 pad 28: /Buttons/DPAD_LEFT -> unconnected-(Module0-Pad28)
- Module0 pad 29: /Buttons/BTN_B -> /Buttons/__B_B
- Module0 pad 31: /Buttons/DPAD_RIGHT -> /Buttons/__DP_R
- Module0 pad 34: unconnected-(Module0-Pad34) -> /Buttons/__DP_D
- Module0 pad 41: /Buttons/BTN_A -> /Buttons/__B_A
- Module0 pad 50: /Buttons/DPAD_UP -> /Buttons/__DP_U
- R10 pad 1: /+3.3v -> /Buttons/+3.3v
- R12 pad 1: /+3.3v -> /Buttons/+3.3v
- R2 pad 1: /+3.3v -> /Buttons/+3.3v
- R27 pad 1: /+3.3v -> /Buttons/+3.3v
- R30 pad 1: /+3.3v -> /Buttons/+3.3v
- R31 pad 1: /+3.3v -> /Buttons/+3.3v
- R33 pad 1: /+3.3v -> /Buttons/+3.3v
- R35 pad 1: /+3.3v -> /Buttons/+3.3v
- R48 pad 2: GND -> /Battery Charger/_CHIP_VCC
- R5 pad 1: /+3.3v -> /Buttons/+3.3v
- R50 pad 2: GND -> /Battery Charger/_CHIP_VCC
- R6 pad 1: /+3.3v -> /Buttons/+3.3v
- R8 pad 1: /+3.3v -> /Buttons/+3.3v
- TP10 pad 1: /Buttons/BTN_A -> /Buttons/__B_A
- TP11 pad 1: /Buttons/BTN_B -> /Buttons/__B_B
- TP6 pad 1: /Buttons/DPAD_UP -> /Buttons/__DP_U
- TP7 pad 1: /Buttons/DPAD_DOWN -> /Buttons/__DP_D
- TP8 pad 1: /Buttons/DPAD_LEFT -> /Buttons/__DP_L
- TP9 pad 1: /Buttons/DPAD_RIGHT -> /Buttons/__DP_R
Routing:
- net /CM4/AUX1: track 0.00 -> 38.4 mm
- net /Buttons/__DP_L: track 46.9 -> 65.3 mm, vias 0 -> 1
- net Net-(C9-Pad2): track 11.3 -> 28.5 mm
- net GND: track 154.1 -> 169.6 mm, vias 24 -> 28
- net GNDA: track 1.99 -> 17.2 mm, vias 0 -> 3
- net /Battery Charger/_CHIP_VCC: track 18.1 -> 33.2 mm, vias 2 -> 3
- net /Buttons/DPAD_RIGHT: track 14.9 -> 0.00 mm
- net Net-(R36-Pad2): track 0.00 -> 12.6 mm
- net /CM4/AUX0: track 0.00 -> 11.3 mm
- net /Buttons/DPAD_DOWN: track 11.1 -> 0.00 mm
- net Net-(U3-Pad22): track 0.00 -> 11.1 mm, vias 0 -> 1
- net /Buttons/DPAD_UP: track 10.2 -> 0.00 mm
- net /Buttons/__DP_R: track 13.7 -> 23.4 mm
- net Net-(C17-Pad1): track 0.00 -> 9.15 mm
- net Net-(R4-Pad1): track 8.86 -> 0.00 mm
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Other:
- board text added: "how tf do you wire this?"

Commit message: commit
Parts:
- moved J2 4.13 mm to (155.6, 80.2)
- moved TP1 4.13 mm to (152.2, 71.1)
- moved TP12 4.13 mm to (152.4, 85.0)
- moved TP13 4.13 mm to (166.0, 81.3)
- moved TP3 4.13 mm to (159.1, 85.0)
- moved TP4 4.13 mm to (156.9, 85.0)
- moved TP5 4.13 mm to (154.6, 85.0)
- moved R28 0.63 mm to (136.8, 74.8), turned to 0 degrees
Routing:
- net /Buttons/BTN_BACKLIGHT: track 0.00 -> 11.8 mm
- net GND: track 169.6 -> 181.1 mm
- net Net-(R28-Pad1): track 0.00 -> 5.56 mm

Commit message: we are nearing completion for this version
maybe one day we will make a second version
Parts:
- D1, R13: moved to F.Cu
- R40, R41, R43, R44, R45, R63: footprint Resistor_SMD:R_0603_1608Metric_Pad0.98x0.95mm_HandSolder -> Resistor_SMD:R_0402_1005Metric_Pad0.72x0.64mm_HandSolder
- moved C15 256.9 mm to (125.9, 77.5), turned to 0 degrees
- moved D3 229.9 mm to (163.5, 124.3)
- moved R50 229.9 mm to (163.5, 120.5)
- moved J4 114.6 mm to (126.8, 243.8)
- moved R25 104.1 mm to (102.6, 92.2)
- moved R22 99.1 mm to (101.8, 102.9), turned to 0 degrees
- moved J3 96.6 mm to (108.2, 83.5), turned to -90 degrees
- moved U4 94.1 mm to (101.8, 99.7), turned to -90 degrees
- moved C8 90.7 mm to (103.6, 95.6), turned to 180 degrees
- moved R13 29.8 mm to (167.7, 120.5), turned to 90 degrees
- moved D1 24.6 mm to (167.8, 124.2), turned to 90 degrees
- moved R43 1.92 mm to (368.8, 120.2)
- moved R40 1.57 mm to (372.8, 107.8)
- moved R41 1.50 mm to (370.2, 107.8)
- moved R44 0.66 mm to (370.4, 118.0)
Routing:
- net /Display board (SNAP OFF BOARD)/+3.3v: track 21.4 -> 56.4 mm, vias 0 -> 2
- net Net-(R7-Pad1): track 8.42 -> 28.6 mm
- net /CM4/SD_PWR_ON: track 2.26 -> 19.8 mm, vias 0 -> 2
- net Net-(D3-Pad1): track 0.00 -> 14.8 mm, vias 0 -> 1
- net /Battery Charger/_CHIP_VCC: track 33.2 -> 25.3 mm
- net /CM4/SD_PWR: track 19.2 -> 24.3 mm
- net Net-(J3-Pad9): track 2.80 -> 7.66 mm
- net GNDA: track 17.2 -> 21.4 mm, vias 3 -> 4
- net GND1: track 67.0 -> 63.9 mm
- net Net-(R38-Pad2): track 9.61 -> 6.51 mm
- net GND: track 181.1 -> 178.6 mm, vias 28 -> 34
- net Net-(D1-Pad1): track 2.13 -> 0.00 mm
- net Net-(R43-Pad1): track 8.50 -> 6.69 mm
- net /Battery Charger/CHRG: track 7.99 -> 6.47 mm, vias 5 -> 8
- net Net-(R40-Pad2): track 4.44 -> 3.06 mm
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- added copper zone on B.Cu, net /Battery Charger/CHRG
- added copper zone on B.Cu, net GNDA

Commit message: getting there!!
Parts:
- removed J4: HDMI_D_1.4, Connector_HDMI:HDMI_Micro-D_Molex_46765-1x01
- added REF**: OSHW-Logo_11.4x12mm_SilkScreen, Symbol:OSHW-Logo_11.4x12mm_SilkScreen, B.Cu at (86.2, 57.4)
- D1: value LED -> ACT
- D2: value LED -> CHRG
- D3: value LED -> PWR
- R42: moved to B.Cu
- R51: moved to F.Cu
- moved R44 318.6 mm to (53.4, 85.8)
- moved C16 316.5 mm to (82.7, 133.2)
- moved C21 316.5 mm to (111.5, 155.4)
- moved C22 316.5 mm to (108.7, 159.0)
- moved R59 316.5 mm to (121.2, 153.6)
- moved R61 316.5 mm to (120.2, 159.6)
- moved R63 316.5 mm to (105.8, 159.0)
- moved U5 316.5 mm to (115.2, 158.8)
- moved R40 316.4 mm to (59.9, 60.5)
- moved R41 316.4 mm to (57.4, 60.5)
- moved R49 316.4 mm to (60.4, 71.9)
- moved R53 316.4 mm to (53.0, 74.9)
- moved R45 315.7 mm to (49.4, 84.2)
- moved R46 315.0 mm to (52.4, 68.2)
- moved R54 315.0 mm to (52.4, 70.6)
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Connections:
- net Net-(L1-Pad1) renamed /Battery Charger/__SW
- net Net-(L1-Pad2) renamed /Battery Charger/__CSP
- R44 pad 2: GND -> GNDA
- R45 pad 2: GND -> GNDA
Routing:
- net /CM4/AUX0: track 11.3 -> 71.5 mm, vias 0 -> 2
- net /CM4/SD_PWR_ON: track 19.8 -> 60.0 mm
- net /CM4/AUX1: track 38.4 -> 67.1 mm
- net /Buttons/__DP_L: track 65.3 -> 42.4 mm, vias 1 -> 4
- net /Battery Charger/_CHIP_VCC: track 25.3 -> 3.72 mm, vias 3 -> 1
- net /Battery Charger/BATT: track 0.00 -> 17.8 mm, vias 0 -> 2
- net /Buttons/GLOBAL_EN: track 24.3 -> 41.4 mm
- net Net-(R53-Pad2): track 13.2 -> 0.00 mm
- net Net-(D3-Pad1): track 14.8 -> 2.62 mm
- net Net-(R42-Pad1): track 0.00 -> 9.92 mm
- net Net-(R51-Pad2): track 10.8 -> 1.60 mm
- net Net-(R4-Pad1): track 0.00 -> 9.00 mm
- net Net-(R46-Pad2): track 8.07 -> 0.00 mm
- net Net-(R45-Pad1): track 7.88 -> 0.00 mm
- net Net-(C17-Pad1): track 9.15 -> 1.51 mm
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- added copper zone on B.Cu, net /+5v
- added copper zone on In1.Cu, net /Battery Charger/CHRG
- added copper zone on B.Cu, net /Battery Charger/__CSP
- added copper zone on B.Cu, net /Battery Charger/__SW
- removed copper zone on B.Cu, net GNDA
Other:
- outline, holes or cut-outs redrawn
- board text added: "IMPORTANT: WE NEED TO ADD A BATTERY CONNECTOR!!!!! NOTE 2: change rating and size for current resistor? this seems a little bit ludicrous"
- board text added: "github.com/cinnamondev"
- board text added: "pwr"
- board text removed: "BOOST | CHARGE"
