File: carrier/_autosave-carrier.kicad_pcb (KiCad board)
At the start: 4 copper layers, 103.3 x 77.2 mm, 142 parts, among them J1 USB_C_Receptacle_USB2.0, J2 52271-0879, J3 Micro_SD_Card, J4 HDMI_D_1.4, J5 USB_C_Receptacle_USB2.0, J6 52271-0879, J7 AudioJack3_Switch, SW1 SKRRACE010, SW10 SKRBAAE010, SW11 SW_Push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

Commit message: a
Parts:
- D6, D7: footprint Package_TO_SOT_SMD:SOT-143_Handsoldering -> CM4IO:SOT143-4L
- TP19, TP26: moved to B.Cu
- moved D6 2.20 mm to (121.1, 74.1), turned to 0 degrees
- turned TP19 to 180 degrees
- turned TP26 to 180 degrees
Routing:
- net Net-(J5-PadA7): track 15.1 -> 12.4 mm
- net Net-(J5-PadA6): track 10.4 -> 8.39 mm
- net GND: vias 21 -> 23
- net /Battery Charger/CHRG: vias 8 -> 4
- net (no net): vias 1 -> 0
- added copper zone on B.Cu, net GND
