File: carrier/_autosave-carrier.kicad_pcb (KiCad board)
At the start: 4 copper layers, 103.3 x 77.2 mm, 140 parts, among them J1 USB_C_Receptacle_USB2.0, J2 52271-0879, J3 Micro_SD_Card, J5 USB_C_Receptacle_USB2.0, J6 52271-0879, J7 AudioJack3_Switch, SW1 SKRRACE010, SW10 SKRBAAE010, SW11 SW_Push, SW12 SW_DIP_x04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

Commit message: a
Parts:
- D6: moved to F.Cu
- turned D6 to 180 degrees
Changed lines of the file:
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@@
     )
   )
+  (footprint "CM4IO:SOT143-4L" (layer "F.Cu")
+    (at 119.6625 74.1 180)
+    (property "Description" "Wurth Elektronik 824011 Dual Uni-Directional TVS Diode Array, 5-Pin SOT-23")
+    (property "Height" "1.45")
+    (property "Manufacturer_Name" "Wurth Elektronik")
+    (property "Manufacturer_Part_Number" "824011")
+    (property "Mouser Part Number" "710-824011")
+    (property "Mouser Price/Stock" "https://www.mouser.co.uk/ProductDetail/Wurth-Elektronik/824011?qs=Wn16VcyqZWrHR48Vn%2FB8%252Bg%3D%3D")
+    (property "Sheetfile" "connectors.kicad_sch")
+    (property "Sheetname" "Connectors")
+    (fp_text reference "D6" (at 0 -0.5 180 unlocked) (layer "F.SilkS")
+      (effects (font (size 1 1) (thickness 0.15)))
+    )
+    (fp_text value "8240119" (at 0 1 180 unlocked) (layer "F.Fab")
+      (effects (font (size 1 1) (thickness 0.15)))
+    )
+    (fp_text user "${REFERENCE}" (at 0 2.5 180 unlocked) (layer "F.Fab")
+      (effects (font (size 1 1) (thickness 0.15)))
+    )
+    (fp_line (start -1.6 0.8) (end -1.6 0.4) (layer "F.SilkS") (width 0.1))
+    (fp_line (start 1.3 -0.8) (end 1.6 -0.8) (layer "F.SilkS") (width 0.1))
+    (fp_line (start 1.6 -0.8) (end 1.6 -0.2) (layer "F.SilkS") (width 0.1))
+    (fp_line (start -1.6 -0.8) (end -1.6 -0.2) (layer "F.SilkS") (width 0.1))
+    (fp_line (start 1.3 0.8) (end 1.6 0.8) (layer "F.SilkS") (width 0.1))
+    (fp_line (start -1.3 -0.8) (end -1.6 -0.8) (layer "F.SilkS") (width 0.1))
+    (fp_line (start 1.6 0.8) (end 1.6 0.3) (layer "F.SilkS") (width 0.1))
+    (fp_line (start -1.3 0.8) (end -1.6 0.8) (layer "F.SilkS") (width 0.1))
+    (fp_line (start -1.3 0.8) (end -1.3 1.27) (layer "F.SilkS") (width 0.1))
+    (fp_line (start 1.75 -2) (end 1.75 2) (layer "F.CrtYd") (width 0.05))
+    (fp_line (start -1.75 -2) (end -1.75 2) (layer "F.CrtYd") (width 0.05))
+    (fp_line (start 1.75 2) (end -1.75 2) (layer "F.CrtYd") (width 0.05))
+    (fp_line (start 1.75 -2) (end -1.75 -2) (layer "F.CrtYd") (width 0.05))
+    (fp_line (start 1.46 -0.65) (end -1.46 -0.65) (layer "F.Fab") (width 0.1))
+    (fp_line (start -1.46 0.65) (end 1.46 0.65) (layer "F.Fab") (width 0.1))
+    (fp_line (start -1.46 0.65) (end -1.46 -0.65) (layer "F.Fab") (width 0.1))
+    (fp_line (start 1.46 -0.65) (end 1.46 0.65) (layer "F.Fab") (width 0.1))
+    (pad "1" smd rect locked (at -0.76 1 180) (size 0.94 1.31) (layers "F.Cu" "F.Paste" "F.Mask")
+      (net 2 "GND") (pinfunction "GND") (pintype "power_in"))
+    (pad "2" smd rect locked (at 0.96 1 180) (size 0.55 1.31) (layers "F.Cu" "F.Paste" "F.Mask")
+      (net 105 "Net-(D6-Pad2)") (pinfunction "I/O1") (pintype "bidirectional"))
+    (pad "3" smd rect locked (at 0.96 -1 180) (size 0.55 1.31) (layers "F.Cu" "F.Paste" "F.Mask")
+      (net 106 "Net-(D6-Pad3)") (pinfunction "I/O2") (pintype "bidirectional"))
+    (pad "4" smd rect locked (at -0.96 -1 180) (size 0.55 1.31) (layers "F.Cu" "F.Paste" "F.Mask")
+      (net 25 "/Battery Charger/CHRG") (pinfunction "VDD") (pintype "power_in"))
+  )
   (footprint "sw:TE_Connectivity-1-1825027-1-0-0-Recommended_Land_Pattern_" (layer "F.Cu")
     (at 284.7192 -14.1622)
@@
     )
   )
-  (footprint "CM4IO:SOT143-4L" (layer "B.Cu")
-    (at 119.6625 74.1)
-    (property "Description" "Wurth Elektronik 824011 Dual Uni-Directional TVS Diode Array, 5-Pin SOT-23")
-    (property "Height" "1.45")
-    (property "Manufacturer_Name" "Wurth Elektronik")
-    (property "Manufacturer_Part_Number" "824011")
-    (property "Mouser Part Number" "710-824011")
-    (property "Mouser Price/Stock" "https://www.mouser.co.uk/ProductDetail/Wurth-Elektronik/824011?qs=Wn16VcyqZWrHR48Vn%2FB8%252Bg%3D%3D")
-    (property "Sheetfile" "connectors.kicad_sch")
-    (property "Sheetname" "Connectors")
-    (fp_text reference "D6" (at 0 0.5 180 unlocked) (layer "B.SilkS")
-      (effects (font (size 1 1) (thickness 0.15)) (justify mirror))
-    )
-    (fp_text value "8240119" (at 0 -1 180 unlocked) (layer "B.Fab")
-      (effects (font (size 1 1) (thickness 0.15)) (justify mirror))
-    )
-    (fp_text user "${REFERENCE}" (at 0 -2.5 180 unlocked) (layer "B.Fab")
-      (effects (font (size 1 1) (thickness 0.15)) (justify mirror))
-    )
-    (fp_line (start -1.6 -0.8) (end -1.6 -0.4) (layer "B.SilkS") (width 0.1))
-    (fp_line (start 1.3 0.8) (end 1.6 0.8) (layer "B.SilkS") (width 0.1))
-    (fp_line (start 1.6 0.8) (end 1.6 0.2) (layer "B.SilkS") (width 0.1))
-    (fp_line (start -1.6 0.8) (end -1.6 0.2) (layer "B.SilkS") (width 0.1))
-    (fp_line (start 1.3 -0.8) (end 1.6 -0.8) (layer "B.SilkS") (width 0.1))
-    (fp_line (start -1.3 0.8) (end -1.6 0.8) (layer "B.SilkS") (width 0.1))
-    (fp_line (start 1.6 -0.8) (end 1.6 -0.3) (layer "B.SilkS") (width 0.1))
-    (fp_line (start -1.3 -0.8) (end -1.6 -0.8) (layer "B.SilkS") (width 0.1))
-    (fp_line (start -1.3 -0.8) (end -1.3 -1.27) (layer "B.SilkS") (width 0.1))
-    (fp_line (start 1.75 2) (end 1.75 -2) (layer "B.CrtYd") (width 0.05))
-    (fp_line (start -1.75 2) (end -1.75 -2) (layer "B.CrtYd") (width 0.05))
-    (fp_line (start 1.75 -2) (end -1.75 -2) (layer "B.CrtYd") (width 0.05))
-    (fp_line (start 1.75 2) (end -1.75 2) (layer "B.CrtYd") (width 0.05))
-    (fp_line (start 1.46 0.65) (end -1.46 0.65) (layer "B.Fab") (width 0.1))
-    (fp_line (start -1.46 -0.65) (end 1.46 -0.65) (layer "B.Fab") (width 0.1))
-    (fp_line (start -1.46 -0.65) (end -1.46 0.65) (layer "B.Fab") (width 0.1))
-    (fp_line (start 1.46 0.65) (end 1.46 -0.65) (layer "B.Fab") (width 0.1))
-    (pad "1" smd rect locked (at -0.76 -1) (size 0.94 1.31) (layers "B.Cu" "B.Paste" "B.Mask")
-      (net 2 "GND") (pinfunction "GND") (pintype "power_in"))
-    (pad "2" smd rect locked (at 0.96 -1) (size 0.55 1.31) (layers "B.Cu" "B.Paste" "B.Mask")
-      (net 105 "Net-(D6-Pad2)") (pinfunction "I/O1") (pintype "bidirectional"))
-    (pad "3" smd rect locked (at 0.96 1) (size 0.55 1.31) (layers "B.Cu" "B.Paste" "B.Mask")
-      (net 106 "Net-(D6-Pad3)") (pinfunction "I/O2") (pintype "bidirectional"))
-    (pad "4" smd rect locked (at -0.96 1) (size 0.55 1.31) (layers "B.Cu" "B.Paste" "B.Mask")
-      (net 25 "/Battery Charger/CHRG") (pinfunction "VDD") (pintype "power_in"))
-  )
   (footprint "Resistor_SMD:R_0603_1608Metric_Pad0.98x0.95mm_HandSolder" (layer "B.Cu")
