File: carrier/MCU.kicad_sch (KiCad schematic)
At the start: 0 parts

Commit message: thingy
Changed lines of the file:
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@@
     (effects (font (size 1.27 1.27)) (justify left bottom))
   )
+  (hierarchical_label "BTN_POW" (shape input) (at 50.165 104.775 0)
+    (effects (font (size 1.27 1.27)) (justify left))
+  )
 )
