File: carrier/display_board.kicad_sch (KiCad schematic)
At the start: 9 parts, among them J6 52271-0879, U2 ER-CON40HT-1

Commit message: a
Connections:
- no-connect marks 16 -> 22
Changed lines of the file:
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@@
   (junction (at 145.415 104.14) (diameter 0.9144) (color 0 0 0 0))
   (junction (at 145.415 106.045) (diameter 0.9144) (color 0 0 0 0))
+  (no_connect (at 149.225 34.29))
+  (no_connect (at 149.225 36.195))
+  (no_connect (at 149.225 38.1))
+  (no_connect (at 149.225 40.005))
+  (no_connect (at 149.225 53.34))
+  (no_connect (at 149.225 55.245))
   (no_connect (at 149.225 64.77))
   (no_connect (at 149.225 66.675))

Commit message: fixed switching and added fuel gague
Parts:
- renumbered J6 to J7, R19 to R48, TP20 to TP19, TP24 to TP20, TP23 to TP21, TP21 to TP23, TP25 to TP24, U2 to U4
Changed lines of the file:
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@@
     (rev "indevRev2")
   )
+  (junction (at 145.415 62.865) (diameter 0.9144) (color 0 0 0 0))
   (junction (at 143.51 43.815) (diameter 0.9144) (color 0 0 0 0))
+  (junction (at 144.145 109.855) (diameter 0.9144) (color 0 0 0 0))
+  (junction (at 145.415 98.425) (diameter 0.9144) (color 0 0 0 0))
+  (junction (at 145.415 106.045) (diameter 0.9144) (color 0 0 0 0))
+  (junction (at 145.415 102.235) (diameter 0.9144) (color 0 0 0 0))
+  (junction (at 64.77 46.355) (diameter 0.9144) (color 0 0 0 0))
+  (junction (at 64.77 43.18) (diameter 0.9144) (color 0 0 0 0))
   (junction (at 145.415 100.33) (diameter 0.9144) (color 0 0 0 0))
-  (junction (at 145.415 98.425) (diameter 0.9144) (color 0 0 0 0))
-  (junction (at 144.145 109.855) (diameter 0.9144) (color 0 0 0 0))
-  (junction (at 64.77 46.355) (diameter 0.9144) (color 0 0 0 0))
-  (junction (at 145.415 62.865) (diameter 0.9144) (color 0 0 0 0))
+  (junction (at 145.415 104.14) (diameter 0.9144) (color 0 0 0 0))
   (junction (at 64.77 48.26) (diameter 0.9144) (color 0 0 0 0))
-  (junction (at 145.415 106.045) (diameter 0.9144) (color 0 0 0 0))
+  (junction (at 64.77 66.04) (diameter 0.9144) (color 0 0 0 0))
   (junction (at 64.77 41.91) (diameter 0.9144) (color 0 0 0 0))
-  (junction (at 145.415 104.14) (diameter 0.9144) (color 0 0 0 0))
-  (junction (at 145.415 102.235) (diameter 0.9144) (color 0 0 0 0))
-  (junction (at 64.77 43.18) (diameter 0.9144) (color 0 0 0 0))
-  (junction (at 64.77 66.04) (diameter 0.9144) (color 0 0 0 0))
   (no_connect (at 149.225 34.29))
   (no_connect (at 149.225 36.195))
@@
   (no_connect (at 149.225 55.245))
   (no_connect (at 149.225 53.34))
+  (no_connect (at 149.225 92.71))
+  (no_connect (at 149.225 94.615))
   (no_connect (at 149.225 64.77))
   (no_connect (at 149.225 66.675))
@@
   (no_connect (at 149.225 88.9))
   (no_connect (at 149.225 90.805))
-  (no_connect (at 149.225 92.71))
-  (no_connect (at 149.225 94.615))
   (wire (pts (xy 64.77 60.96) (xy 88.9 60.96))
     (stroke (width 0) (type solid) (color 0 0 0 0))
@@
     (stroke (width 0) (type solid) (color 0 0 0 0))
   )
+  (wire (pts (xy 137.795 43.815) (xy 143.51 43.815))
+    (stroke (width 0) (type solid) (color 0 0 0 0))
+  )
   (wire (pts (xy 143.51 43.815) (xy 149.225 43.815))
     (stroke (width 0) (type solid) (color 0 0 0 0))
   )
-  (wire (pts (xy 137.795 43.815) (xy 143.51 43.815))
-    (stroke (width 0) (type solid) (color 0 0 0 0))
-  )
   (wire (pts (xy 80.645 51.435) (xy 80.645 53.34))
     (stroke (width 0) (type solid) (color 0 0 0 0))
@@
     (stroke (width 0) (type solid) (color 0 0 0 0))
   )
+  (wire (pts (xy 145.415 106.045) (xy 145.415 104.14))
+    (stroke (width 0) (type solid) (color 0 0 0 0))
+  )
+  (wire (pts (xy 145.415 62.865) (xy 145.415 98.425))
+    (stroke (width 0) (type solid) (color 0 0 0 0))
+  )
+  (wire (pts (xy 145.415 102.235) (xy 145.415 104.14))
+    (stroke (width 0) (type solid) (color 0 0 0 0))
+  )
+  (wire (pts (xy 145.415 111.125) (xy 145.415 106.045))
+    (stroke (width 0) (type solid) (color 0 0 0 0))
+  )
+  (wire (pts (xy 145.415 100.33) (xy 145.415 102.235))
+    (stroke (width 0) (type solid) (color 0 0 0 0))
+  )
+  (wire (pts (xy 145.415 98.425) (xy 145.415 100.33))
+    (stroke (width 0) (type solid) (color 0 0 0 0))
+  )
+  (wire (pts (xy 145.415 62.865) (xy 145.415 41.91))
+    (stroke (width 0) (type solid) (color 0 0 0 0))
+  )
   (wire (pts (xy 145.415 41.91) (xy 149.225 41.91))
-    (stroke (width 0) (type solid) (color 0 0 0 0))
-  )
-  (wire (pts (xy 145.415 62.865) (xy 145.415 41.91))
-    (stroke (width 0) (type solid) (color 0 0 0 0))
-  )
-  (wire (pts (xy 145.415 62.865) (xy 145.415 98.425))
-    (stroke (width 0) (type solid) (color 0 0 0 0))
-  )
-  (wire (pts (xy 145.415 106.045) (xy 145.415 104.14))
-    (stroke (width 0) (type solid) (color 0 0 0 0))
-  )
-  (wire (pts (xy 145.415 102.235) (xy 145.415 104.14))
-    (stroke (width 0) (type solid) (color 0 0 0 0))
-  )
-  (wire (pts (xy 145.415 111.125) (xy 145.415 106.045))
-    (stroke (width 0) (type solid) (color 0 0 0 0))
-  )
-  (wire (pts (xy 145.415 100.33) (xy 145.415 102.235))
-    (stroke (width 0) (type solid) (color 0 0 0 0))
-  )
-  (wire (pts (xy 145.415 98.425) (xy 145.415 100.33))
     (stroke (width 0) (type solid) (color 0 0 0 0))
   )
@@
   (symbol (lib_id "Connector:TestPoint") (at 90.805 46.355 270) (unit 1)
     (in_bom yes) (on_board yes)
-    (property "Reference" "TP20" (id 0) (at 95.885 45.0849 90)
+    (property "Reference" "TP19" (id 0) (at 95.885 45.0849 90)
       (effects (font (size 1.27 1.27)) (justify left))
     )
@@
   (symbol (lib_id "Connector:TestPoint") (at 90.805 71.12 270) (unit 1)
     (in_bom yes) (on_board yes) (fields_autoplaced)
-    (property "Reference" "TP25" (id 0) (at 95.885 69.8499 90)
+    (property "Reference" "TP24" (id 0) (at 95.885 69.8499 90)
       (effects (font (size 1.27 1.27)) (justify left))
     )
@@
   (symbol (lib_id "Connector:TestPoint") (at 90.805 66.04 270) (unit 1)
     (in_bom yes) (on_board yes) (fields_autoplaced)
-    (property "Reference" "TP21" (id 0) (at 95.885 64.7699 90)
+    (property "Reference" "TP23" (id 0) (at 95.885 64.7699 90)
       (effects (font (size 1.27 1.27)) (justify left))
     )
@@
   (symbol (lib_id "Connector:TestPoint") (at 90.805 51.435 270) (unit 1)
     (in_bom yes) (on_board yes) (fields_autoplaced)
-    (property "Reference" "TP24" (id 0) (at 95.885 50.1649 90)
+    (property "Reference" "TP20" (id 0) (at 95.885 50.1649 90)
       (effects (font (size 1.27 1.27)) (justify left))
     )
@@
   (symbol (lib_id "Device:R") (at 134.62 96.52 90) (unit 1)
     (in_bom yes) (on_board yes)
-    (property "Reference" "R19" (id 0) (at 134.62 94.615 90))
+    (property "Reference" "R48" (id 0) (at 134.62 94.615 90))
     (property "Value" "33" (id 1) (at 134.62 96.52 90))
     (property "Footprint" "Resistor_SMD:R_0805_2012Metric_Pad1.20x1.40mm_HandSolder" (id 2) (at 134.62 98.298 90)
@@
   (symbol (lib_id "Connector:TestPoint") (at 90.805 55.88 270) (unit 1)
     (in_bom yes) (on_board yes) (fields_autoplaced)
-    (property "Reference" "TP23" (id 0) (at 95.885 54.6099 90)
+    (property "Reference" "TP21" (id 0) (at 95.885 54.6099 90)
       (effects (font (size 1.27 1.27)) (justify left))
     )
@@
   (symbol (lib_id "power:GND1") (at 64.77 41.91 90) (unit 1)
     (in_bom yes) (on_board yes) (fields_autoplaced)
-    (property "Reference" "#PWR0104" (id 0) (at 71.12 41.91 0)
+    (property "Reference" "#PWR044" (id 0) (at 71.12 41.91 0)
       (effects (font (size 1.27 1.27)) hide)
     )
@@
   (symbol (lib_id "power:GND1") (at 145.415 111.125 0) (unit 1)
     (in_bom yes) (on_board yes) (fields_autoplaced)
-    (property "Reference" "#PWR0101" (id 0) (at 145.415 117.475 0)
+    (property "Reference" "#PWR045" (id 0) (at 145.415 117.475 0)
       (effects (font (size 1.27 1.27)) hide)
     )
@@
   (symbol (lib_id "CON40:ER-CON40HT-1") (at 149.225 34.29 0) (unit 1)
     (in_bom yes) (on_board yes) (fields_autoplaced)
-    (property "Reference" "U2" (id 0) (at 170.18 72.0216 0)
+    (property "Reference" "U4" (id 0) (at 170.18 72.0216 0)
       (effects (font (size 1.27 1.27)) (justify left))
     )
@@
   (symbol (lib_id "MOLEXZIF:52271-0879") (at 67.31 66.04 90) (unit 1)
     (in_bom yes) (on_board yes) (fields_autoplaced)
-    (property "Reference" "J6" (id 0) (at 61.1505 32.385 90))
+    (property "Reference" "J7" (id 0) (at 61.1505 32.385 90))
     (property "Value" "52271-0879" (id 1) (at 61.1505 34.925 90))
     (property "Footprint" "MOLEXZIF:Molex-52271-0879-Manufacturer_Recommended" (id 2) (at 49.53 66.04 0)

Commit message: new footprints - order stuff soon
Parts:
- removed J7: 52271-0879, MOLEXZIF:Molex-52271-0879-Manufacturer_Recommended, symbol MOLEXZIF:52271-0879
- added J7: Conn_01x10, CM4IO:522711169, symbol Connector_Generic:Conn_01x10
- TP19, TP20, TP21, TP22, TP23, TP24: footprint TestPoint:TestPoint_Pad_1.0x1.0mm -> TestPoint:TestPoint_Pad_2.0x2.0mm
- renumbered R48 to R47
Connections:
- net +3.3v: now also J7.10 (Pin_10), J7.8 (Pin_8), J7.9 (Pin_9)
- net GND1: no longer TP19.1
- net SPI0_CE0_N: now also J7.7 (Pin_7)
- net SPI0_MOSI: now also J7.4 (Pin_4)
- net SPI0_SCLK: now also J7.6 (Pin_6)
- net SPI_MISO: now also J7.5 (Pin_5)
- new net: J7.1 (Pin_1), J7.2 (Pin_2), J7.3 (Pin_3), TP19.1
Other:
- moved on the sheet: TP19
