File: adaptor/adaptor.kicad_sch (KiCad schematic)
At the start: 2 parts, among them J1 1-84952-5, J2 1-84952-5

Commit message: adaptor + some design wrork
Connections:
- net at J2.1: now also J1.15; no longer J1.1
- net at J2.10: now also J1.6; no longer J1.10
- net at J2.11: now also J1.5; no longer J1.11
- net at J2.12: now also J1.4; no longer J1.12
- net at J2.13: now also J1.3; no longer J1.13
- net at J2.14: now also J1.2; no longer J1.14
- net at J2.15: now also J1.1; no longer J1.15
- net at J2.2: now also J1.14; no longer J1.2
- net at J2.3: now also J1.13; no longer J1.3
- net at J2.4: now also J1.12; no longer J1.4
- net at J2.5: now also J1.11; no longer J1.5
- net at J2.6: now also J1.10; no longer J1.6
- net at J2.7: now also J1.9; no longer J1.7
- net at J2.9: now also J1.7; no longer J1.9
Other:
- moved on the sheet: J2
Changed lines of the file:
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@@
 (kicad_sch (version 20211123) (generator eeschema)
   (paper "A4")
-  (wire (pts (xy 134.62 96.52) (xy 149.86 96.52))
-    (stroke (width 0) (type default) (color 0 0 0 0))
-  )
-  (wire (pts (xy 134.62 114.3) (xy 149.86 114.3))
-    (stroke (width 0) (type default) (color 0 0 0 0))
-  )
-  (wire (pts (xy 134.62 101.6) (xy 149.86 101.6))
-    (stroke (width 0) (type default) (color 0 0 0 0))
-  )
-  (wire (pts (xy 134.62 119.38) (xy 149.86 119.38))
-    (stroke (width 0) (type default) (color 0 0 0 0))
-  )
-  (wire (pts (xy 134.62 99.06) (xy 149.86 99.06))
-    (stroke (width 0) (type default) (color 0 0 0 0))
-  )
-  (wire (pts (xy 134.62 91.44) (xy 149.86 91.44))
-    (stroke (width 0) (type default) (color 0 0 0 0))
-  )
-  (wire (pts (xy 134.62 109.22) (xy 149.86 109.22))
-    (stroke (width 0) (type default) (color 0 0 0 0))
-  )
-  (wire (pts (xy 134.62 116.84) (xy 149.86 116.84))
-    (stroke (width 0) (type default) (color 0 0 0 0))
-  )
-  (wire (pts (xy 134.62 106.68) (xy 149.86 106.68))
-    (stroke (width 0) (type default) (color 0 0 0 0))
-  )
-  (wire (pts (xy 134.62 104.14) (xy 149.86 104.14))
-    (stroke (width 0) (type default) (color 0 0 0 0))
-  )
-  (wire (pts (xy 134.62 121.92) (xy 149.86 121.92))
-    (stroke (width 0) (type default) (color 0 0 0 0))
-  )
-  (wire (pts (xy 134.62 111.76) (xy 149.86 111.76))
-    (stroke (width 0) (type default) (color 0 0 0 0))
-  )
-  (wire (pts (xy 134.62 86.36) (xy 149.86 86.36))
-    (stroke (width 0) (type default) (color 0 0 0 0))
-  )
-  (wire (pts (xy 134.62 88.9) (xy 149.86 88.9))
-    (stroke (width 0) (type default) (color 0 0 0 0))
-  )
-  (wire (pts (xy 134.62 93.98) (xy 149.86 93.98))
-    (stroke (width 0) (type default) (color 0 0 0 0))
-  )
-  (symbol (lib_id "1-84952-5:1-84952-5") (at 175.26 86.36 0) (mirror y) (unit 1)
+  (symbol (lib_id "1-84952-5:1-84952-5") (at 160.02 121.92 180) (unit 1)
     (in_bom yes) (on_board yes) (fields_autoplaced)
-    (property "Reference" "J2" (id 0) (at 162.56 78.74 0))
-    (property "Value" "1-84952-5" (id 1) (at 162.56 81.28 0))
-    (property "Footprint" "pretty:1849525" (id 2) (at 153.67 83.82 0)
+    (property "Reference" "J2" (id 0) (at 147.32 78.74 0))
+    (property "Value" "1-84952-5" (id 1) (at 147.32 81.28 0))
+    (property "Footprint" "pretty:1849525" (id 2) (at 138.43 124.46 0)
       (effects (font (size 1.27 1.27)) (justify left) hide)
     )
-    (property "Datasheet" "https://datasheet.datasheetarchive.com/originals/distributors/Datasheets_SAMA/2b17d88214b230a9ac6dbaafb3962f09.pdf" (id 3) (at 153.67 86.36 0)
+    (property "Datasheet" "https://datasheet.datasheetarchive.com/originals/distributors/Datasheets_SAMA/2b17d88214b230a9ac6dbaafb3962f09.pdf" (id 3) (at 138.43 121.92 0)
       (effects (font (size 1.27 1.27)) (justify left) hide)
     )
-    (property "Description" "FFC & FPC Connectors 15P 1MM FPC Horz Bottom Cont. Assy" (id 4) (at 153.67 88.9 0)
+    (property "Description" "FFC & FPC Connectors 15P 1MM FPC Horz Bottom Cont. Assy" (id 4) (at 138.43 119.38 0)
       (effects (font (size 1.27 1.27)) (justify left) hide)
     )
-    (property "Height" "2.56" (id 5) (at 153.67 91.44 0)
+    (property "Height" "2.56" (id 5) (at 138.43 116.84 0)
       (effects (font (size 1.27 1.27)) (justify left) hide)
     )
-    (property "Mouser Part Number" "571-1-84952-5" (id 6) (at 153.67 93.98 0)
+    (property "Mouser Part Number" "571-1-84952-5" (id 6) (at 138.43 114.3 0)
       (effects (font (size 1.27 1.27)) (justify left) hide)
     )
-    (property "Mouser Price/Stock" "https://www.mouser.co.uk/ProductDetail/TE-Connectivity/1-84952-5/?qs=uUkeXfjQ8uTcXVIsXQkRfw%3D%3D" (id 7) (at 153.67 96.52 0)
+    (property "Mouser Price/Stock" "https://www.mouser.co.uk/ProductDetail/TE-Connectivity/1-84952-5/?qs=uUkeXfjQ8uTcXVIsXQkRfw%3D%3D" (id 7) (at 138.43 111.76 0)
       (effects (font (size 1.27 1.27)) (justify left) hide)
     )
-    (property "Manufacturer_Name" "TE Connectivity" (id 8) (at 153.67 99.06 0)
+    (property "Manufacturer_Name" "TE Connectivity" (id 8) (at 138.43 109.22 0)
       (effects (font (size 1.27 1.27)) (justify left) hide)
     )
-    (property "Manufacturer_Part_Number" "1-84952-5" (id 9) (at 153.67 101.6 0)
+    (property "Manufacturer_Part_Number" "1-84952-5" (id 9) (at 138.43 106.68 0)
       (effects (font (size 1.27 1.27)) (justify left) hide)
     )
