File: adaptor/adaptor.kicad_pcb (KiCad board)
At the start: 2 copper layers, 37.6 x 23.6 mm, 7 parts, among them J1 1-84952-5, J2 1-84952-5

Commit message: adaptor + some design wrork
Parts:
- J2: moved to F.Cu
- turned J2 to 180 degrees
Connections:
- J2 pad 1: Net-(J1-Pad1) -> Net-(J1-Pad15)
- J2 pad 10: Net-(J1-Pad10) -> Net-(J1-Pad6)
- J2 pad 11: Net-(J1-Pad11) -> Net-(J1-Pad5)
- J2 pad 12: Net-(J1-Pad12) -> Net-(J1-Pad4)
- J2 pad 13: Net-(J1-Pad13) -> Net-(J1-Pad3)
- J2 pad 14: Net-(J1-Pad14) -> Net-(J1-Pad2)
- J2 pad 15: Net-(J1-Pad15) -> Net-(J1-Pad1)
- J2 pad 2: Net-(J1-Pad2) -> Net-(J1-Pad14)
- J2 pad 3: Net-(J1-Pad3) -> Net-(J1-Pad13)
- J2 pad 4: Net-(J1-Pad4) -> Net-(J1-Pad12)
- J2 pad 5: Net-(J1-Pad5) -> Net-(J1-Pad11)
- J2 pad 6: Net-(J1-Pad6) -> Net-(J1-Pad10)
- J2 pad 7: Net-(J1-Pad7) -> Net-(J1-Pad9)
- J2 pad 9: Net-(J1-Pad9) -> Net-(J1-Pad7)
Routing:
- net Net-(J1-Pad9): vias 1 -> 0
- net Net-(J1-Pad8): vias 1 -> 0
- net Net-(J1-Pad7): vias 1 -> 0
- net Net-(J1-Pad6): vias 1 -> 0
- net Net-(J1-Pad5): vias 1 -> 0
- net Net-(J1-Pad4): vias 1 -> 0
- net Net-(J1-Pad3): vias 1 -> 0
- net Net-(J1-Pad2): vias 1 -> 0
- net Net-(J1-Pad15): vias 1 -> 0
- net Net-(J1-Pad14): vias 1 -> 0
- net Net-(J1-Pad13): vias 1 -> 0
- net Net-(J1-Pad12): vias 1 -> 0
- net Net-(J1-Pad11): vias 1 -> 0
- net Net-(J1-Pad10): vias 1 -> 0
- net Net-(J1-Pad1): vias 1 -> 0

Commit message: model & add break off board tommorow
Parts:
- removed the REF** at (126.7, 114.0)
- moved REF** 5.33 mm to (142.0, 112.3)
- moved REF** 5.33 mm to (111.5, 112.3)
- moved J1 2.79 mm to (126.7, 112.5)
- moved REF** 1.78 mm to (142.0, 102.4)
- moved REF** 1.78 mm to (111.5, 102.4)
- moved J2 0.76 mm to (126.7, 102.1)
Routing:
- net Net-(J1-Pad9): track 5.15 -> 3.37 mm
- net Net-(J1-Pad8): track 5.15 -> 3.37 mm
- net Net-(J1-Pad7): track 5.15 -> 3.37 mm
- net Net-(J1-Pad6): track 5.15 -> 3.37 mm
- net Net-(J1-Pad5): track 5.15 -> 3.37 mm
- net Net-(J1-Pad4): track 5.15 -> 3.37 mm
- net Net-(J1-Pad3): track 5.15 -> 3.37 mm
- net Net-(J1-Pad2): track 5.15 -> 3.37 mm
- net Net-(J1-Pad15): track 5.15 -> 3.37 mm
- net Net-(J1-Pad14): track 5.15 -> 3.37 mm
- net Net-(J1-Pad13): track 5.15 -> 3.37 mm
- net Net-(J1-Pad12): track 5.15 -> 3.37 mm
- net Net-(J1-Pad11): track 5.15 -> 3.37 mm
- net Net-(J1-Pad10): track 5.15 -> 3.37 mm
- net Net-(J1-Pad1): track 5.15 -> 3.37 mm
Other:
- board size 37.6 x 23.6 mm -> 37.6 x 16.5 mm
