File: CM4Carrier/heiarchy/io.kicad_sch (KiCad schematic)
At the start: 2 parts

Commit message: aa
Connections:
- net GND: now reaches Module?.1 (GND)
- net GND: now also Module?.13 (GND), Module?.14 (GND), Module?.2 (GND), Module?.22 (GND), Module?.23 (GND), Module?.32 (GND), Module?.33 (GND), Module?.42 (GND), Module?.43 (GND), Module?.52 (GND), Module?.53 (GND), Module?.59 (GND), Module?.60 (GND), Module?.65 (GND), Module?.66 (GND), Module?.7 (GND), Module?.71 (GND), Module?.74 (GND), Module?.8 (GND), Module?.98 (GND)
- net _5v: now reaches Module?.77 (+5v_(Input))
- net _5v: now also Module?.79 (+5v_(Input)), Module?.81 (+5v_(Input)), Module?.83 (+5v_(Input)), Module?.85 (+5v_(Input)), Module?.87 (+5v_(Input))
- net 3v3: now reaches Module?.78 (GPIO_VREF(1.8v/3.3v_Input))
- net 3v3: now also Module?.84 (+3.3v_(Output)), Module?.86 (+3.3v_(Output))
- net 1v8: now reaches Module?.88 (+1.8v_(Output))
- net 1v8: now also Module?.90 (+1.8v_(Output))
Other:
- moved on the sheet: Module?B

Commit message: kjkl
Parts:
- gave numbers to parts that had none: 1
Changed lines of the file:
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@@
   (symbol (lib_id "power:GND") (at 93.98 162.56 0) (unit 1)
     (in_bom yes) (on_board yes) (fields_autoplaced)
-    (property "Reference" "#PWR?" (id 0) (at 93.98 168.91 0)
+    (property "Reference" "#PWR02" (id 0) (at 93.98 168.91 0)
       (effects (font (size 1.27 1.27)) hide)
     )
@@
   (symbol (lib_id "power:GND") (at 22.86 162.56 0) (unit 1)
     (in_bom yes) (on_board yes) (fields_autoplaced)
-    (property "Reference" "#PWR?" (id 0) (at 22.86 168.91 0)
+    (property "Reference" "#PWR01" (id 0) (at 22.86 168.91 0)
       (effects (font (size 1.27 1.27)) hide)
     )
@@
   (symbol (lib_id "CM4IO:ComputeModule4-CM4") (at 60.96 91.44 0) (unit 1)
     (in_bom yes) (on_board yes) (fields_autoplaced)
-    (property "Reference" "Module?" (id 0) (at 58.42 22.86 0))
+    (property "Reference" "Module1" (id 0) (at 58.42 22.86 0))
     (property "Value" "ComputeModule4-CM4" (id 1) (at 58.42 25.4 0))
     (property "Footprint" "CM4IO:Raspberry-Pi-4-Compute-Module" (id 2) (at 203.2 118.11 0)
@@
   (symbol (lib_id "CM4IO:ComputeModule4-CM4") (at 63.5 91.44 0) (unit 2)
     (in_bom yes) (on_board yes) (fields_autoplaced)
-    (property "Reference" "Module?" (id 0) (at 203.2 17.145 0))
+    (property "Reference" "Module1" (id 0) (at 203.2 17.145 0))
     (property "Value" "ComputeModule4-CM4" (id 1) (at 203.2 19.685 0))
     (property "Footprint" "CM4IO:Raspberry-Pi-4-Compute-Module" (id 2) (at 205.74 118.11 0)

Commit message: aaa
Parts:
- added J?: Micro_SD_Card, symbol Connector:Micro_SD_Card
- added R?: 10M, symbol Device:R
Connections:
- net GND: now also R?.2
- net SD_DAT3: now reaches Module1.61 (SD_DAT3)
- net SD_DAT3: now also J?.2 (DAT3/CD)
- net SD_DAT0: now reaches Module1.63 (SD_DAT0)
- net SD_DAT0: now also J?.7 (DAT0)
- net SD_DAT1: now reaches Module1.67 (SD_DAT1)
- net SD_DAT1: now also J?.8 (DAT1)
- net SD_DAT2: now reaches Module1.69 (SD_DAT2)
- net SD_DAT2: now also J?.1 (DAT2)
- new net: J?.9 (SHIELD), R?.1
Other:
- moved on the sheet: Module1A
