File: CM4Carrier/heiarchy/io.kicad_sch (KiCad schematic)
At the start: 10 parts, among them J1 Micro_SD_Card, U1 MIC2025-2YMM

Commit message: pcb babeee les goooo
Parts:
- D1: footprint (none) -> LED_SMD:LED_0805_2012Metric_Pad1.15x1.40mm_HandSolder; Field4 (none) -> https://www.mouser.co.uk/ProductDetail/Wurth-Elektronik/150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
- R1: footprint (none) -> Resistor_SMD:R_0805_2012Metric_Pad1.20x1.40mm_HandSolder
- TP1: footprint (none) -> TestPoint:TestPoint_THTPad_1.0x1.0mm_Drill0.5mm
Connections:
- net FUEL_ALRT: now reaches Module1.54 (GPIO4)
- net FUEL_SDA: now reaches Module1.80 (SCL0)
- net FUEL_SCLK: now reaches Module1.82 (SDA0)
- no-connect marks 7 -> 41
Changed lines of the file:
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@@
   (title_block
     (rev "indev.")
+    (comment 1 "https://github.com/cinnamondev/gamepithing")
   )
   (junction (at 111.76 102.87) (diameter 0) (color 0 0 0 0)
@@
   (no_connect (at 251.46 35.56))
   (no_connect (at 106.68 153.67))
+  (no_connect (at 45.72 186.69))
+  (no_connect (at 45.72 181.61))
+  (no_connect (at 45.72 179.07))
+  (no_connect (at 45.72 176.53))
+  (no_connect (at 45.72 133.35))
+  (no_connect (at 45.72 130.81))
+  (no_connect (at 106.68 176.53))
+  (no_connect (at 106.68 173.99))
+  (no_connect (at 106.68 184.15))
+  (no_connect (at 106.68 64.77))
+  (no_connect (at 106.68 67.31))
+  (no_connect (at 106.68 80.01))
+  (no_connect (at 106.68 74.93))
+  (no_connect (at 106.68 72.39))
+  (no_connect (at 106.68 85.09))
+  (no_connect (at 106.68 82.55))
+  (no_connect (at 106.68 105.41))
+  (no_connect (at 106.68 179.07))
+  (no_connect (at 45.72 105.41))
+  (no_connect (at 45.72 95.25))
+  (no_connect (at 45.72 97.79))
+  (no_connect (at 45.72 102.87))
+  (no_connect (at 45.72 64.77))
+  (no_connect (at 45.72 67.31))
+  (no_connect (at 45.72 72.39))
+  (no_connect (at 45.72 74.93))
+  (no_connect (at 45.72 80.01))
+  (no_connect (at 45.72 82.55))
+  (no_connect (at 45.72 85.09))
+  (no_connect (at 45.72 90.17))
+  (no_connect (at 45.72 92.71))
+  (no_connect (at 45.72 118.11))
+  (no_connect (at 45.72 120.65))
+  (no_connect (at 45.72 123.19))
   (wire (pts (xy 124.46 87.63) (xy 106.68 87.63))
     (stroke (width 0) (type default) (color 0 0 0 0))
@@
     (stroke (width 0) (type default) (color 0 0 0 0))
   )
+  (wire (pts (xy 29.21 128.27) (xy 45.72 128.27))
+    (stroke (width 0) (type default) (color 0 0 0 0))
+  )
   (wire (pts (xy 40.64 113.03) (xy 40.64 125.73))
     (stroke (width 0) (type default) (color 0 0 0 0))
@@
     (stroke (width 0) (type default) (color 0 0 0 0))
   )
+  (wire (pts (xy 29.21 163.83) (xy 45.72 163.83))
+    (stroke (width 0) (type default) (color 0 0 0 0))
+  )
   (wire (pts (xy 142.24 27.94) (xy 149.86 27.94))
     (stroke (width 0) (type solid) (color 0 0 0 0))
@@
   )
   (wire (pts (xy 218.44 48.26) (xy 220.98 48.26))
+    (stroke (width 0) (type default) (color 0 0 0 0))
+  )
+  (wire (pts (xy 29.21 161.29) (xy 45.72 161.29))
     (stroke (width 0) (type default) (color 0 0 0 0))
   )
@@
     (effects (font (size 1.27 1.27)) (justify right bottom))
   )
+  (label "I2C_SDA" (at 30.48 161.29 0)
+    (effects (font (size 1.27 1.27)) (justify left bottom))
+  )
   (label "SD_CLK" (at 154.94 35.56 0)
+    (effects (font (size 1.27 1.27)) (justify left bottom))
+  )
+  (label "I2C_SCLK" (at 30.48 163.83 0)
     (effects (font (size 1.27 1.27)) (justify left bottom))
   )
@@
     (effects (font (size 1.27 1.27)) (justify right))
   )
+  (hierarchical_label "FUEL_SDA" (shape bidirectional) (at 29.21 161.29 180)
+    (effects (font (size 1.27 1.27)) (justify right))
+  )
   (hierarchical_label "B" (shape input) (at 113.03 130.81 0)
     (effects (font (size 1.27 1.27)) (justify left))
@@
   )
   (hierarchical_label "IO_VREF" (shape output) (at 34.29 158.75 180)
+    (effects (font (size 1.27 1.27)) (justify right))
+  )
+  (hierarchical_label "FUEL_ALRT" (shape input) (at 29.21 128.27 180)
+    (effects (font (size 1.27 1.27)) (justify right))
+  )
+  (hierarchical_label "FUEL_SCLK" (shape bidirectional) (at 29.21 163.83 180)
     (effects (font (size 1.27 1.27)) (justify right))
   )
@@
   (symbol (lib_id "power:GND") (at 142.24 39.37 0) (unit 1)
     (in_bom yes) (on_board yes)
-    (property "Reference" "#PWR0103" (id 0) (at 142.24 45.72 0)
+    (property "Reference" "#PWR03" (id 0) (at 142.24 45.72 0)
       (effects (font (size 1.27 1.27)) hide)
     )
@@
   (symbol (lib_id "power:GND") (at 261.62 41.91 0) (unit 1)
     (in_bom yes) (on_board yes) (fields_autoplaced)
-    (property "Reference" "#PWR0105" (id 0) (at 261.62 48.26 0)
+    (property "Reference" "#PWR05" (id 0) (at 261.62 48.26 0)
       (effects (font (size 1.27 1.27)) hide)
     )
@@
       (effects (font (size 1.27 1.27)) (justify left))
     )
-    (property "Footprint" "" (id 2) (at 116.84 186.69 0)
+    (property "Footprint" "TestPoint:TestPoint_THTPad_1.0x1.0mm_Drill0.5mm" (id 2) (at 116.84 186.69 0)
       (effects (font (size 1.27 1.27)) hide)
     )
@@
   (symbol (lib_id "power:GND") (at 111.76 189.23 0) (unit 1)
     (in_bom yes) (on_board yes) (fields_autoplaced)
-    (property "Reference" "#PWR0101" (id 0) (at 111.76 195.58 0)
+    (property "Reference" "#PWR02" (id 0) (at 111.76 195.58 0)
       (effects (font (size 1.27 1.27)) hide)
     )
@@
       (effects (font (size 1.27 1.27)) (justify right))
     )
-    (property "Footprint" "" (id 2) (at 124.46 72.39 0)
+    (property "Footprint" "LED_SMD:LED_0805_2012Metric_Pad1.15x1.40mm_HandSolder" (id 2) (at 124.46 72.39 0)
       (effects (font (size 1.27 1.27)) hide)
     )
@@
       (effects (font (size 1.27 1.27)) hide)
     )
+    (property "Field4" "https://www.mouser.co.uk/ProductDetail/Wurth-Elektronik/150080GS75000?qs=2kOmHSv6VfQRoTEZVk1mGA%3D%3D" (id 4) (at 124.46 72.39 90)
+      (effects (font (size 1.27 1.27)) hide)
+    )
     (pin "1")
     (pin "2")
@@
   (symbol (lib_id "power:GND") (at 40.64 189.23 0) (unit 1)
     (in_bom yes) (on_board yes) (fields_autoplaced)
-    (property "Reference" "#PWR0102" (id 0) (at 40.64 195.58 0)
+    (property "Reference" "#PWR01" (id 0) (at 40.64 195.58 0)
       (effects (font (size 1.27 1.27)) hide)
     )
@@
       (effects (font (size 1.27 1.27)) (justify left))
     )
-    (property "Footprint" "" (id 2) (at 122.682 82.55 90)
+    (property "Footprint" "Resistor_SMD:R_0805_2012Metric_Pad1.20x1.40mm_HandSolder" (id 2) (at 122.682 82.55 90)
       (effects (font (size 1.27 1.27)) hide)
     )
@@
   (symbol (lib_id "power:GND") (at 220.98 49.53 0) (unit 1)
     (in_bom yes) (on_board yes)
-    (property "Reference" "#PWR0104" (id 0) (at 220.98 55.88 0)
-      (effects (font (size 1.27 1.27)) hide)
-    )
+    (property "Reference" "#PWR04" (id 0) (at 220.98 55.88 0)
+      (effects (font (size 1.27 1.27)) hide)
+    )

Commit message: LAYOUT DONE!!
:)
Parts:
- added C27, C28, C29, C30: (no value), symbol Device:C
- added D4: (no value), symbol Diode:BAV99S
- added J6: AudioJack3_Dual_Ground_Switch, Connector_Audio:Jack_3.5mm_CUI_SJ-3524-SMT_Horizontal, symbol Connector:AudioJack3_Dual_Ground_Switch
- added R39, R40, R41, R42: (no value), symbol Device:R
Connections:
- net GND: now also C27.2, C28.2, C29.2, C30.2, D4.1 (A1), D4.4 (A3), J6.S
- net IO_VREF: now also D4.2 (K2), D4.5 (K4)
- net AUX_L: now reaches Module1.46 (GPIO22)
- net AUX_L: now also R40.2
- net AUX_R: now reaches Module1.48 (GPIO27)
- net AUX_R: now also R39.2
- new net: C29.1, D4.3 (K1A2), J6.R, R41.1
- new net: C27.1, R39.1, R41.2
- new net: C30.1, D4.6 (K3A4), J6.T, R42.1
- new net: C28.1, R40.1, R42.2
- no-connect marks 41 -> 39
Other:
- note added: "pretty much 100% from the original pi. later revisions could improve on this!"
