File: CM4Carrier/heiarchy/battery.kicad_sch (KiCad schematic)
At the start: 1 part

Commit message: aa
Connections:
- net GNDPWR: now reaches U?.18 (PGND)
- net GNDPWR: now also U?.19 (PGND)
- net GND: now reaches U?.9 (GND)
Other:
- note added: "511-STEF05PUR Integrate for EFUSE CURRENT PROTECTION!!"
- note added: "Switching start/reboot circuit Initial state: GLOBAL_EN high"
Changed lines of the file:
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@@
 (kicad_sch (version 20211123) (generator eeschema)
   (paper "A4")
+  (junction (at 191.77 146.05) (diameter 0) (color 0 0 0 0)
+  )
   (junction (at 172.72 100.33) (diameter 0) (color 0 0 0 0)
   )
@@
     (stroke (width 0) (type default) (color 0 0 0 0))
   )
+  (wire (pts (xy 185.42 147.32) (xy 185.42 146.05))
+    (stroke (width 0) (type default) (color 0 0 0 0))
+  )
+  (wire (pts (xy 185.42 146.05) (xy 186.69 146.05))
+    (stroke (width 0) (type default) (color 0 0 0 0))
+  )
   (wire (pts (xy 173.99 102.87) (xy 172.72 102.87))
+    (stroke (width 0) (type default) (color 0 0 0 0))
+  )
+  (wire (pts (xy 193.04 146.05) (xy 193.04 147.32))
     (stroke (width 0) (type default) (color 0 0 0 0))
   )
@@
     (stroke (width 0) (type default) (color 0 0 0 0))
   )
+  (wire (pts (xy 189.23 146.05) (xy 191.77 146.05))
+    (stroke (width 0) (type default) (color 0 0 0 0))
+  )
   (wire (pts (xy 170.18 100.33) (xy 172.72 100.33))
     (stroke (width 0) (type default) (color 0 0 0 0))
+  )
+  (wire (pts (xy 191.77 146.05) (xy 193.04 146.05))
+    (stroke (width 0) (type default) (color 0 0 0 0))
+  )
+  (text "Switching start/reboot circuit\nInitial state: GLOBAL_EN high"
+    (at 66.04 27.94 0)
+    (effects (font (size 1.27 1.27)) (justify left bottom))
+  )
+  (text "511-STEF05PUR\n\nIntegrate for EFUSE CURRENT PROTECTION!!"
+    (at 40.64 55.88 0)
+    (effects (font (size 1.27 1.27)) (justify left bottom))
   )
   (hierarchical_label "CHRG-CC1" (shape bidirectional) (at 173.99 119.38 180)
@@
   (hierarchical_label "CHRG-D+" (shape bidirectional) (at 173.99 110.49 180)
     (effects (font (size 1.27 1.27)) (justify right))
+  )
+  (hierarchical_label "_5v" (shape output) (at 119.38 73.66 0)
+    (effects (font (size 1.27 1.27)) (justify left))
   )
   (symbol (lib_id "CM4IO:MAX77751") (at 189.23 96.52 0) (unit 1)
@@
     (pin "9")
   )
+  (symbol (lib_id "power:GNDPWR") (at 193.04 147.32 0) (unit 1)
+    (in_bom yes) (on_board yes) (fields_autoplaced)
+    (property "Reference" "#PWR?" (id 0) (at 193.04 152.4 0)
+      (effects (font (size 1.27 1.27)) hide)
+    )
+    (property "Value" "GNDPWR" (id 1) (at 192.913 152.4 0))
+    (property "Footprint" "" (id 2) (at 193.04 148.59 0)
+      (effects (font (size 1.27 1.27)) hide)
+    )
+    (property "Datasheet" "" (id 3) (at 193.04 148.59 0)
+      (effects (font (size 1.27 1.27)) hide)
+    )
+    (pin "1")
+  )
+  (symbol (lib_id "power:GND") (at 185.42 147.32 0) (unit 1)
+    (in_bom yes) (on_board yes) (fields_autoplaced)
+    (property "Reference" "#PWR?" (id 0) (at 185.42 153.67 0)
+      (effects (font (size 1.27 1.27)) hide)
+    )
+    (property "Value" "GND" (id 1) (at 185.42 152.4 0))
+    (property "Footprint" "" (id 2) (at 185.42 147.32 0)
+      (effects (font (size 1.27 1.27)) hide)
+    )
+    (property "Datasheet" "" (id 3) (at 185.42 147.32 0)
+      (effects (font (size 1.27 1.27)) hide)
+    )
+    (pin "1")
+  )
 )

Commit message: kjkl
Parts:
- added BT1: Battery_Cell, symbol Device:Battery_Cell
- added C1, C2, C4, C5, C6, C7, C8: C, symbol Device:C
- added C3: 100n, symbol Device:C
- added D1, D2: LED, symbol Device:LED
- added L1: 1, symbol Device:L
- added R1, R2, R3, R4: R, symbol Device:R
- gave numbers to parts that had none: 1
Connections:
- net CHRG-VBUS: now also C2.1
- net GND: now also U1.8 (ENBST), BT1.2 (-), C1.2, C2.2, C4.2, C5.2, C6.2, C7.2, R3.2, R4.2; no longer U1.9 (GND)
- net at U1.1 (BST): now also C3.1
- net at U1.10 (VDD): now also C1.1
- net at U1.11 (ITOPOFF): now also R4.1
- net at U1.12 (IFAST): now also R3.1
- net at U1.13 (BATT): now also U1.14 (BATT), BT1.1 (+), C6.1
- net BATT_SYS: now reaches U1.15 (SYS)
- net BATT_SYS: now also U1.16 (SYS), C5.1, C7.1, L1.2
- net at U1.17 (PVL): now also C4.1
- net at U1.2 (INOKB): now also R1.2
- net at U1.20 (LX): now also U1.21 (LX), C3.2, L1.1
- net at U1.22 (BYP): now also C8.1
- net at U1.3 (STAT): now also R2.2
- net GNDPWR: no longer names the net of U1.18 (PGND), U1.19 (PGND)
- net GNDPWR: now also U1.9 (GND)
- new net: D1.1 (K), R2.1
- new net: D2.1 (K), R1.1
Other:
- note added: "INOKB high when invalid power"
- note added: "stat flicker during charge off when done high when fault"

Commit message: aaa
Parts:
- added C? (x5): C, symbol Device:C
- added L?: L, symbol Device:L
- added R? (x5): R, symbol Device:R
- added U?: MP3424, CM4IO:MP3424GGP, symbol CM4IO:MP3424
Connections:
- net BATT_SYS: now also D1.2 (A), D2.2 (A), C?.1, C?.1, L?.1, U?.8 (IN)
- net GND: now also C8.2, C?.2, C?.2, C?.2, C?.2, R?.2, R?.2, R?.2, U?.10 (AGND), U?.13 (PGND), U?.2 (PGND)
- net _5v: now also R?.2, U?.1 (SENSE)
- new net: C?.1, R?.1, U?.9 (ILIM)
- new net: C?.2, R?.1
- new net: C?.1, C?.1, R?.1, R?.1, U?.12 (SOUT), U?.4 (OUT), U?.5 (OUT), U?.6 (OUT)
- new net: R?.1, R?.2, U?.11 (FB)
- new net: L?.2, U?.14 (SW), U?.3 (SW)
- new net EN: U?.7 (EN)
Other:
- moved on the sheet: BT1, C1, C2, C3, C4, C5, C6, C7, C8, D1, D2, L1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

Commit message: footprints  + values
need to do some 3d babeeeeeeeeee
Parts:
- removed C? (x3): C, symbol Device:C
- removed R? (x3): R, symbol Device:R
- added R? (x2): (no value), symbol Device:R
- added TP?: (no value), symbol Connector:TestPoint_2Pole
- C? (x2): value C -> (none)
- C?: renamed from C5; value C -> (none)
- C?: renamed from C7; value C -> (none)
- L?: renamed from L1; value 1 -> (none)
- L?: value L -> (none)
- R? (x2): value R -> (none)
- renumbered BT1 to BT?, C6 to C?, C8 to C?, C1 to C?, C2 to C?, C4 to C?, C3 to C?, D1 to D?, D2 to D?, R4 to R?, R3 to R?, R2 to R?, R1 to R?, U1 to U?
Connections:
- net BATT_SYS: now also R?.1
- net GND: now also R?.2, TP?.1
- net _5v: now also C?.1, C?.1, R?.1, U?.12 (SOUT), U?.4 (OUT), U?.5 (OUT), U?.6 (OUT), TP?.2
- net EN: no longer names the net of U?.7 (EN)
- net EN: now also R?.1, R?.2
Other:
- note added: "EN can be used for UVLO. UVLO is 2.4v"
- note added: "No current limiting needed..."
- note added: "Page 15 Overload and SCP"
- title: (none) -> Battery / Power

Commit message: aa
Parts:
- removed C? (x2): (no value), symbol Device:C
- added C? (x7): (no value), symbol Device:C
- added D?: (no value), symbol Device:D_Schottky
- added L?: (no value), symbol Device:L
- added R?: (no value), symbol Device:R
- added U?: (no value), symbol CM4IO:MIC2877
- added U?: (no value), symbol CM4IO:MAX1709
- C? (x2): value (none) -> 22u
- L?: value (none) -> 1uH
- L?: value (none) -> 1.6uH
- R?: value (none) -> 453k
- R?: value (none) -> 86.6k
- R? (x2): value (none) -> 100k
- TP?: value (none) -> +5v; footprint (none) -> TestPoint:TestPoint_Bridge_Pitch5.08mm_Drill1.3mm
Connections:
- net BATT_SYS: now also C?.1, C?.1, L?.1
- net GND: now also C?.1, C?.2, C?.2, C?.2, C?.2, C?.2, C?.2, U?.11 (GND), U?.14 (GND)
- new net: C?.1, C?.1, D?.1 (K), R?.2
- new net: C?.2, R?.1, U?.15 (OUT)
- new net: C?.1, U?.12 (SS/LM) (x2)
- new net LX: D?.2 (A), L?.2, U?.2 (LX), U?.3 (LX), U?.4 (LX), U?.5 (LX), U?.6 (LX), U?.7 (LX), U?.8 (LX)
- new net PGND: U?.18 (PGND), U?.19 (PGND), U?.20 (PGND), U?.21 (PGND), U?.22 (PGND), U?.23 (PGND)

Commit message: commit
Parts:
- removed C? (x7): (no value), symbol Device:C
- removed C? (x2): 22u, symbol Device:C
- removed D?: (no value), symbol Device:D_Schottky
- removed L?: 1.6uH, symbol Device:L
- removed L?: (no value), symbol Device:L
- removed R?: (no value), symbol Device:R
- removed R?: 453k, symbol Device:R
- removed R?: 86.6k, symbol Device:R
- removed R? (x2): 100k, symbol Device:R
- removed TP?: +5v, TestPoint:TestPoint_Bridge_Pitch5.08mm_Drill1.3mm, symbol Connector:TestPoint_2Pole
- removed U?: MP3424, CM4IO:MP3424GGP, symbol CM4IO:MP3424
- removed U?: (no value), symbol CM4IO:MAX1709
- added C? (x4): (no value), symbol Device:C
- added L?: (no value), symbol Device:L
- added R?: (no value), symbol Device:R
- added TP? (x2): (no value), symbol Connector:TestPoint_Flag
Connections:
- net BATT_SYS: now also U?.1 (VIN), C?.1, C?.1, L?.1, R?.1
- net GND: now also U?.2 (AGND), U?.3 (PGND), C?.2, C?.2, C?.2, C?.2
- net _5v: now also U?.5 (VOUT), U?.7 (VOUTS), C?.1, C?.1, TP?.1
- net at U?.4 (SW): now also L?.2
- net at U?.8 (PG): now also R?.2, TP?.1
Other:
- note added: "Batt --> 5v BOOST"
- note added: "Battery charger"
- note added: "TBD: BATTERY MONITOR!!!"
- note removed: "EN can be used for UVLO. UVLO is 2.4v"
- note removed: "No current limiting needed..."
- note removed: "Page 15 Overload and SCP"
- moved on the sheet: U?

Commit message: pcb next :sunglasses:
Parts:
- added C10: (no value), symbol Device:C
- added C5: C, symbol Device:C
- added R10, R8, R9: (no value), symbol Device:R
- added TH1: (no value), symbol Device:Thermistor_NTC
- added U3: (no value), symbol Battery_Management:MAX17261xxTD
- C11, C12, C13, C9: renamed from C?; value (none) -> 22u
- C2, C3, C6, C8: renamed from C?; value C -> (none)
- L1: renamed from L?; value 1uH -> (none)
- L2: renamed from L?; value (none) -> 1u
- R11: renamed from R?; value (none) -> 1M
- R4, R5: renamed from R?; value R -> (none)
- TP3: renamed from TP?; value (none) -> TP_PG
- TP4: renamed from TP?; value (none) -> TestPoint_Flag
- U2: renamed from U?; value MAX77751 -> (none)
- gave numbers to parts that had none: 8
Connections:
- net GND: now also U2.18 (PGND), U2.19 (PGND), U2.9 (GND), C10.2, C5.2, R10.2, R8.1, R8.2, TH1.2, U3.15 (GND), U3.7 (CSN), U3.8 (GND), U3.9 (CSPL)
- net BATT: now reaches BT1.1 (+), C6.1, U2.13 (BATT), U2.14 (BATT)
- net BATT: now also R9.1, U3.6 (BATT)
- net at C7.1, U2.22 (BYP): now also C5.1
- new net: TH1.1, U3.1 (TH)
- new net: R10.1, R9.2, U3.10 (CELLX)
- new net: C10.1, U3.11 (REG)
- new net ALRT: U3.12 (ALRT)
- new net FUEL_SCL: U3.14 (SCL)
- new net FUEL_SDA: U3.13 (SDA)
Other:
- note added: "radio 6:4 output is 40pc"
- note added: "says to regulate but itsll be fine... hopefully"
- moved on the sheet: C8
