File: CM4Carrier/heiarchy/battery.kicad_sch (KiCad schematic)
At the start: 31 parts

Commit message: pcb babeee les goooo
Parts:
- added R12: 10k, Resistor_SMD:R_0805_2012Metric_Pad1.20x1.40mm_HandSolder, symbol Device:R
- added TP4: 5VREG_EN, TestPoint:TestPoint_THTPad_1.0x1.0mm_Drill0.5mm, symbol Connector:TestPoint_Alt
- BT1: footprint (none) -> Connector_JST:JST_XH_S2B-XH-A_1x02_P2.50mm_Horizontal
- C10: value (none) -> 470n
- C11, C12, C13, C4, C5, C7, C9: footprint (none) -> Capacitor_SMD:C_0805_2012Metric_Pad1.18x1.45mm_HandSolder
- C2, C3, C8: value (none) -> 2.2u; footprint (none) -> Capacitor_SMD:C_0805_2012Metric_Pad1.18x1.45mm_HandSolder
- C6: value (none) -> 22u; footprint (none) -> Capacitor_SMD:C_0805_2012Metric_Pad1.18x1.45mm_HandSolder
- D2, D3: footprint (none) -> LED_SMD:LED_0805_2012Metric_Pad1.15x1.40mm_HandSolder; Field4 (none) -> https://www.mouser.co.uk/ProductDetail/Wurth-Elektronik/150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
- L1: value (none) -> 0.47u; footprint (none) -> Inductor_SMD:L_1008_2520Metric_Pad1.43x2.20mm_HandSolder
- L2: footprint (none) -> Inductor_SMD:L_1008_2520Metric_Pad1.43x2.20mm_HandSolder
- R10: value (none) -> 400k
- R11, R6, R7: footprint (none) -> Resistor_SMD:R_0805_2012Metric_Pad1.20x1.40mm_HandSolder
- R4, R5: value (none) -> 1k; footprint (none) -> Resistor_SMD:R_0805_2012Metric_Pad1.20x1.40mm_HandSolder
- R8: value (none) -> R; footprint (none) -> Resistor_SMD:R_0805_2012Metric_Pad1.20x1.40mm_HandSolder
- R9: value (none) -> 600k
- TH1: value (none) -> 10k 5%; footprint (none) -> Resistor_SMD:R_0805_2012Metric_Pad1.20x1.40mm_HandSolder
- TP3: footprint (none) -> TestPoint:TestPoint_THTPad_1.0x1.0mm_Drill0.5mm
- TP5: renamed from TP4; footprint (none) -> TestPoint:TestPoint_THTPad_1.0x1.0mm_Drill0.5mm
- U2: value (none) -> MAX77751; footprint (none) -> CM4IO:IC_MAX77751FEFG+
- U3: value (none) -> MAX17261xxTD; footprint (none) -> Package_DFN_QFN:TDFN-14-1EP_3x3mm_P0.4mm_EP1.78x2.35mm
- U4: value (none) -> MIC2877; footprint (none) -> CM4IO:MIC2877-AYFT-TR
Connections:
- net BATT_SYS is gone; now on net BATT: C11.1, C9.1, D2.2 (A), D3.2 (A), L1.2, L2.1, R11.1, U2.15 (SYS), U2.16 (SYS), U4.1 (VIN)
- net BATT: now also R12.1
- net at U4.6 (EN): now also R12.2, TP4.1
- no-connect marks 0 -> 1

Commit message: foo
Parts:
- C10: footprint (none) -> Capacitor_SMD:C_0603_1608Metric_Pad1.08x0.95mm_HandSolder
- R10, R9: footprint (none) -> Resistor_SMD:R_0603_1608Metric_Pad0.98x0.95mm_HandSolder
Changed lines of the file:
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@@
+    (effects (font (size 1.27 1.27)) (justify left bottom))
+  )
+  (label "CSN" (at 139.7 124.46 0)
     (effects (font (size 1.27 1.27)) (justify left bottom))
   )
@@
       (effects (font (size 1.27 1.27)) (justify left))
     )
-    (property "Footprint" "" (id 2) (at 167.3352 133.35 0)
+    (property "Footprint" "Capacitor_SMD:C_0603_1608Metric_Pad1.08x0.95mm_HandSolder" (id 2) (at 167.3352 133.35 0)
       (effects (font (size 1.27 1.27)) hide)
     )
@@
       (effects (font (size 1.27 1.27)) (justify left))
     )
-    (property "Footprint" "" (id 2) (at 125.222 119.38 90)
+    (property "Footprint" "Resistor_SMD:R_0603_1608Metric_Pad0.98x0.95mm_HandSolder" (id 2) (at 125.222 119.38 90)
       (effects (font (size 1.27 1.27)) hide)
     )
@@
     (property "Reference" "R9" (id 0) (at 121.92 105.41 90))
     (property "Value" "600k" (id 1) (at 121.92 107.95 90))
-    (property "Footprint" "" (id 2) (at 121.92 113.538 90)
-      (effects (font (size 1.27 1.27)) hide)
-    )
+    (property "Footprint" "Resistor_SMD:R_0603_1608Metric_Pad0.98x0.95mm_HandSolder" (id 2) (at 121.92 113.538 90)
+      (effects (font (size 1.27 1.27)) hide)
+    )

Commit message: PCB work
Home-stretch! Remaining things:
- Forgot Headphone jack / audio in design - add.
- route power supply (aaaaa)
Parts:
- C8: value 2.2u -> (none); footprint Capacitor_SMD:C_0805_2012Metric_Pad1.18x1.45mm_HandSolder -> (none)
- R6, R7: value R -> (none); footprint Resistor_SMD:R_0805_2012Metric_Pad1.20x1.40mm_HandSolder -> (none)
Connections:
- net BATT: now also U2.13_14 (BATT), U2.15_16 (SYS); no longer U2.13 (BATT), U2.14 (BATT), U2.15 (SYS), U2.16 (SYS)
- net CHRG-VBUS: now also U2.23_24 (CHGIN); no longer U2.23 (CHGIN), U2.24 (CHGIN)
- net GND: now also U2.18_19 (PGND); no longer BT1.2 (-), R8.1, U2.18 (PGND), U2.19 (PGND), U3.9 (CSPL)
- net at C4.2, L1.1: now also U2.20_21 (LX); no longer U2.20 (LX), U2.21 (LX)
- new net: BT1.2 (-), R8.1, U3.9 (CSPL)
Other:
- moved on the sheet: U2
Changed lines of the file:
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@@
   (junction (at 175.26 72.39) (diameter 0) (color 0 0 0 0)
-  )
-  (junction (at 132.08 127) (diameter 0) (color 0 0 0 0)
   )
   (junction (at 53.34 39.37) (diameter 0) (color 0 0 0 0)
@@
     (stroke (width 0) (type default) (color 0 0 0 0))
   )
-  (wire (pts (xy 113.03 127) (xy 132.08 127))
+  (wire (pts (xy 113.03 127) (xy 143.51 127))
     (stroke (width 0) (type default) (color 0 0 0 0))
   )
@@
     (stroke (width 0) (type default) (color 0 0 0 0))
   )
-  (wire (pts (xy 132.08 127) (xy 132.08 132.08))
-    (stroke (width 0) (type default) (color 0 0 0 0))
-  )
   (wire (pts (xy 116.84 86.36) (xy 113.03 86.36))
     (stroke (width 0) (type default) (color 0 0 0 0))
@@
   )
   (wire (pts (xy 166.37 111.76) (xy 163.83 111.76))
-    (stroke (width 0) (type default) (color 0 0 0 0))
-  )
-  (wire (pts (xy 143.51 127) (xy 132.08 127))
     (stroke (width 0) (type default) (color 0 0 0 0))
   )
@@
     (pin "11")
     (pin "12")
-    (pin "13")
-    (pin "14")
-    (pin "15")
-    (pin "16")
+    (pin "13_14")
+    (pin "13_14")
+    (pin "15_16")
+    (pin "15_16")
     (pin "17")
-    (pin "18")
-    (pin "19")
-    (pin "2")
-    (pin "20")
-    (pin "21")
+    (pin "18_19")
+    (pin "18_19")
+    (pin "2")
+    (pin "20_21")
+    (pin "20_21")
     (pin "22")
-    (pin "23")
-    (pin "24")
+    (pin "23_24")
+    (pin "23_24")
     (pin "3")
     (pin "4")
@@
       (effects (font (size 1.27 1.27)) (justify left))
     )
-    (property "Value" "R" (id 1) (at 90.17 82.5499 0)
-      (effects (font (size 1.27 1.27)) (justify left))
-    )
-    (property "Footprint" "Resistor_SMD:R_0805_2012Metric_Pad1.20x1.40mm_HandSolder" (id 2) (at 85.852 81.28 90)
+    (property "Value" "" (id 1) (at 90.17 82.5499 0)
+      (effects (font (size 1.27 1.27)) (justify left))
+    )
+    (property "Footprint" "" (id 2) (at 85.852 81.28 90)
       (effects (font (size 1.27 1.27)) hide)
     )
@@
       (effects (font (size 1.27 1.27)) (justify left))
     )
-    (property "Value" "R" (id 1) (at 53.34 83.8199 0)
-      (effects (font (size 1.27 1.27)) (justify left))
-    )
-    (property "Footprint" "Resistor_SMD:R_0805_2012Metric_Pad1.20x1.40mm_HandSolder" (id 2) (at 49.022 82.55 90)
+    (property "Value" "" (id 1) (at 53.34 83.8199 0)
+      (effects (font (size 1.27 1.27)) (justify left))
+    )
+    (property "Footprint" "" (id 2) (at 49.022 82.55 90)
       (effects (font (size 1.27 1.27)) hide)
     )
@@
       (effects (font (size 1.27 1.27)) (justify left))
     )
-    (property "Value" "2.2u" (id 1) (at 130.81 67.3099 0)
-      (effects (font (size 1.27 1.27)) (justify left))
-    )
-    (property "Footprint" "Capacitor_SMD:C_0805_2012Metric_Pad1.18x1.45mm_HandSolder" (id 2) (at 127.9652 69.85 0)
-      (effects (font (size 1.27 1.27)) hide)
-    )
+    (property "Value" "" (id 1) (at 130.81 67.3099 0)
+      (effects (font (size 1.27 1.27)) (justify left))
+    )
+    (property "Footprint" "" (id 2) (at 127.9652 69.85 0)
+      (effects (font (size 1.27 1.27)) hide)
+    )

Commit message: LAYOUT DONE!!
:)
Parts:
- C8: value (none) -> 2.2u; footprint (none) -> Capacitor_SMD:C_0603_1608Metric_Pad1.08x0.95mm_HandSolder
- R6, R7: value (none) -> R; footprint (none) -> Resistor_SMD:R_0603_1608Metric_Pad0.98x0.95mm_HandSolder
Connections:
- net BATT renamed BATT_SYSTEM
- net BATT_SYSTEM: no longer BT1.1 (+), C6.1, R9.1, U2.13_14 (BATT), U3.6 (BATT)
- new net BATT__: BT1.1 (+), C6.1, R9.1, U2.13_14 (BATT), U3.6 (BATT)
Other:
- note added: "D2: Flashing during charge, solid when charged if low & d3 is lit, charger issue D3: Power good, solid on when charge present"
- note removed: "INOKB high when invalid power"
- note removed: "stat flicker during charge off when done high when fault"
Changed lines of the file:
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@@
     (effects (font (size 2.54 2.54)) (justify left bottom))
-  )
-  (text "stat flicker during charge\noff when done\nhigh when fault"
-    (at -19.05 12.7 0)
-    (effects (font (size 1.27 1.27)) (justify left bottom))
   )
   (text "Battery charger" (at 15.24 99.06 0)
@@
     (effects (font (size 1.27 1.27)) (justify left bottom))
   )
-  (text "INOKB high when invalid power \n" (at -22.86 5.08 0)
+  (text "D2:\nFlashing during charge, solid when charged\nif low & d3 is lit, charger issue\nD3:\nPower good, solid on when charge present\n"
+    (at 13.97 125.73 0)
     (effects (font (size 1.27 1.27)) (justify left bottom))
   )
@@
     (effects (font (size 1.27 1.27)) (justify right bottom))
   )
-  (label "BATT" (at 113.03 71.12 0)
+  (label "BATT__" (at 113.03 71.12 0)
     (effects (font (size 1.27 1.27)) (justify left bottom))
   )
@@
     (effects (font (size 1.27 1.27)) (justify left bottom))
   )
-  (label "BATT" (at 115.57 105.41 0)
+  (label "BATT__" (at 115.57 105.41 0)
     (effects (font (size 1.27 1.27)) (justify left bottom))
   )
@@
     (effects (font (size 1.27 1.27)) (justify right))
   )
-  (hierarchical_label "BATT" (shape output) (at 124.46 50.8 0)
+  (hierarchical_label "BATT_SYSTEM" (shape output) (at 124.46 50.8 0)
     (effects (font (size 1.27 1.27)) (justify left))
   )
@@
       (effects (font (size 1.27 1.27)) (justify left))
     )
-    (property "Value" "" (id 1) (at 90.17 82.5499 0)
-      (effects (font (size 1.27 1.27)) (justify left))
-    )
-    (property "Footprint" "" (id 2) (at 85.852 81.28 90)
+    (property "Value" "R" (id 1) (at 90.17 82.5499 0)
+      (effects (font (size 1.27 1.27)) (justify left))
+    )
+    (property "Footprint" "Resistor_SMD:R_0603_1608Metric_Pad0.98x0.95mm_HandSolder" (id 2) (at 85.852 81.28 90)
       (effects (font (size 1.27 1.27)) hide)
     )
@@
       (effects (font (size 1.27 1.27)) (justify left))
     )
-    (property "Value" "" (id 1) (at 53.34 83.8199 0)
-      (effects (font (size 1.27 1.27)) (justify left))
-    )
-    (property "Footprint" "" (id 2) (at 49.022 82.55 90)
+    (property "Value" "R" (id 1) (at 53.34 83.8199 0)
+      (effects (font (size 1.27 1.27)) (justify left))
+    )
+    (property "Footprint" "Resistor_SMD:R_0603_1608Metric_Pad0.98x0.95mm_HandSolder" (id 2) (at 49.022 82.55 90)
       (effects (font (size 1.27 1.27)) hide)
     )
@@
       (effects (font (size 1.27 1.27)) (justify left))
     )
-    (property "Value" "" (id 1) (at 130.81 67.3099 0)
-      (effects (font (size 1.27 1.27)) (justify left))
-    )
-    (property "Footprint" "" (id 2) (at 127.9652 69.85 0)
-      (effects (font (size 1.27 1.27)) hide)
-    )
+    (property "Value" "2.2u" (id 1) (at 130.81 67.3099 0)
+      (effects (font (size 1.27 1.27)) (justify left))
+    )
+    (property "Footprint" "Capacitor_SMD:C_0603_1608Metric_Pad1.08x0.95mm_HandSolder" (id 2) (at 127.9652 69.85 0)
+      (effects (font (size 1.27 1.27)) hide)
+    )
