File: CM4Carrier/heiarchy/buttons.kicad_sch (KiCad schematic)
At the start: 73 parts

Commit message: aa
Parts:
- TP? (x3): value (none) -> A
- TP?: value (none) -> (A.B)' (0)
- TP?: value (none) -> U/D
- TP?: value (none) -> SEL
- TP?: value (none) -> X
- TP?: value (none) -> START
- TP? (x3): value (none) -> B
- TP?: value (none) -> (A.B)' (1)
- TP?: value (none) -> L/R
- TP?: value (none) -> R
- TP?: value (none) -> U
- TP?: value (none) -> L
- TP?: value (none) -> Y
- TP?: value (none) -> D
- U? (x2): value (none) -> 74HC00
Changed lines of the file:
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@@
       (effects (font (size 1.27 1.27)) (justify left))
     )
-    (property "Value" "" (id 1) (at 143.51 190.4999 0)
+    (property "Value" "A" (id 1) (at 143.51 190.4999 0)
       (effects (font (size 1.27 1.27)) (justify left))
     )
@@
       (effects (font (size 1.27 1.27)) (justify left))
     )
-    (property "Value" "" (id 1) (at 163.83 179.0699 0)
+    (property "Value" "(A.B)' (0)" (id 1) (at 163.83 179.0699 0)
       (effects (font (size 1.27 1.27)) (justify left))
     )
@@
       (effects (font (size 1.27 1.27)) (justify left))
     )
-    (property "Value" "" (id 1) (at 234.95 134.4929 0)
+    (property "Value" "U/D" (id 1) (at 234.95 134.4929 0)
       (effects (font (size 1.27 1.27)) (justify left))
     )
@@
       (effects (font (size 1.27 1.27)) (justify left))
     )
-    (property "Value" "" (id 1) (at 64.77 128.1429 0)
+    (property "Value" "SEL" (id 1) (at 64.77 128.1429 0)
       (effects (font (size 1.27 1.27)) (justify left) hide)
     )
@@
       (effects (font (size 1.27 1.27)) (justify left))
     )
-    (property "Value" "" (id 1) (at 219.71 46.8629 0)
+    (property "Value" "A" (id 1) (at 219.71 46.8629 0)
       (effects (font (size 1.27 1.27)) (justify left) hide)
     )
@@
       (effects (font (size 1.27 1.27)) (justify left))
     )
-    (property "Value" "" (id 1) (at 232.41 78.6129 0)
+    (property "Value" "X" (id 1) (at 232.41 78.6129 0)
       (effects (font (size 1.27 1.27)) (justify left) hide)
     )
@@
       (effects (font (size 1.27 1.27)) (justify left))
     )
-    (property "Value" "" (id 1) (at 114.3 129.4129 0)
+    (property "Value" "START" (id 1) (at 114.3 129.4129 0)
       (effects (font (size 1.27 1.27)) (justify left) hide)
     )
@@
       (effects (font (size 1.27 1.27)) (justify left))
     )
-    (property "Value" "" (id 1) (at 262.89 34.1629 0)
+    (property "Value" "B" (id 1) (at 262.89 34.1629 0)
       (effects (font (size 1.27 1.27)) (justify left) hide)
     )
@@
       (effects (font (size 1.27 1.27)) (justify left))
     )
-    (property "Value" "" (id 1) (at 143.51 181.6099 0)
+    (property "Value" "B" (id 1) (at 143.51 181.6099 0)
       (effects (font (size 1.27 1.27)) (justify left))
     )
@@
       (effects (font (size 1.27 1.27)) (justify left))
     )
-    (property "Value" "" (id 1) (at 143.51 195.5799 0)
+    (property "Value" "B" (id 1) (at 143.51 195.5799 0)
       (effects (font (size 1.27 1.27)) (justify left))
     )
@@
       (effects (font (size 1.27 1.27)) (justify left))
     )
-    (property "Value" "" (id 1) (at 163.83 193.0399 0)
+    (property "Value" "(A.B)' (1)" (id 1) (at 163.83 193.0399 0)
       (effects (font (size 1.27 1.27)) (justify left))
     )
@@
       (effects (font (size 1.27 1.27)) (justify left))
     )
-    (property "Value" "" (id 1) (at 236.22 124.3329 0)
+    (property "Value" "L/R" (id 1) (at 236.22 124.3329 0)
       (effects (font (size 1.27 1.27)) (justify left))
     )
@@
     (in_bom yes) (on_board yes) (fields_autoplaced)
     (property "Reference" "U?" (id 0) (at 152.4 182.88 0))
-    (property "Value" "" (id 1) (at 152.4 185.42 0))
+    (property "Value" "74HC00" (id 1) (at 152.4 185.42 0))
     (property "Footprint" "" (id 2) (at 152.4 191.77 0)
       (effects (font (size 1.27 1.27)) hide)
@@
       (effects (font (size 1.27 1.27)) (justify left))
     )
-    (property "Value" "" (id 1) (at 142.24 63.3729 0)
+    (property "Value" "R" (id 1) (at 142.24 63.3729 0)
       (effects (font (size 1.27 1.27)) (justify left) hide)
     )
@@
       (effects (font (size 1.27 1.27)) (justify left))
     )
-    (property "Value" "" (id 1) (at 104.14 41.7829 0)
+    (property "Value" "U" (id 1) (at 104.14 41.7829 0)
       (effects (font (size 1.27 1.27)) (justify left) hide)
     )
@@
       (effects (font (size 1.27 1.27)) (justify left))
     )
-    (property "Value" "" (id 1) (at 64.77 63.3729 0)
+    (property "Value" "L" (id 1) (at 64.77 63.3729 0)
       (effects (font (size 1.27 1.27)) (justify left) hide)
     )
@@
       (effects (font (size 1.27 1.27)) (justify left))
     )
-    (property "Value" "" (id 1) (at 275.59 65.9129 0)
+    (property "Value" "Y" (id 1) (at 275.59 65.9129 0)
       (effects (font (size 1.27 1.27)) (justify left) hide)
     )
@@
       (effects (font (size 1.27 1.27)) (justify left))
     )
-    (property "Value" "" (id 1) (at 104.14 90.0429 0)
+    (property "Value" "D" (id 1) (at 104.14 90.0429 0)
       (effects (font (size 1.27 1.27)) (justify left) hide)
     )
@@
     (in_bom yes) (on_board yes) (fields_autoplaced)
     (property "Reference" "U?" (id 0) (at 152.4 168.91 0))
-    (property "Value" "" (id 1) (at 152.4 171.45 0))
+    (property "Value" "74HC00" (id 1) (at 152.4 171.45 0))
     (property "Footprint" "" (id 2) (at 152.4 177.8 0)
       (effects (font (size 1.27 1.27)) hide)
@@
       (effects (font (size 1.27 1.27)) (justify left))
     )
-    (property "Value" "" (id 1) (at 143.51 176.5299 0)
-      (effects (font (size 1.27 1.27)) (justify left))
-    )
+    (property "Value" "A" (id 1) (at 143.51 176.5299 0)
+      (effects (font (size 1.27 1.27)) (justify left))
+    )

Commit message: pcb next :sunglasses:
Parts:
- U6: renamed from U?; value MCP3002 -> (none)
- gave numbers to parts that had none: 68

Commit message: pcb babeee les goooo
Parts:
- C14, C15, C16, C17, C18, C19, C20, C21, C22, C23, C24, C25: footprint (none) -> Capacitor_SMD:C_0805_2012Metric_Pad1.18x1.45mm_HandSolder
- J2: footprint (none) -> Connector_Wire:SolderWire-0.1sqmm_1x04_P3.6mm_D0.4mm_OD1mm
- R13: renamed from R12; footprint (none) -> Resistor_SMD:R_0805_2012Metric_Pad1.20x1.40mm_HandSolder
- R14: renamed from R13; footprint (none) -> Resistor_SMD:R_0805_2012Metric_Pad1.20x1.40mm_HandSolder
- R15: renamed from R14; footprint (none) -> Resistor_SMD:R_0805_2012Metric_Pad1.20x1.40mm_HandSolder
- R16: renamed from R15; footprint (none) -> Resistor_SMD:R_0805_2012Metric_Pad1.20x1.40mm_HandSolder
- R17: renamed from R16; footprint (none) -> Resistor_SMD:R_0805_2012Metric_Pad1.20x1.40mm_HandSolder
- R18: renamed from R17; footprint (none) -> Resistor_SMD:R_0805_2012Metric_Pad1.20x1.40mm_HandSolder
- R19: renamed from R18; footprint (none) -> Resistor_SMD:R_0805_2012Metric_Pad1.20x1.40mm_HandSolder
- R20: renamed from R19; footprint (none) -> Resistor_SMD:R_0805_2012Metric_Pad1.20x1.40mm_HandSolder
- R21: renamed from R20; footprint (none) -> Resistor_SMD:R_0805_2012Metric_Pad1.20x1.40mm_HandSolder
- R22: renamed from R21; footprint (none) -> Resistor_SMD:R_0805_2012Metric_Pad1.20x1.40mm_HandSolder
- R23: renamed from R22; footprint (none) -> Resistor_SMD:R_0805_2012Metric_Pad1.20x1.40mm_HandSolder
- R24: renamed from R23; footprint (none) -> Resistor_SMD:R_0805_2012Metric_Pad1.20x1.40mm_HandSolder
- R25: renamed from R24; footprint (none) -> Resistor_SMD:R_0805_2012Metric_Pad1.20x1.40mm_HandSolder
- R26: renamed from R25; footprint (none) -> Resistor_SMD:R_0805_2012Metric_Pad1.20x1.40mm_HandSolder
- R27: renamed from R26; footprint (none) -> Resistor_SMD:R_0805_2012Metric_Pad1.20x1.40mm_HandSolder
- R28: renamed from R27; footprint (none) -> Resistor_SMD:R_0805_2012Metric_Pad1.20x1.40mm_HandSolder
- R29: renamed from R28; footprint (none) -> Resistor_SMD:R_0805_2012Metric_Pad1.20x1.40mm_HandSolder
- R30: renamed from R29; footprint (none) -> Resistor_SMD:R_0805_2012Metric_Pad1.20x1.40mm_HandSolder
- R31: renamed from R30; footprint (none) -> Resistor_SMD:R_0805_2012Metric_Pad1.20x1.40mm_HandSolder
- R32: renamed from R31; footprint (none) -> Resistor_SMD:R_0805_2012Metric_Pad1.20x1.40mm_HandSolder
- R33: renamed from R32; footprint (none) -> Resistor_SMD:R_0805_2012Metric_Pad1.20x1.40mm_HandSolder
- R34: renamed from R33; footprint (none) -> Resistor_SMD:R_0805_2012Metric_Pad1.20x1.40mm_HandSolder
- R35: renamed from R34; footprint (none) -> Resistor_SMD:R_0805_2012Metric_Pad1.20x1.40mm_HandSolder
- R36: renamed from R35; footprint (none) -> Resistor_SMD:R_0805_2012Metric_Pad1.20x1.40mm_HandSolder
- R37: renamed from R36; footprint (none) -> Resistor_SMD:R_0805_2012Metric_Pad1.20x1.40mm_HandSolder
- SW1, SW10, SW11, SW2, SW3, SW4, SW5, SW6, SW7, SW8, SW9: footprint (none) -> CM4IO:SW_PTS526_SMG15_SMTR2_LFS
- TP10: renamed from TP9; footprint (none) -> TestPoint:TestPoint_THTPad_1.0x1.0mm_Drill0.5mm
- TP11: renamed from TP10; footprint (none) -> TestPoint:TestPoint_THTPad_1.0x1.0mm_Drill0.5mm
- TP12: renamed from TP11; footprint (none) -> TestPoint:TestPoint_THTPad_1.0x1.0mm_Drill0.5mm
- TP13: renamed from TP12; footprint (none) -> TestPoint:TestPoint_THTPad_1.0x1.0mm_Drill0.5mm
- TP14: renamed from TP13; footprint (none) -> TestPoint:TestPoint_THTPad_1.0x1.0mm_Drill0.5mm
- TP15: renamed from TP14; footprint (none) -> TestPoint:TestPoint_THTPad_1.0x1.0mm_Drill0.5mm
- TP16: renamed from TP15; footprint (none) -> TestPoint:TestPoint_THTPad_1.0x1.0mm_Drill0.5mm
- TP17: renamed from TP16; footprint (none) -> TestPoint:TestPoint_THTPad_1.0x1.0mm_Drill0.5mm
- TP18: renamed from TP17; footprint (none) -> TestPoint:TestPoint_THTPad_1.0x1.0mm_Drill0.5mm
- TP19: renamed from TP18; footprint (none) -> TestPoint:TestPoint_THTPad_1.0x1.0mm_Drill0.5mm
- TP20: renamed from TP19; footprint (none) -> TestPoint:TestPoint_THTPad_1.0x1.0mm_Drill0.5mm
- TP21: renamed from TP20; footprint (none) -> TestPoint:TestPoint_THTPad_1.0x1.0mm_Drill0.5mm
- TP22: renamed from TP21; footprint (none) -> TestPoint:TestPoint_THTPad_1.0x1.0mm_Drill0.5mm
- TP23: renamed from TP22; footprint (none) -> TestPoint:TestPoint_THTPad_1.0x1.0mm_Drill0.5mm
- TP6: renamed from TP5; footprint (none) -> TestPoint:TestPoint_THTPad_1.0x1.0mm_Drill0.5mm
- TP7: renamed from TP6; footprint (none) -> TestPoint:TestPoint_THTPad_1.0x1.0mm_Drill0.5mm
- TP8: renamed from TP7; footprint (none) -> TestPoint:TestPoint_THTPad_1.0x1.0mm_Drill0.5mm
- TP9: renamed from TP8; footprint (none) -> TestPoint:TestPoint_THTPad_1.0x1.0mm_Drill0.5mm
- U5: footprint (none) -> Package_DIP:DIP-14_W7.62mm_Socket_LongPads
- U6: value (none) -> MCP3002; footprint (none) -> Package_DIP:DIP-8_W7.62mm_LongPads
Other:
- moved on the sheet: U5E
