File: CM4Carrier/heiarchy/buttons.kicad_sch (KiCad schematic)
At the start: 90 parts, among them J2 Conn_01x04_Female, SW1 SW_Push, SW10 SW_Push, SW11 SW_Push, SW2 SW_Push, SW3 SW_Push, SW4 SW_Push, SW5 SW_Push, SW6 SW_Push, SW7 SW_Push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

Commit message: aa
Parts:
- gave numbers to parts that had none: 20
Changed lines of the file:
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@@
   (symbol (lib_id "Device:R") (at 30.48 93.98 0) (unit 1)
     (in_bom yes) (on_board yes) (fields_autoplaced)
-    (property "Reference" "R?" (id 0) (at 33.02 92.7099 0)
+    (property "Reference" "R49" (id 0) (at 33.02 92.7099 0)
       (effects (font (size 1.27 1.27)) (justify left))
     )
@@
   (symbol (lib_id "Device:R") (at 30.48 24.13 0) (unit 1)
     (in_bom yes) (on_board yes) (fields_autoplaced)
-    (property "Reference" "R?" (id 0) (at 33.02 22.8599 0)
+    (property "Reference" "R47" (id 0) (at 33.02 22.8599 0)
       (effects (font (size 1.27 1.27)) (justify left))
     )
@@
   (symbol (lib_id "Device:R") (at 24.13 62.23 90) (unit 1)
     (in_bom yes) (on_board yes) (fields_autoplaced)
-    (property "Reference" "R?" (id 0) (at 24.13 55.88 90))
+    (property "Reference" "R44" (id 0) (at 24.13 55.88 90))
     (property "Value" "1k" (id 1) (at 24.13 58.42 90))
     (property "Footprint" "Resistor_SMD:R_0805_2012Metric_Pad1.20x1.40mm_HandSolder" (id 2) (at 24.13 64.008 90)
@@
   (symbol (lib_id "power:GND") (at 15.24 76.2 0) (unit 1)
     (in_bom yes) (on_board yes) (fields_autoplaced)
-    (property "Reference" "#PWR?" (id 0) (at 15.24 82.55 0)
+    (property "Reference" "#PWR0104" (id 0) (at 15.24 82.55 0)
       (effects (font (size 1.27 1.27)) hide)
     )
@@
   (symbol (lib_id "Device:C") (at 30.48 71.12 0) (unit 1)
     (in_bom yes) (on_board yes) (fields_autoplaced)
-    (property "Reference" "C?" (id 0) (at 34.29 69.8499 0)
+    (property "Reference" "C32" (id 0) (at 34.29 69.8499 0)
       (effects (font (size 1.27 1.27)) (justify left))
     )
@@
   (symbol (lib_id "Device:R") (at 30.48 127 0) (unit 1)
     (in_bom yes) (on_board yes) (fields_autoplaced)
-    (property "Reference" "R?" (id 0) (at 33.02 125.7299 0)
+    (property "Reference" "R50" (id 0) (at 33.02 125.7299 0)
       (effects (font (size 1.27 1.27)) (justify left))
     )
@@
   (symbol (lib_id "Device:C") (at 30.48 140.97 0) (unit 1)
     (in_bom yes) (on_board yes) (fields_autoplaced)
-    (property "Reference" "C?" (id 0) (at 34.29 139.6999 0)
+    (property "Reference" "C34" (id 0) (at 34.29 139.6999 0)
       (effects (font (size 1.27 1.27)) (justify left))
     )
@@
   (symbol (lib_id "Switch:SW_Push") (at 17.78 69.85 90) (unit 1)
     (in_bom yes) (on_board yes) (fields_autoplaced)
-    (property "Reference" "SW?" (id 0) (at 19.05 68.5799 90)
+    (property "Reference" "SW13" (id 0) (at 19.05 68.5799 90)
       (effects (font (size 1.27 1.27)) (justify right))
     )
@@
   (symbol (lib_id "power:GND") (at 15.24 146.05 0) (unit 1)
     (in_bom yes) (on_board yes) (fields_autoplaced)
-    (property "Reference" "#PWR?" (id 0) (at 15.24 152.4 0)
+    (property "Reference" "#PWR0101" (id 0) (at 15.24 152.4 0)
       (effects (font (size 1.27 1.27)) hide)
     )
@@
   (symbol (lib_id "Device:R") (at 24.13 29.21 90) (unit 1)
     (in_bom yes) (on_board yes) (fields_autoplaced)
-    (property "Reference" "R?" (id 0) (at 24.13 22.86 90))
+    (property "Reference" "R43" (id 0) (at 24.13 22.86 90))
     (property "Value" "1k" (id 1) (at 24.13 25.4 90))
     (property "Footprint" "Resistor_SMD:R_0805_2012Metric_Pad1.20x1.40mm_HandSolder" (id 2) (at 24.13 30.988 90)
@@
   (symbol (lib_id "Device:R") (at 24.13 99.06 90) (unit 1)
     (in_bom yes) (on_board yes) (fields_autoplaced)
-    (property "Reference" "R?" (id 0) (at 24.13 92.71 90))
+    (property "Reference" "R45" (id 0) (at 24.13 92.71 90))
     (property "Value" "1k" (id 1) (at 24.13 95.25 90))
     (property "Footprint" "Resistor_SMD:R_0805_2012Metric_Pad1.20x1.40mm_HandSolder" (id 2) (at 24.13 100.838 90)
@@
   (symbol (lib_id "Device:C") (at 30.48 38.1 0) (unit 1)
     (in_bom yes) (on_board yes) (fields_autoplaced)
-    (property "Reference" "C?" (id 0) (at 34.29 36.8299 0)
+    (property "Reference" "C31" (id 0) (at 34.29 36.8299 0)
       (effects (font (size 1.27 1.27)) (justify left))
     )
@@
   (symbol (lib_id "Device:R") (at 30.48 57.15 0) (unit 1)
     (in_bom yes) (on_board yes) (fields_autoplaced)
-    (property "Reference" "R?" (id 0) (at 33.02 55.8799 0)
+    (property "Reference" "R48" (id 0) (at 33.02 55.8799 0)
       (effects (font (size 1.27 1.27)) (justify left))
     )
@@
   (symbol (lib_id "Switch:SW_Push") (at 17.78 36.83 90) (unit 1)
     (in_bom yes) (on_board yes) (fields_autoplaced)
-    (property "Reference" "SW?" (id 0) (at 19.05 35.5599 90)
+    (property "Reference" "SW12" (id 0) (at 19.05 35.5599 90)
       (effects (font (size 1.27 1.27)) (justify right))
     )
@@
   (symbol (lib_id "Switch:SW_Push") (at 17.78 139.7 90) (unit 1)
     (in_bom yes) (on_board yes) (fields_autoplaced)
-    (property "Reference" "SW?" (id 0) (at 19.05 138.4299 90)
+    (property "Reference" "SW15" (id 0) (at 19.05 138.4299 90)
       (effects (font (size 1.27 1.27)) (justify right))
     )
@@
   (symbol (lib_id "Connector:TestPoint_Flag") (at 38.1 100.33 0) (unit 1)
     (in_bom yes) (on_board yes)
-    (property "Reference" "TP?" (id 0) (at 39.37 96.52 0)
+    (property "Reference" "TP27" (id 0) (at 39.37 96.52 0)
       (effects (font (size 1.27 1.27)) (justify left))
     )
@@
   (symbol (lib_id "Connector:TestPoint_Flag") (at 38.1 63.5 0) (unit 1)
     (in_bom yes) (on_board yes)
-    (property "Reference" "TP?" (id 0) (at 39.37 59.69 0)
+    (property "Reference" "TP26" (id 0) (at 39.37 59.69 0)
       (effects (font (size 1.27 1.27)) (justify left))
     )
@@
   (symbol (lib_id "power:GND") (at 15.24 43.18 0) (unit 1)
     (in_bom yes) (on_board yes) (fields_autoplaced)
-    (property "Reference" "#PWR?" (id 0) (at 15.24 49.53 0)
+    (property "Reference" "#PWR0103" (id 0) (at 15.24 49.53 0)
       (effects (font (size 1.27 1.27)) hide)
     )
@@
   (symbol (lib_id "Device:R") (at 24.13 132.08 90) (unit 1)
     (in_bom yes) (on_board yes) (fields_autoplaced)
-    (property "Reference" "R?" (id 0) (at 24.13 125.73 90))
+    (property "Reference" "R46" (id 0) (at 24.13 125.73 90))
     (property "Value" "1k" (id 1) (at 24.13 128.27 90))
     (property "Footprint" "Resistor_SMD:R_0805_2012Metric_Pad1.20x1.40mm_HandSolder" (id 2) (at 24.13 133.858 90)
@@
   (symbol (lib_id "Device:C") (at 30.48 107.95 0) (unit 1)
     (in_bom yes) (on_board yes) (fields_autoplaced)
-    (property "Reference" "C?" (id 0) (at 34.29 106.6799 0)
+    (property "Reference" "C33" (id 0) (at 34.29 106.6799 0)
       (effects (font (size 1.27 1.27)) (justify left))
     )
@@
   (symbol (lib_id "power:GND") (at 15.24 113.03 0) (unit 1)
     (in_bom yes) (on_board yes) (fields_autoplaced)
-    (property "Reference" "#PWR?" (id 0) (at 15.24 119.38 0)
+    (property "Reference" "#PWR0102" (id 0) (at 15.24 119.38 0)
       (effects (font (size 1.27 1.27)) hide)
     )
@@
   (symbol (lib_id "Connector:TestPoint_Flag") (at 38.1 133.35 0) (unit 1)
     (in_bom yes) (on_board yes)
-    (property "Reference" "TP?" (id 0) (at 39.37 129.54 0)
+    (property "Reference" "TP28" (id 0) (at 39.37 129.54 0)
       (effects (font (size 1.27 1.27)) (justify left))
     )
@@
   (symbol (lib_id "Connector:TestPoint_Flag") (at 38.1 30.48 0) (unit 1)
     (in_bom yes) (on_board yes)
-    (property "Reference" "TP?" (id 0) (at 39.37 26.67 0)
+    (property "Reference" "TP25" (id 0) (at 39.37 26.67 0)
       (effects (font (size 1.27 1.27)) (justify left))
     )
@@
   (symbol (lib_id "Switch:SW_Push") (at 17.78 106.68 90) (unit 1)
     (in_bom yes) (on_board yes) (fields_autoplaced)
-    (property "Reference" "SW?" (id 0) (at 19.05 105.4099 90)
-      (effects (font (size 1.27 1.27)) (justify right))
-    )
+    (property "Reference" "SW14" (id 0) (at 19.05 105.4099 90)
+      (effects (font (size 1.27 1.27)) (justify right))
+    )

Commit message: a
Parts:
- removed TP20: U/D, TestPoint:TestPoint_THTPad_1.0x1.0mm_Drill0.5mm, symbol Connector:TestPoint_Flag
- removed TP21: L/R, TestPoint:TestPoint_THTPad_1.0x1.0mm_Drill0.5mm, symbol Connector:TestPoint_Flag
Changed lines of the file:
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@@
   (junction (at 130.81 39.37) (diameter 0) (color 0 0 0 0)
   )
-  (junction (at 228.6 124.46) (diameter 0) (color 0 0 0 0)
-  )
   (junction (at 115.57 171.45) (diameter 0) (color 0 0 0 0)
   )
@@
   (junction (at 217.17 78.74) (diameter 0) (color 0 0 0 0)
   )
-  (junction (at 227.33 134.62) (diameter 0) (color 0 0 0 0)
-  )
   (wire (pts (xy 118.11 139.7) (xy 118.11 140.97))
     (stroke (width 0) (type default) (color 0 0 0 0))
@@
     (stroke (width 0) (type default) (color 0 0 0 0))
   )
-  (wire (pts (xy 227.33 134.62) (xy 243.84 134.62))
+  (wire (pts (xy 208.28 134.62) (xy 243.84 134.62))
     (stroke (width 0) (type default) (color 0 0 0 0))
   )
@@
     (stroke (width 0) (type default) (color 0 0 0 0))
   )
-  (wire (pts (xy 208.28 134.62) (xy 227.33 134.62))
-    (stroke (width 0) (type default) (color 0 0 0 0))
-  )
   (wire (pts (xy 30.48 133.35) (xy 38.1 133.35))
     (stroke (width 0) (type default) (color 0 0 0 0))
@@
     (stroke (width 0) (type default) (color 0 0 0 0))
   )
-  (wire (pts (xy 219.71 124.46) (xy 228.6 124.46))
-    (stroke (width 0) (type default) (color 0 0 0 0))
-  )
   (polyline (pts (xy 283.21 101.6) (xy 177.8 101.6))
     (stroke (width 0) (type default) (color 0 0 0 0))
@@
     (stroke (width 0) (type default) (color 0 0 0 0))
   )
-  (wire (pts (xy 228.6 124.46) (xy 243.84 124.46))
+  (wire (pts (xy 219.71 124.46) (xy 243.84 124.46))
     (stroke (width 0) (type default) (color 0 0 0 0))
   )
@@
     (pin "1")
     (pin "2")
-  )
-  (symbol (lib_id "Connector:TestPoint_Flag") (at 227.33 134.62 0) (unit 1)
-    (in_bom yes) (on_board yes) (fields_autoplaced)
-    (property "Reference" "TP20" (id 0) (at 234.95 131.9529 0)
-      (effects (font (size 1.27 1.27)) (justify left))
-    )
-    (property "Value" "U/D" (id 1) (at 234.95 134.4929 0)
-      (effects (font (size 1.27 1.27)) (justify left))
-    )
-    (property "Footprint" "TestPoint:TestPoint_THTPad_1.0x1.0mm_Drill0.5mm" (id 2) (at 232.41 134.62 0)
-      (effects (font (size 1.27 1.27)) hide)
-    )
-    (property "Datasheet" "~" (id 3) (at 232.41 134.62 0)
-      (effects (font (size 1.27 1.27)) hide)
-    )
-    (pin "1")
   )
   (symbol (lib_id "Device:R") (at 123.19 33.02 0) (unit 1)
@@
       (effects (font (size 1.27 1.27)) hide)
     )
-    (pin "1")
-  )
-  (symbol (lib_id "Connector:TestPoint_Flag") (at 228.6 124.46 0) (unit 1)
-    (in_bom yes) (on_board yes) (fields_autoplaced)
-    (property "Reference" "TP21" (id 0) (at 236.22 121.7929 0)
-      (effects (font (size 1.27 1.27)) (justify left))
-    )
-    (property "Value" "L/R" (id 1) (at 236.22 124.3329 0)
-      (effects (font (size 1.27 1.27)) (justify left))
-    )
-    (property "Footprint" "TestPoint:TestPoint_THTPad_1.0x1.0mm_Drill0.5mm" (id 2) (at 233.68 124.46 0)
-      (effects (font (size 1.27 1.27)) hide)
-    )
-    (property "Datasheet" "~" (id 3) (at 233.68 124.46 0)
-      (effects (font (size 1.27 1.27)) hide)
-    )
