File: CM4Carrier/CM4Carrier.kicad_pcb (KiCad board)
At the start: 2 copper layers, 125 x 80 mm, 4 parts

Commit message: pcb babeee les goooo
Parts:
- added BT1: Battery_Cell, Connector_JST:JST_XH_S2B-XH-A_1x02_P2.50mm_Horizontal, B.Cu at (141.0, 87.3)
- added C1: 10u, Capacitor_SMD:C_0805_2012Metric_Pad1.18x1.45mm_HandSolder, F.Cu at (154.6, -69.7)
- added C10: 470n, Capacitor_SMD:C_0603_1608Metric_Pad1.08x0.95mm_HandSolder, B.Cu at (144.6, 147.3)
- added C11: 22u, Capacitor_SMD:C_0805_2012Metric_Pad1.18x1.45mm_HandSolder, F.Cu at (276.9, 46.4)
- added C12: 22u, Capacitor_SMD:C_0805_2012Metric_Pad1.18x1.45mm_HandSolder, F.Cu at (285.7, 40.5)
- added C13: 22u, Capacitor_SMD:C_0805_2012Metric_Pad1.18x1.45mm_HandSolder, F.Cu at (281.7, 45.6)
- added C14: 100n, Capacitor_SMD:C_0805_2012Metric_Pad1.18x1.45mm_HandSolder, F.Cu at (146.0, -6.34)
- added C15: 100n, Capacitor_SMD:C_0805_2012Metric_Pad1.18x1.45mm_HandSolder, F.Cu at (150.8, -9.35)
- added C16: 1u, Capacitor_SMD:C_0805_2012Metric_Pad1.18x1.45mm_HandSolder, F.Cu at (122.5, 20.9)
- added C17: 1u, Capacitor_SMD:C_0805_2012Metric_Pad1.18x1.45mm_HandSolder, F.Cu at (154.9, -13.5)
- added C18: 100n, Capacitor_SMD:C_0805_2012Metric_Pad1.18x1.45mm_HandSolder, F.Cu at (146.0, -9.35)
- added C19: 100n, Capacitor_SMD:C_0805_2012Metric_Pad1.18x1.45mm_HandSolder, F.Cu at (146.0, -3.33)
- added C2: 2.2u, Capacitor_SMD:C_0805_2012Metric_Pad1.18x1.45mm_HandSolder, F.Cu at (276.9, 49.4)
- added C20: 100n, Capacitor_SMD:C_0805_2012Metric_Pad1.18x1.45mm_HandSolder, F.Cu at (150.8, -6.34)
- added C21: 100n, Capacitor_SMD:C_0805_2012Metric_Pad1.18x1.45mm_HandSolder, F.Cu at (113.4, 28.1)
- added C22: 100nF, Capacitor_SMD:C_0805_2012Metric_Pad1.18x1.45mm_HandSolder, F.Cu at (154.9, -16.5)
- added C23: 100n, Capacitor_SMD:C_0805_2012Metric_Pad1.18x1.45mm_HandSolder, F.Cu at (131.6, 12.1)
- added C24: 100n, Capacitor_SMD:C_0805_2012Metric_Pad1.18x1.45mm_HandSolder, F.Cu at (113.4, 31.1)
- added C25: 100n, Capacitor_SMD:C_0805_2012Metric_Pad1.18x1.45mm_HandSolder, F.Cu at (159.7, -16.5)
- added C26: 100n, Capacitor_SMD:C_0805_2012Metric_Pad1.18x1.45mm_HandSolder, B.Cu at (133.1, 55.9)
- added C3: 2.2u, Capacitor_SMD:C_0805_2012Metric_Pad1.18x1.45mm_HandSolder, F.Cu at (290.5, 37.5)
- added C4: 100n, Capacitor_SMD:C_0805_2012Metric_Pad1.18x1.45mm_HandSolder, F.Cu at (280.0, 42.6)
- added C5: C, Capacitor_SMD:C_0805_2012Metric_Pad1.18x1.45mm_HandSolder, F.Cu at (270.6, 62.6)
- added C6: 22u, Capacitor_SMD:C_0805_2012Metric_Pad1.18x1.45mm_HandSolder, F.Cu at (276.9, 52.4)
- added C7: C, Capacitor_SMD:C_0805_2012Metric_Pad1.18x1.45mm_HandSolder, F.Cu at (281.7, 48.6)
- added C8: 2.2u, Capacitor_SMD:C_0805_2012Metric_Pad1.18x1.45mm_HandSolder, F.Cu at (265.3, 67.2)
- added C9: 22u, Capacitor_SMD:C_0805_2012Metric_Pad1.18x1.45mm_HandSolder, F.Cu at (285.7, 37.5)
- added D1: LED, LED_SMD:LED_0805_2012Metric_Pad1.15x1.40mm_HandSolder, F.Cu at (171.5, -85.6)
- added D2: LED, LED_SMD:LED_0805_2012Metric_Pad1.15x1.40mm_HandSolder, F.Cu at (276.9, 55.4)
- added D3: LED, LED_SMD:LED_0805_2012Metric_Pad1.15x1.40mm_HandSolder, F.Cu at (295.3, 37.5)
- added J1: Micro_SD_Card, CM4IO:GCT_MEM2067-02-180-00-A_REVB, B.Cu at (124.4, 109.2)
- added J2: Conn_01x04_Female, Connector_Wire:SolderWire-0.1sqmm_1x04_P3.6mm_D0.4mm_OD1mm, F.Cu at (112.8, 3.32)
- added J3: USB_A, CM4IO:GCT_USB1125-GF-B_REVA, B.Cu at (96.5, 53.3)
- added J4: USB_C_Receptacle_USB2.0, CM4IO:GCT_USB4110-GF-A_REVB, B.Cu at (139.7, 116.8)
- added J5: 1-84952-5, CM4IO:TE_1-84952-5, B.Cu at (121.9, 54.5)
- added L1: 0.47u, Inductor_SMD:L_1008_2520Metric_Pad1.43x2.20mm_HandSolder, F.Cu at (280.6, 37.9)
- added L2: 1u, Inductor_SMD:L_1008_2520Metric_Pad1.43x2.20mm_HandSolder, F.Cu at (257.7, 43.2)
- added Module1: ComputeModule4-CM4, CM4IO:Raspberry-Pi-4-Compute-Module, B.Cu at (85.2, 95.2)
- added R1: 1k, Resistor_SMD:R_0805_2012Metric_Pad1.20x1.40mm_HandSolder, F.Cu at (120.8, -29.6)
- added R10: 400k, Resistor_SMD:R_0603_1608Metric_Pad0.98x0.95mm_HandSolder, B.Cu at (149.6, 147.3)
- added R11: 1M, Resistor_SMD:R_0805_2012Metric_Pad1.20x1.40mm_HandSolder, F.Cu at (286.5, 49.4)
- added R12: 10k, Resistor_SMD:R_0805_2012Metric_Pad1.20x1.40mm_HandSolder, F.Cu at (286.5, 46.5)
- added R13: 1k, Resistor_SMD:R_0805_2012Metric_Pad1.20x1.40mm_HandSolder, F.Cu at (155.6, -4.61)
- added R14: 1k, Resistor_SMD:R_0805_2012Metric_Pad1.20x1.40mm_HandSolder, F.Cu at (160.4, -7.62)
- added R15: 10k, Resistor_SMD:R_0805_2012Metric_Pad1.20x1.40mm_HandSolder, F.Cu at (146.0, -0.35)
- added R16: 10k, Resistor_SMD:R_0805_2012Metric_Pad1.20x1.40mm_HandSolder, F.Cu at (131.5, 15.1)
- added R17: 100k, Resistor_SMD:R_0805_2012Metric_Pad1.20x1.40mm_HandSolder, F.Cu at (146.0, 2.60)
- added R18: 5M, Resistor_SMD:R_0805_2012Metric_Pad1.20x1.40mm_HandSolder, F.Cu at (113.4, 34.1)
- added R19: 100k, Resistor_SMD:R_0805_2012Metric_Pad1.20x1.40mm_HandSolder, F.Cu at (164.5, -13.6)
- added R2: nc, Resistor_SMD:R_0805_2012Metric_Pad1.20x1.40mm_HandSolder, F.Cu at (113.4, -25.0)
- added R20: 1k, Resistor_SMD:R_0805_2012Metric_Pad1.20x1.40mm_HandSolder, F.Cu at (118.2, 28.1)
- added R21: 1k, Resistor_SMD:R_0805_2012Metric_Pad1.20x1.40mm_HandSolder, F.Cu at (164.5, -16.5)
- added R22: 10k, Resistor_SMD:R_0805_2012Metric_Pad1.20x1.40mm_HandSolder, F.Cu at (136.3, 12.1)
- added R23: 10k, Resistor_SMD:R_0805_2012Metric_Pad1.20x1.40mm_HandSolder, F.Cu at (127.2, 23.9)
- added R24: 1k, Resistor_SMD:R_0805_2012Metric_Pad1.20x1.40mm_HandSolder, F.Cu at (155.6, -10.5)
- added R25: 10k, Resistor_SMD:R_0805_2012Metric_Pad1.20x1.40mm_HandSolder, F.Cu at (118.2, 31.0)
- added R26: 1k, Resistor_SMD:R_0805_2012Metric_Pad1.20x1.40mm_HandSolder, F.Cu at (160.4, -10.6)
- added R27: 2K7, Resistor_SMD:R_0805_2012Metric_Pad1.20x1.40mm_HandSolder, F.Cu at (140.6, 7.87)
- added R28: 10k, Resistor_SMD:R_0805_2012Metric_Pad1.20x1.40mm_HandSolder, F.Cu at (150.8, -3.36)
- added R29: 10k, Resistor_SMD:R_0805_2012Metric_Pad1.20x1.40mm_HandSolder, F.Cu at (123.0, 26.9)
- added R3: 10k, Resistor_SMD:R_0805_2012Metric_Pad1.20x1.40mm_HandSolder, F.Cu at (154.5, -66.7)
- added R30: 1k, Resistor_SMD:R_0805_2012Metric_Pad1.20x1.40mm_HandSolder, F.Cu at (140.6, 4.92)
- added R31: 10k, Resistor_SMD:R_0805_2012Metric_Pad1.20x1.40mm_HandSolder, F.Cu at (150.8, -0.41)
- added R32: 1k, Resistor_SMD:R_0805_2012Metric_Pad1.20x1.40mm_HandSolder, F.Cu at (159.7, -13.5)
- added R33: 10k, Resistor_SMD:R_0805_2012Metric_Pad1.20x1.40mm_HandSolder, F.Cu at (122.5, 23.9)
- added R34: 1k, Resistor_SMD:R_0805_2012Metric_Pad1.20x1.40mm_HandSolder, F.Cu at (127.3, 20.9)
- added R35: 10k, Resistor_SMD:R_0805_2012Metric_Pad1.20x1.40mm_HandSolder, F.Cu at (132.0, 18.0)
- added R36: 1k, Resistor_SMD:R_0805_2012Metric_Pad1.20x1.40mm_HandSolder, F.Cu at (155.6, -7.56)
- added R37: 10k, Resistor_SMD:R_0805_2012Metric_Pad1.20x1.40mm_HandSolder, F.Cu at (123.0, 29.8)
- added R38: nc, Resistor_SMD:R_0805_2012Metric_Pad1.20x1.40mm_HandSolder, B.Cu at (144.8, 111.8)
- added R4: 1k, Resistor_SMD:R_0805_2012Metric_Pad1.20x1.40mm_HandSolder, F.Cu at (281.7, 51.6)
- added R5: 1k, Resistor_SMD:R_0805_2012Metric_Pad1.20x1.40mm_HandSolder, F.Cu at (275.4, 62.6)
- added R6: R, Resistor_SMD:R_0805_2012Metric_Pad1.20x1.40mm_HandSolder, F.Cu at (290.5, 40.5)
- added R7: R, Resistor_SMD:R_0805_2012Metric_Pad1.20x1.40mm_HandSolder, F.Cu at (281.7, 54.6)
- added R8: R, Resistor_SMD:R_0805_2012Metric_Pad1.20x1.40mm_HandSolder, F.Cu at (291.3, 43.4)
- added R9: 600k, Resistor_SMD:R_0603_1608Metric_Pad0.98x0.95mm_HandSolder, B.Cu at (149.6, 142.2)
- added SW1: SW_Push, CM4IO:SW_PTS526_SMG15_SMTR2_LFS, F.Cu at (139.3, -7.28)
- added SW10: SW_Push, CM4IO:SW_PTS526_SMG15_SMTR2_LFS, F.Cu at (130.3, -2.68)
- added SW11: SW_Push, CM4IO:SW_PTS526_SMG15_SMTR2_LFS, F.Cu at (115.8, 15.9)
- added SW2: SW_Push, CM4IO:SW_PTS526_SMG15_SMTR2_LFS, F.Cu at (139.3, -0.13)
- added SW3: SW_Push, CM4IO:SW_PTS526_SMG15_SMTR2_LFS, F.Cu at (148.2, -14.4)
- added SW4: SW_Push, CM4IO:SW_PTS526_SMG15_SMTR2_LFS, F.Cu at (134.0, 7.02)
- added SW5: SW_Push, CM4IO:SW_PTS526_SMG15_SMTR2_LFS, F.Cu at (124.9, 8.72)
- added SW6: SW_Push, CM4IO:SW_PTS526_SMG15_SMTR2_LFS, F.Cu at (139.2, -14.4)
- added SW7: SW_Push, CM4IO:SW_PTS526_SMG15_SMTR2_LFS, F.Cu at (124.9, 15.9)
- added SW8: SW_Push, CM4IO:SW_PTS526_SMG15_SMTR2_LFS, F.Cu at (115.8, 8.72)
- added SW9: SW_Push, CM4IO:SW_PTS526_SMG15_SMTR2_LFS, F.Cu at (115.8, 23.0)
- added TH1: 10k 5%, Resistor_SMD:R_0805_2012Metric_Pad1.20x1.40mm_HandSolder, B.Cu at (162.3, 144.8)
- added TP1: TestPoint POWER PI, TestPoint:TestPoint_THTPad_1.0x1.0mm_Drill0.5mm, F.Cu at (175.4, -85.6)
- added TP10: START, TestPoint:TestPoint_THTPad_1.0x1.0mm_Drill0.5mm, F.Cu at (144.5, 8.65)
- added TP11: R, TestPoint:TestPoint_THTPad_1.0x1.0mm_Drill0.5mm, F.Cu at (164.3, -7.53)
- added TP12: A, TestPoint:TestPoint_THTPad_1.0x1.0mm_Drill0.5mm, F.Cu at (127.0, 2.42)
- added TP13: B, TestPoint:TestPoint_THTPad_1.0x1.0mm_Drill0.5mm, F.Cu at (135.9, 18.1)
- added TP14: A, TestPoint:TestPoint_THTPad_1.0x1.0mm_Drill0.5mm, F.Cu at (159.5, -4.62)
- added TP15: B, TestPoint:TestPoint_THTPad_1.0x1.0mm_Drill0.5mm, F.Cu at (126.9, 26.9)
- added TP16: (A.B)' (0), TestPoint:TestPoint_THTPad_1.0x1.0mm_Drill0.5mm, F.Cu at (164.3, -10.6)
- added TP17: (A.B)' (1), TestPoint:TestPoint_THTPad_1.0x1.0mm_Drill0.5mm, F.Cu at (147.6, 8.65)
- added TP18: A, TestPoint:TestPoint_THTPad_1.0x1.0mm_Drill0.5mm, F.Cu at (144.5, 5.60)
- added TP19: X, TestPoint:TestPoint_THTPad_1.0x1.0mm_Drill0.5mm, F.Cu at (117.4, 34.0)
- added TP2: TestPoint_Flag, TestPoint:TestPoint_THTPad_1.0x1.0mm_Drill0.5mm, F.Cu at (153.7, -63.7)
- added TP20: U/D, TestPoint:TestPoint_THTPad_1.0x1.0mm_Drill0.5mm, F.Cu at (154.7, -1.61)
- added TP21: L/R, TestPoint:TestPoint_THTPad_1.0x1.0mm_Drill0.5mm, F.Cu at (154.7, 1.44)
- added TP22: B, TestPoint:TestPoint_THTPad_1.0x1.0mm_Drill0.5mm, F.Cu at (135.9, 15.1)
- added TP23: Y, TestPoint:TestPoint_THTPad_1.0x1.0mm_Drill0.5mm, F.Cu at (131.2, 21.0)
- added TP3: TP_PG, TestPoint:TestPoint_THTPad_1.0x1.0mm_Drill0.5mm, F.Cu at (264.4, 73.2)
- added TP4: 5VREG_EN, TestPoint:TestPoint_THTPad_1.0x1.0mm_Drill0.5mm, F.Cu at (290.4, 46.5)
- added TP5: TestPoint_Flag, TestPoint:TestPoint_THTPad_1.0x1.0mm_Drill0.5mm, F.Cu at (299.2, 37.5)
- added TP6: L, TestPoint:TestPoint_THTPad_1.0x1.0mm_Drill0.5mm, F.Cu at (140.2, 13.9)
- added TP7: SEL, TestPoint:TestPoint_THTPad_1.0x1.0mm_Drill0.5mm, F.Cu at (147.6, 5.60)
- added TP8: U, TestPoint:TestPoint_THTPad_1.0x1.0mm_Drill0.5mm, F.Cu at (120.4, 34.0)
- added TP9: D, TestPoint:TestPoint_THTPad_1.0x1.0mm_Drill0.5mm, F.Cu at (140.2, 10.9)
- added U1: MIC2025-2YMM, Package_SO:MSOP-8_3x3mm_P0.65mm, F.Cu at (114.7, -28.8)
- added U2: MAX77751, CM4IO:IC_MAX77751FEFG+, F.Cu at (251.5, 25.4)
- added U3: MAX17261xxTD, Package_DFN_QFN:TDFN-14-1EP_3x3mm_P0.4mm_EP1.78x2.35mm, B.Cu at (156.3, 144.8)
- added U4: MIC2877, CM4IO:MIC2877-AYFT-TR, F.Cu at (259.1, 48.3)
- added U5: 74HC00, Package_DIP:DIP-14_W7.62mm_Socket_LongPads, F.Cu at (160.0, 119.4)
- added U6: MCP3002, Package_DIP:DIP-8_W7.62mm_LongPads, B.Cu at (92.7, 111.8)
Other:
- outline, holes or cut-outs redrawn

Commit message: foo
Parts:
- C1, R2, R8, U1: moved to B.Cu
- moved C1 192.3 mm to (119.4, 119.4), turned to -90 degrees
- moved R8 157.4 mm to (142.2, 94.0), turned to -90 degrees
- moved U1 148.4 mm to (124.5, 119.4), turned to 180 degrees
- moved R2 135.9 mm to (134.6, 109.2), turned to 90 degrees
- moved SW11 116.3 mm to (203.2, -61.0)
- moved SW8 107.6 mm to (188.0, -71.1)
- moved SW9 105.0 mm to (188.0, -53.3)
- moved SW1 103.4 mm to (40.6, -38.1)
- moved SW4 102.3 mm to (53.3, -55.9)
- moved SW10 101.8 mm to (203.2, -73.7)
- moved SW5 80.5 mm to (50.8, -22.9)
- moved SW7 78.0 mm to (68.6, -38.1)
- moved SW2 69.1 mm to (129.5, -68.6)
- moved SW3 64.7 mm to (96.5, -53.3)
- moved SW6 57.7 mm to (119.4, -68.6)
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
Commit message: pcb w proper design
Parts:
- removed the REF** at (202.0, 120.0)
- removed the REF** at (85.0, 48.0)
- removed the REF** at (85.0, 120.0)
- removed the REF** at (202.0, 48.0)
- added REF**: MountingHole_2.7mm_M2.5, MountingHole:MountingHole_2.7mm_M2.5, F.Cu at (428.9, 160.6)
- added REF**: OSHW-Logo2_24.3x20mm_SilkScreen, Symbol:OSHW-Logo2_24.3x20mm_SilkScreen, F.Cu at (476.0, 101.0)
- added REF**: MountingHole_2.7mm_M2.5, MountingHole:MountingHole_2.7mm_M2.5, F.Cu at (414.0, 87.6)
- added REF**: MountingHole_2.7mm_M2.5, MountingHole:MountingHole_2.7mm_M2.5, F.Cu at (325.9, 87.6)
- added REF**: MountingHole_2.7mm_M2.5, MountingHole:MountingHole_2.7mm_M2.5, F.Cu at (428.9, 112.6)
- added REF**: MountingHole_2.7mm_M2.5, MountingHole:MountingHole_2.7mm_M2.5, F.Cu at (311.0, 160.6)
- added REF**: MountingHole_2.7mm_M2.5, MountingHole:MountingHole_2.7mm_M2.5, F.Cu at (311.0, 112.6)
- R3: moved to B.Cu
- moved SW3 362.4 mm to (416.2, 117.4)
- moved SW4 352.4 mm to (352.1, 131.1), turned to 180 degrees
- moved SW1 351.7 mm to (344.8, 138.4), turned to 180 degrees
- moved R3 345.8 mm to (355.6, 214.6), turned to 90 degrees
- moved SW5 345.2 mm to (352.1, 145.6)
- moved SW6 341.8 mm to (376.2, 156.9)
- moved SW7 340.2 mm to (359.4, 138.4)
- moved TP19 327.8 mm to (425.4, 146.1)
- moved SW2 325.1 mm to (363.7, 156.9)
- moved R37 323.0 mm to (426.7, 139.7), turned to 90 degrees
- moved R33 321.3 mm to (419.1, 147.3), turned to 90 degrees
- moved C23 320.0 mm to (421.6, 147.3), turned to -90 degrees
- moved TP23 314.8 mm to (426.7, 129.5)
- moved C25 311.5 mm to (429.3, 139.7), turned to -90 degrees
- moved R36 306.7 mm to (426.7, 135.9), turned to -90 degrees
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Other:
- board size 125 x 80 mm -> 125 x 84 mm
- board text added: "https://github.com/cinnamondev/gamepithing"

Commit message: PCB work
Home-stretch! Remaining things:
- Forgot Headphone jack / audio in design - add.
- route power supply (aaaaa)
Parts:
- added TP24: TP-GLOBALEN, TestPoint:TestPoint_THTPad_1.0x1.0mm_Drill0.5mm, F.Cu at (127.6, 67.3)
- C8: footprint Capacitor_SMD:C_0805_2012Metric_Pad1.18x1.45mm_HandSolder -> Capacitor_SMD:C_0603_1608Metric_Pad1.08x0.95mm_HandSolder
- J2, R27, R29, TP12, TP13, TP14, TP15, TP16, TP17, U5: moved to B.Cu
- R6, R7: footprint Resistor_SMD:R_0805_2012Metric_Pad1.20x1.40mm_HandSolder -> Resistor_SMD:R_0603_1608Metric_Pad0.98x0.95mm_HandSolder
- moved REF** 415.2 mm to (61.0, 88.9)
- moved R2 233.6 mm to (160.7, 116.8)
- moved J3 232.7 mm to (108.6, 65.2)
- moved R32 229.9 mm to (190.5, 119.4)
- moved R33 229.9 mm to (190.5, 123.2)
- moved R36 229.9 mm to (198.1, 111.8)
- moved R37 229.9 mm to (198.1, 115.6)
- moved SW1 229.9 mm to (116.2, 114.3)
- moved SW4 229.9 mm to (123.5, 107.0), turned to 0 degrees
- moved SW5 229.9 mm to (123.5, 121.5), turned to 180 degrees
- moved C23 229.9 mm to (193.0, 123.2)
- moved C25 229.9 mm to (200.7, 115.6)
- moved REF** 229.9 mm to (200.3, 136.5)
- moved REF** 229.9 mm to (185.4, 63.5)
- moved REF** 229.9 mm to (200.3, 88.5)
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Connections:
- BT1 pad 2: GND -> Net-(BT1-Pad2)
- R8 pad 1: GND -> Net-(BT1-Pad2)
- U2 pad 13_14: (no net) -> /BATT
- U2 pad 15_16: (no net) -> /BATT
- U2 pad 18_19: (no net) -> GND
- U2 pad 20_21: (no net) -> Net-(C4-Pad2)
- U2 pad 23_24: (no net) -> /Battery/CHRG-VBUS
- U3 pad 9: GND -> Net-(BT1-Pad2)

Commit message: LAYOUT DONE!!
:)
Parts:
- added C27: C, Capacitor_SMD:C_0805_2012Metric_Pad1.18x1.45mm_HandSolder, B.Cu at (165.1, 120.0)
- added C28: C, Capacitor_SMD:C_0805_2012Metric_Pad1.18x1.45mm_HandSolder, B.Cu at (167.0, 127.6)
- added C29: C, Capacitor_SMD:C_0805_2012Metric_Pad1.18x1.45mm_HandSolder, B.Cu at (160.7, 121.9)
- added C30: C, Capacitor_SMD:C_0805_2012Metric_Pad1.18x1.45mm_HandSolder, B.Cu at (160.7, 127.4)
- added D4: BAV99S, Package_TO_SOT_SMD:SOT-363_SC-70-6, B.Cu at (156.8, 125.1)
- added J6: AudioJack3_Dual_Ground_Switch, Connector_Audio:Jack_3.5mm_CUI_SJ-3524-SMT_Horizontal, B.Cu at (149.2, 130.8)
- added R39: R, Resistor_SMD:R_0805_2012Metric_Pad1.20x1.40mm_HandSolder, B.Cu at (167.6, 122.3)
- added R40: R, Resistor_SMD:R_0805_2012Metric_Pad1.20x1.40mm_HandSolder, B.Cu at (170.2, 125.7)
- added R41: R, Resistor_SMD:R_0805_2012Metric_Pad1.20x1.40mm_HandSolder, B.Cu at (163.8, 123.2)
- added R42: R, Resistor_SMD:R_0805_2012Metric_Pad1.20x1.40mm_HandSolder, B.Cu at (163.8, 126.4)
- U5: footprint Package_DIP:DIP-14_W7.62mm_Socket_LongPads -> Package_SO:SOIC-14_3.9x8.7mm_P1.27mm
- U6: footprint Package_DIP:DIP-8_W7.62mm_LongPads -> Package_SO:TSSOP-8_4.4x3mm_P0.65mm
- moved REF** 186.6 mm to (240.7, 139.1)
- moved D3 119.8 mm to (189.9, 136.9), turned to -90 degrees
- moved R4 119.2 mm to (189.9, 132.5), turned to 90 degrees
- moved TP2 117.9 mm to (83.2, 68.6), turned to -90 degrees
- moved D2 114.5 mm to (186.1, 136.9), turned to -90 degrees
- moved R5 113.8 mm to (186.1, 132.5), turned to 90 degrees
- moved D1 113.5 mm to (83.2, 64.8), turned to -90 degrees
- moved R1 108.3 mm to (83.2, 60.1), turned to -90 degrees
- moved TP5 97.0 mm to (166.7, 88.9), turned to 180 degrees
- moved U3 92.1 mm to (178.4, 62.2), turned to 180 degrees
- moved R8 89.1 mm to (178.4, 65.4), turned to 0 degrees
- moved C10 88.9 mm to (174.0, 61.0), turned to 90 degrees
- moved R10 87.7 mm to (168.3, 62.2)
- moved TP4 85.5 mm to (169.3, 94.6), turned to 180 degrees
- moved R9 83.8 mm to (172.1, 62.9), turned to 90 degrees
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Connections:
- BT1 pad 1: /BATT -> /Battery/BATT__
- C11 pad 1: /BATT -> /BATT_S
- C6 pad 1: /BATT -> /Battery/BATT__
- C9 pad 1: /BATT -> /BATT_S
- D2 pad 2: /BATT -> /BATT_S
- D3 pad 2: /BATT -> /BATT_S
- J3 pad S1: (no net) -> GND
- J3 pad S2: (no net) -> GND
- J4 pad A1/B12: (no net) -> GND
- J4 pad A4/B9: (no net) -> /Battery/CHRG-VBUS
- J4 pad B1/A12: (no net) -> GND
- J4 pad B4/A9: (no net) -> /Battery/CHRG-VBUS
- L1 pad 2: /BATT -> /BATT_S
- L2 pad 1: /BATT -> /BATT_S
- Module1 pad 46: unconnected-(Module1-Pad46) -> /IO/AUX_L
- Module1 pad 48: unconnected-(Module1-Pad48) -> /IO/AUX_R
- R11 pad 1: /BATT -> /BATT_S
- R12 pad 1: /BATT -> /BATT_S
- R17 pad 2: /Buttons/_BATT+ -> /BATT_S
- R19 pad 2: /Buttons/_BATT+ -> /BATT_S
- R9 pad 1: /BATT -> /Battery/BATT__
- U2 pad 13_14: /BATT -> /Battery/BATT__
- U2 pad 15_16: /BATT -> /BATT_S
- U3 pad 6: /BATT -> /Battery/BATT__
- U4 pad 1: /BATT -> /BATT_S
- U5 pad 14: /Buttons/_BATT+ -> /BATT_S
Other:
- board text added: "Hack the planet!"
