File: boardDesigns/CM4Carrier/heiarchy/battery.kicad_sch (KiCad schematic)
At the start: 33 parts, among them U2 MAX77751, U3 MAX17261xxTD, U4 MIC2877

Commit message: rev1
Other:
- note added: "Replace with 10k resist"
Changed lines of the file:
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@@
   (title_block
     (title "Battery / Power")
-    (date "2022-04-23")
-    (rev "Rev1-Pre")
+    (date "2022-05-14")
+    (rev "Rev1")
     (comment 1 "https://github.com/cinnamondev/gamepithing")
   )
@@
     (effects (font (size 1.27 1.27)) (justify left bottom))
   )
+  (text "Replace with 10k resist" (at 140.335 149.225 0)
+    (effects (font (size 1.27 1.27)) (justify left bottom))
+  )

Commit message: some fixes....
small details, should not affect assembly
Parts:
- R10: value 400k -> 200k
- R7: value R -> 8.06k
- R9: value 600k -> 300k
Other:
- note removed: "TBD: BATTERY MONITOR!!!"
Changed lines of the file:
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@@
     (effects (font (size 1.27 1.27)) (justify left bottom))
-  )
-  (text "TBD: BATTERY MONITOR!!!" (at 2.54 113.03 0)
-    (effects (font (size 2.54 2.54)) (justify left bottom))
   )
   (text "radio 6:4\noutput is 40pc\n" (at 107.95 118.11 0)
@@
       (effects (font (size 1.27 1.27)) (justify left))
     )
-    (property "Value" "R" (id 1) (at 90.17 82.5499 0)
+    (property "Value" "8.06k" (id 1) (at 90.17 82.5499 0)
       (effects (font (size 1.27 1.27)) (justify left))
     )
@@
       (effects (font (size 1.27 1.27)) (justify left))
     )
-    (property "Value" "400k" (id 1) (at 129.54 120.6499 0)
+    (property "Value" "200k" (id 1) (at 129.54 120.6499 0)
       (effects (font (size 1.27 1.27)) (justify left))
     )
@@
     (in_bom yes) (on_board yes) (fields_autoplaced)
     (property "Reference" "R9" (id 0) (at 121.92 105.41 90))
-    (property "Value" "600k" (id 1) (at 121.92 107.95 90))
+    (property "Value" "300k" (id 1) (at 121.92 107.95 90))
     (property "Footprint" "Resistor_SMD:R_0603_1608Metric_Pad0.98x0.95mm_HandSolder" (id 2) (at 121.92 113.538 90)
       (effects (font (size 1.27 1.27)) hide)
