File: boardDesigns/CM4Carrier/heiarchy/io.kicad_sch (KiCad schematic)
At the start: 20 parts, among them J1 Micro_SD_Card, J6 AudioJack3_Dual_Ground_Switch, U1 MIC2025-2YMM

Commit message: rev1
Connections:
- net SHOULDERL: now reaches Module1.24 (GPIO26)
- net SHOULDERL2: now reaches Module1.34 (GPIO5)
- net SHOULDERR2: now reaches Module1.50 (GPIO17)
- net SHOULDERR: now reaches Module1.58 (GPIO2)
- net 1v8: no longer names the net of Module1.88 (+1.8v_(Output))
- net 1v8: no longer Module1.90 (+1.8v_(Output))
- no-connect marks 39 -> 37
Changed lines of the file:
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@@
   (paper "A4")
   (title_block
-    (date "2022-04-23")
-    (rev "Rev1-Pre")
+    (date "2022-05-14")
+    (rev "Rev1")
     (comment 1 "https://github.com/cinnamondev/gamepithing")
   )
@@
   (junction (at 124.46 67.31) (diameter 0) (color 0 0 0 0)
   )
-  (junction (at 45.72 171.45) (diameter 0) (color 0 0 0 0)
-  )
   (junction (at 45.72 166.37) (diameter 0) (color 0 0 0 0)
   )
@@
   (junction (at 40.64 113.03) (diameter 0) (color 0 0 0 0)
   )
+  (no_connect (at 45.72 173.99))
+  (no_connect (at 45.72 171.45))
   (no_connect (at 45.72 146.05))
   (no_connect (at 45.72 148.59))
@@
   (no_connect (at 45.72 179.07))
   (no_connect (at 45.72 176.53))
-  (no_connect (at 45.72 133.35))
   (no_connect (at 45.72 130.81))
   (no_connect (at 106.68 176.53))
@@
   (no_connect (at 45.72 95.25))
   (no_connect (at 45.72 97.79))
-  (no_connect (at 45.72 102.87))
   (no_connect (at 45.72 64.77))
   (no_connect (at 45.72 67.31))
@@
   (no_connect (at 45.72 82.55))
   (no_connect (at 45.72 85.09))
-  (no_connect (at 45.72 90.17))
   (no_connect (at 45.72 92.71))
-  (no_connect (at 45.72 123.19))
   (wire (pts (xy 124.46 87.63) (xy 106.68 87.63))
     (stroke (width 0) (type default) (color 0 0 0 0))
@@
     (stroke (width 0) (type default) (color 0 0 0 0))
   )
-  (wire (pts (xy 45.72 171.45) (xy 45.72 173.99))
-    (stroke (width 0) (type default) (color 0 0 0 0))
-  )
   (wire (pts (xy 220.98 48.26) (xy 220.98 49.53))
     (stroke (width 0) (type default) (color 0 0 0 0))
@@
     (stroke (width 0) (type solid) (color 0 0 0 0))
   )
+  (wire (pts (xy 29.21 102.87) (xy 45.72 102.87))
+    (stroke (width 0) (type default) (color 0 0 0 0))
+  )
   (wire (pts (xy 34.29 166.37) (xy 45.72 166.37))
     (stroke (width 0) (type default) (color 0 0 0 0))
@@
     (stroke (width 0) (type default) (color 0 0 0 0))
   )
+  (wire (pts (xy 29.21 123.19) (xy 45.72 123.19))
+    (stroke (width 0) (type default) (color 0 0 0 0))
+  )
   (wire (pts (xy 153.67 102.87) (xy 161.29 102.87))
     (stroke (width 0) (type default) (color 0 0 0 0))
@@
     (stroke (width 0) (type default) (color 0 0 0 0))
   )
-  (wire (pts (xy 34.29 171.45) (xy 45.72 171.45))
-    (stroke (width 0) (type default) (color 0 0 0 0))
-  )
   (wire (pts (xy 218.44 48.26) (xy 220.98 48.26))
     (stroke (width 0) (type default) (color 0 0 0 0))
@@
   )
   (wire (pts (xy 106.68 97.79) (xy 113.03 97.79))
+    (stroke (width 0) (type default) (color 0 0 0 0))
+  )
+  (wire (pts (xy 29.21 133.35) (xy 45.72 133.35))
+    (stroke (width 0) (type default) (color 0 0 0 0))
+  )
+  (wire (pts (xy 29.21 90.17) (xy 45.72 90.17))
     (stroke (width 0) (type default) (color 0 0 0 0))
   )
@@
     (effects (font (size 1.27 1.27)) (justify left bottom))
   )
-  (label "1v8" (at 34.29 171.45 0)
-    (effects (font (size 1.27 1.27)) (justify left bottom))
-  )
   (label "SD_DAT3" (at 121.92 138.43 180)
     (effects (font (size 1.27 1.27)) (justify right bottom))
@@
     (effects (font (size 1.27 1.27)) (justify right))
   )
+  (hierarchical_label "SHOULDERL" (shape output) (at 29.21 90.17 180)
+    (effects (font (size 1.27 1.27)) (justify right))
+  )
   (hierarchical_label "B" (shape input) (at 113.03 130.81 0)
     (effects (font (size 1.27 1.27)) (justify left))
@@
     (effects (font (size 1.27 1.27)) (justify right))
   )
+  (hierarchical_label "SHOULDERR" (shape output) (at 29.21 133.35 180)
+    (effects (font (size 1.27 1.27)) (justify right))
+  )
   (hierarchical_label "GLOBAL_EN" (shape input) (at 113.03 186.69 0)
     (effects (font (size 1.27 1.27)) (justify left))
@@
     (effects (font (size 1.27 1.27)) (justify left))
   )
+  (hierarchical_label "SHOULDERR2" (shape output) (at 29.21 123.19 180)
+    (effects (font (size 1.27 1.27)) (justify right))
+  )
+  (hierarchical_label "SHOULDERL2" (shape output) (at 29.21 102.87 180)
+    (effects (font (size 1.27 1.27)) (justify right))
+  )
   (hierarchical_label "ADC_CS'" (shape output) (at 124.46 110.49 0)

Commit message: some fixes....
small details, should not affect assembly
Parts:
- C27, C28: value C -> 33n
- C29: value C -> 10u
- R39, R40: value R -> 270
- R41, R42: value R -> 150
- U1: value MIC2025-2YMM -> MIC2025-1YMM
Connections:
- net GND: now also R41.2, R42.2; no longer C29.2, C30.2
- net at D4.3 (K1A2), J6.R, R41.1: now also C29.2; no longer C29.1
- net at C27.1, R39.1: now also C29.1; no longer R41.2
- net at D4.6 (K3A4), J6.T, R42.1: now also C30.2; no longer C30.1
- net at C28.1, R40.1: now also C30.1; no longer R42.2
Other:
- note added: "ASSEMBLY NOTICE FOR REV1 OF THE BOARD: These have been placed incorrectly swap these pairs: (R41,C29) AND (R42,C30). So where R41 is on the board, put C29 and same for R42 and C30."
- note added: "Assembly notice: Subsituted with MIC2548 a resistor in place from Pin 5 (ILIM) to GND (1kOhm)"
- note removed: "if an sd card is overcurrent... what?"
- moved on the sheet: C29, C30, R41, R42
