File: boardDesigns/shoulderLeft/shoulderButton/shoulderButton.kicad_sch (KiCad schematic)
At the start: 5 parts, among them J1 Conn_01x03_Female, SW1 SW_SPST

Commit message: shoulder button
Parts:
- SW1: footprint (none) -> pretty:SW_EVQ-P7J01P
Changed lines of the file:
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@@
       (effects (font (size 1.27 1.27)) (justify right))
     )
-    (property "Footprint" "" (id 2) (at 123.19 97.79 0)
+    (property "Footprint" "pretty:SW_EVQ-P7J01P" (id 2) (at 123.19 97.79 0)
       (effects (font (size 1.27 1.27)) hide)
     )
@@
     )
     (path "/3a7b0f08-e8ea-4f36-84e1-0496e38a4198"
-      (reference "SW1") (unit 1) (value "SW_SPST") (footprint "")
+      (reference "SW1") (unit 1) (value "SW_SPST") (footprint "pretty:SW_EVQ-P7J01P")
     )
   )

Commit message: update ouptut
Connections:
- net GND: now also SW1.1_1 (A), SW1.1_2 (A); no longer SW1.1 (A)
- net at R2.1: now also SW1.2_1 (B), SW1.2_2 (B); no longer SW1.2 (B)
Other:
- title: (none) -> Left shoulder button
Changed lines of the file:
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@@
 (kicad_sch (version 20211123) (generator eeschema)
   (paper "A4")
+  (title_block
+    (title "Left shoulder button")
+    (date "2022-05-15")
+    (rev "Rev1-F")
+    (comment 1 "https://github.com/cinnamondev/gamepithing")
+  )
   (junction (at 134.62 102.87) (diameter 0) (color 0 0 0 0)
   )
@@
   (symbol (lib_id "Switch:SW_SPST") (at 123.19 97.79 90) (unit 1)
     (in_bom yes) (on_board yes) (fields_autoplaced)
-    (property "Reference" "SW1" (id 0) (at 124.46 96.5199 90)
+    (property "Reference" "SW1" (id 0) (at 121.9199 96.52 90)
       (effects (font (size 1.27 1.27)) (justify right))
     )
-    (property "Value" "SW_SPST" (id 1) (at 124.46 99.0599 90)
+    (property "Value" "SW_SPST" (id 1) (at 124.4599 96.52 90)
       (effects (font (size 1.27 1.27)) (justify right))
     )
-    (property "Footprint" "pretty:SW_EVQ-P7J01P" (id 2) (at 123.19 97.79 0)
+    (property "Footprint" "pretty:SW_EVQ-P7J01P" (id 2) (at 129.54 97.79 0)
       (effects (font (size 1.27 1.27)) hide)
     )
@@
       (effects (font (size 1.27 1.27)) hide)
     )
-    (pin "1")
-    (pin "2")
+    (pin "1_1")
+    (pin "1_2")
+    (pin "2_2")
+    (pin "2_1")
   )
   (symbol (lib_id "Device:R") (at 134.62 85.09 0) (unit 1)
