File: boardDesigns/shoulderLeft/shoulderButton/shoulderButton.kicad_pcb (KiCad board)
At the start: 2 copper layers, 4 parts, among them J1 Conn_01x03_Female

Commit message: shoulder button
Parts:
- added REF**: MountingHole_2.7mm_M2.5, MountingHole:MountingHole_2.7mm_M2.5, F.Cu at (54.1, 53.6)
- added REF**: MountingHole_2.7mm_M2.5, MountingHole:MountingHole_2.7mm_M2.5, F.Cu at (39.2, 78.6)
- added SW1: SW_SPST, pretty:SW_EVQ-P7J01P, F.Cu at (45.0, 48.2)
- C1, R1, R2: moved to F.Cu
- J1: moved to B.Cu
- moved J1 18.7 mm to (54.8, 59.3), turned to -90 degrees
- moved R1 5.46 mm to (45.6, 56.3), turned to 180 degrees
- moved C1 3.74 mm to (41.0, 59.8)
- moved R2 3.74 mm to (41.0, 55.2)
Routing:
- net /3v3: track 28.9 -> 9.47 mm
- net Net-(C1-Pad1): track 30.9 -> 21.6 mm
- net GND: track 14.8 -> 16.9 mm
Other:
- board outline added: 22 x 35 mm

Commit message: update ouptut
Parts:
- added REF**: OSHW-Symbol_8.9x8mm_Copper, Symbol:OSHW-Symbol_8.9x8mm_Copper, F.Cu at (47.9, 72.0)
Connections:
- SW1 pad 1_1: (no net) -> GND
- SW1 pad 1_2: (no net) -> GND
- SW1 pad 2_1: (no net) -> Net-(R2-Pad1)
- SW1 pad 2_2: (no net) -> Net-(R2-Pad1)
Routing:
- net GND: track 16.9 -> 47.2 mm
- net Net-(R2-Pad1): track 0.00 -> 11.5 mm
Other:
- board text added: "For science!"

Commit message: differential impedence
Other:
- board text added: "JLCJLCJLCJLC"
- board text added: "When live gives you lemons, lemons, then lemons, lemons."
- board text removed: "For science!"
Changed lines of the file:
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@@
         (xy 0.738491 -3.397246)
       ) (layer "F.Mask") (width 0.01) (fill solid))
-    (zone (net -454661120) (net_name "") (layer "F.Mask") (hatch edge 0.508)
+    (zone (net 0) (net_name "") (layer "F.Mask") (hatch edge 0.508)
       (connect_pads (clearance 0.508))
       (min_thickness 0.254)
@@
           (xy 47.261905 68.014562)
           (xy 48.504908 68.014562)
-          (xy 48.617491 68.611754)
         )
       )
@@
   (gr_line (start 57.615988 81.561991) (end 57.615988 46.56201) (layer "Edge.Cuts") (width 0.2))
   (gr_line (start 35.616007 81.561991) (end 57.615988 81.561991) (layer "Edge.Cuts") (width 0.2))
-  (gr_text "For science!" (at 51.054 78.994) (layer "F.SilkS")
+  (gr_text "When live gives you lemons,\nlemons, then lemons, lemons." (at 48.739 63.864 -90) (layer "B.SilkS")
+    (effects (font (size 1.5 1.5) (thickness 0.3)) (justify mirror))
+  )
+  (gr_text "JLCJLCJLCJLC\n" (at 51.054 78.994) (layer "F.SilkS")
     (effects (font (size 1 1) (thickness 0.15)))
   )
