File: boardDesigns/CM4Carrier/CM4Carrier.kicad_pcb (KiCad board)
At the start: 4 copper layers, 95.9 x 83.3 mm, 149 parts, among them J1 Micro_SD_Card, J2 Conn_01x04_Female, J3 USB_A, J4 USB_C_Receptacle_USB2.0, J5 1-84952-5, J6 AudioJack3_Dual_Ground_Switch, J7 Conn_01x03_Male, SW1 SW_Push, SW10 SW_Push, SW11 SW_Push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

Commit message: rev1
Parts:
- removed the TP27 at (47.7, 104.5)
- added J8: I2C-ADC, Connector_Wire:SolderWire-0.1sqmm_1x04_P3.6mm_D0.4mm_OD1mm, F.Cu at (135.7, 138.4)
- added REF**: KiCad-Logo2_8mm_SilkScreen, Symbol:KiCad-Logo2_8mm_SilkScreen, B.Cu at (156.2, 131.9)
- SW13: footprint CM4IO:SW_PTS526_SMG15_SMTR2_LFS -> CM4IO:SW_EVQ-P7J01P
- moved R48 155.3 mm to (199.4, 64.1)
- moved R44 153.3 mm to (199.4, 60.3), turned to -90 degrees
- moved C32 152.8 mm to (196.2, 64.1), turned to -90 degrees
- moved TP26 144.4 mm to (190.5, 63.5)
- moved SW13 141.6 mm to (194.9, 58.0), turned to 180 degrees
- moved REF** 119.1 mm to (139.6, 76.1)
- moved R1 107.9 mm to (160.4, 137.0)
- moved D1 104.5 mm to (164.7, 137.0), turned to 0 degrees
- moved TP2 101.4 mm to (160.4, 133.9)
- moved J7 75.5 mm to (144.5, 62.2)
- moved R8 8.89 mm to (182.9, 67.3), turned to 180 degrees
- moved TH1 8.63 mm to (182.9, 59.9)
- moved BT1 7.24 mm to (163.5, 64.1)
- moved TP27 5.08 mm to (122.2, 113.8)
- moved R38 3.17 mm to (193.0, 65.4)
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Connections:
- C32 pad 1: /Buttons/SHOULDERR -> /bi11
- C33 pad 1: /Buttons/SHOULDERL2 -> /bi12
- C34 pad 1: /Buttons/SHOULDERR2 -> /bi13
- J7 pad 2: /Buttons/SHOULDERL -> /bi10
- Module1 pad 24: unconnected-(Module1-Pad24) -> /bi10
- Module1 pad 34: unconnected-(Module1-Pad34) -> /bi12
- Module1 pad 50: unconnected-(Module1-Pad50) -> /bi13
- Module1 pad 58: unconnected-(Module1-Pad58) -> /bi11
- Module1 pad 88: /IO/1v8 -> unconnected-(Module1-Pad88)
- Module1 pad 90: /IO/1v8 -> unconnected-(Module1-Pad90)
- R44 pad 2: /Buttons/SHOULDERR -> /bi11
- R45 pad 2: /Buttons/SHOULDERL2 -> /bi12
- R46 pad 2: /Buttons/SHOULDERR2 -> /bi13
- R48 pad 2: /Buttons/SHOULDERR -> /bi11
- R49 pad 2: /Buttons/SHOULDERL2 -> /bi12
- R50 pad 2: /Buttons/SHOULDERR2 -> /bi13
- TP26 pad 1: /Buttons/SHOULDERR -> /bi11
- TP27 pad 1: /Buttons/SHOULDERL2 -> /bi12
- TP28 pad 1: /Buttons/SHOULDERR2 -> /bi13
Routing:
- net /bi13: track 0.00 -> 87.3 mm, vias 0 -> 2
- net Net-(Module1-Pad21): track 0.00 -> 81.4 mm, vias 0 -> 3
- net /bi11: track 0.00 -> 72.7 mm, vias 0 -> 1
- net /bi12: track 0.00 -> 67.7 mm
- net Net-(R5-Pad2): track 2.56 -> 69.1 mm, vias 0 -> 2
- net Net-(R4-Pad2): track 2.65 -> 67.6 mm, vias 0 -> 2
- net Net-(BT1-Pad2): track 11.7 -> 47.0 mm
- net /bi10: track 0.00 -> 33.2 mm
- net GND: track 138.4 -> 163.0 mm, vias 67 -> 68
- net /IO/SPIO_SCLK: track 82.4 -> 104.5 mm, vias 2 -> 3
- net /IO/SPI0_CE0_N: track 100.1 -> 121.9 mm, vias 2 -> 3
- net Net-(J2-Pad2): track 4.55 -> 22.9 mm
- net /BATT_S: track 102.2 -> 118.5 mm, vias 1 -> 3
- net /Buttons/SHOULDERL2: track 13.0 -> 0.00 mm
- net /IO/SPI0_MISO: track 83.0 -> 94.1 mm
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- added copper zone on B.Cu, net /Battery/CHRG-VBUS
- added copper zone on F.Cu, net /Battery/CHRG-VBUS
- added copper zone on F.Cu, net Net-(C4-Pad2)
- added copper zone on In1.Cu, net Net-(C4-Pad2)
- added copper zone on B.Cu, net Net-(F2-Pad1)
- added copper zone on In1.Cu, net Net-(F2-Pad1)
Other:
- board text added: "Hack the planet!"
- board text added: "github.com/cinnamondev"
- board text removed: "https://github.com/cinnamondev/gamepithing"

Commit message: update ouptut
Parts:
- moved TP2 6.56 mm to (166.9, 134.9)
- moved REF** 1.86 mm to (156.5, 130.0)
Routing:
- net /3v3: track 41.4 -> 37.4 mm
- net Net-(BT1-Pad2): track 47.0 -> 49.4 mm
- net Net-(R26-Pad1): track 0.00 -> 2.19 mm
Changed lines of the file:
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@@
       (drillshape 0)
       (scaleselection 1)
-      (outputdirectory "../output/TESTmini/")
+      (outputdirectory "../output/mainboard/")
     )
   )
@@
   )
   (footprint "TestPoint:TestPoint_THTPad_1.0x1.0mm_Drill0.5mm" (layer "F.Cu")
-    (at 160.401 133.858 180)
+    (at 166.878 134.874 180)
     (descr "THT rectangular pad as test Point, square 1.0mm side length, hole diameter 0.5mm")
     (tags "test point THT pad rectangle square")
@@
     (property "Sheetname" "IO")
     (attr exclude_from_pos_files)
-    (fp_text reference "TP2" (at 0 -1.448) (layer "F.SilkS")
+    (fp_text reference "TP2" (at 0 1.778) (layer "F.SilkS")
       (effects (font (size 1 1) (thickness 0.15)))
     )
@@
     (fp_circle (center 9.6 0) (end 10.75 0) (layer "F.Fab") (width 0.1) (fill none))
     (fp_circle (center 0 0) (end 1.15 0) (layer "F.Fab") (width 0.1) (fill none))
-    (pad "1" thru_hole roundrect (at 0 0 180) (size 2.3 2.3) (drill 1.1) (layers *.Cu *.Mask) (roundrect_rratio 0.108696)
+    (pad "1" thru_hole roundrect (at 0 0 180) (size 2.3 2.3) (drill 1.1) (layers *.Cu *.Mask) (roundrect_rratio 0.108696087)
       (net 192 "/3v3") (pinfunction "Pin_1") (pintype "passive"))
     (pad "2" thru_hole circle (at 4.8 0 180) (size 2.3 2.3) (drill 1.1) (layers *.Cu *.Mask)
@@
   )
   (footprint "Symbol:KiCad-Logo2_8mm_SilkScreen" (layer "B.Cu")
-    (at 156.200107 131.891424 180)
+    (at 156.464 130.048 180)
     (descr "KiCad Logo")
     (tags "Logo KiCad")
@@
   (segment (start 170.18 126.73) (end 169.990077 126.919923) (width 0.25) (layer "F.Cu") (net 170))
   (segment (start 169.990077 126.919923) (end 165.600005 126.919923) (width 0.25) (layer "F.Cu") (net 170))
+  (segment (start 135.89 112.665) (end 134.044989 112.665) (width 0.25) (layer "F.Cu") (net 171))
+  (segment (start 134.044989 112.665) (end 133.799992 112.420003) (width 0.25) (layer "F.Cu") (net 171))
   (segment (start 196.85 106.68) (end 198.12 105.41) (width 0.2) (layer "B.Cu") (net 172))
   (segment (start 198.12 103.951) (end 197.993 103.824) (width 0.2) (layer "B.Cu") (net 172))
@@
   (segment (start 161.02 117.475) (end 162.56 117.475) (width 1.27) (layer "F.Cu") (net 192))
   (segment (start 145.304 114.935) (end 143.891 114.935) (width 1.27) (layer "F.Cu") (net 192))
+  (segment (start 165.744 136.008) (end 166.878 134.874) (width 0.508) (layer "F.Cu") (net 192))
   (segment (start 187.325 118.11) (end 187.325 116.57) (width 1.27) (layer "F.Cu") (net 192))
   (segment (start 114.550995 136.865) (end 114.301217 137.114778) (width 0.381) (layer "F.Cu") (net 192))
@@
   (segment (start 135.89 118.475) (end 135.89 119.126) (width 1.27) (layer "F.Cu") (net 192))
   (segment (start 199.39 65.135) (end 199.39 66.421) (width 0.762) (layer "F.Cu") (net 192))
-  (segment (start 162.569 133.858) (end 165.744 137.033) (width 0.508) (layer "F.Cu") (net 192))
+  (segment (start 165.744 137.033) (end 165.744 136.008) (width 0.508) (layer "F.Cu") (net 192))
   (segment (start 135.89 119.126) (end 136.652 119.888) (width 1.27) (layer "F.Cu") (net 192))
   (segment (start 143.891 114.935) (end 143.764 114.808) (width 1.27) (layer "F.Cu") (net 192))
   (segment (start 130.175 101.6) (end 131.572 101.6) (width 0.762) (layer "F.Cu") (net 192))
-  (segment (start 160.401 133.858) (end 162.569 133.858) (width 0.508) (layer "F.Cu") (net 192))
   (segment (start 113.522 123.698) (end 113.665 123.555) (width 0.508) (layer "F.Cu") (net 192))
   (segment (start 115.8825 136.865) (end 114.550995 136.865) (width 0.381) (layer "F.Cu") (net 192))
@@
   (segment (start 129.4081 130.1169) (end 129.959747 130.1169) (width 0.2) (layer "B.Cu") (net 192))
   (segment (start 187.96 112.395) (end 187.96 117.475) (width 0.762) (layer "B.Cu") (net 192))
-  (segment (start 178.435 60.325) (end 178.435 57.785) (width 0.2) (layer "F.Cu") (net 193))
-  (segment (start 175.26 63.5) (end 178.435 60.325) (width 0.2) (layer "F.Cu") (net 193))
+  (segment (start 178.308 57.277) (end 178.308 60.452) (width 0.2) (layer "F.Cu") (net 193))
+  (segment (start 178.308 60.452) (end 175.26 63.5) (width 0.2) (layer "F.Cu") (net 193))
   (via (at 175.26 63.5) (size 0.8) (drill 0.4) (layers "F.Cu" "B.Cu") (net 193))
-  (via (at 178.435 57.785) (size 0.8) (drill 0.4) (layers "F.Cu" "B.Cu") (net 193))
+  (via (at 178.308 57.277) (size 0.8) (drill 0.4) (layers "F.Cu" "B.Cu") (net 193))
+  (segment (start 186.055 67.31) (end 183.88 67.31) (width 0.762) (layer "B.Cu") (net 193))
   (segment (start 175.727863 63.5) (end 175.26 63.5) (width 0.2) (layer "B.Cu") (net 193))
-  (segment (start 165.8825 57.785) (end 163.47 60.1975) (width 0.762) (layer "B.Cu") (net 193))
-  (segment (start 183.88 67.31) (end 186.055 67.31) (width 0.762) (layer "B.Cu") (net 193))
+  (segment (start 166.3905 57.277) (end 163.47 60.1975) (width 0.762) (layer "B.Cu") (net 193))
+  (segment (start 188.595 64.77) (end 186.055 67.31) (width 0.762) (layer "B.Cu") (net 193))
   (segment (start 163.47 60.1975) (end 163.47 61.615) (width 0.762) (layer "B.Cu") (net 193))
-  (segment (start 178.435 57.785) (end 165.8825 57.785) (width 0.762) (layer "B.Cu") (net 193))
-  (segment (start 184.785 57.785) (end 178.435 57.785) (width 0.762) (layer "B.Cu") (net 193))
-  (segment (start 188.595 64.77) (end 188.595 61.595) (width 0.762) (layer "B.Cu") (net 193))
-  (segment (start 186.055 67.31) (end 188.595 64.77) (width 0.762) (layer "B.Cu") (net 193))
+  (segment (start 178.308 57.277) (end 186.944 57.277) (width 0.762) (layer "B.Cu") (net 193))
+  (segment (start 188.595 58.928) (end 188.595 64.77) (width 0.762) (layer "B.Cu") (net 193))
+  (segment (start 186.944 57.277) (end 188.595 58.928) (width 0.762) (layer "B.Cu") (net 193))
   (segment (start 176.9475 63.03) (end 176.197863 63.03) (width 0.2) (layer "B.Cu") (net 193))
   (segment (start 176.197863 63.03) (end 175.727863 63.5) (width 0.2) (layer "B.Cu") (net 193))
-  (segment (start 188.595 61.595) (end 184.785 57.785) (width 0.762) (layer "B.Cu") (net 193))
+  (segment (start 178.308 57.277) (end 166.3905 57.277) (width 0.762) (layer "B.Cu") (net 193))
   (segment (start 126.844414 132.468086) (end 125.095 134.2175) (width 0.2) (layer "B.Cu") (net 194))
   (segment (start 144.035 133.045) (end 143.367589 132.377589) (width 0.381) (layer "B.Cu") (net 194))

Commit message: differential impedence
Routing:
- net /IO B/DSI0_L1_DN1: track 49.6 -> 56.8 mm, vias 2 -> 0
- net /IO B/DSI0_L1_DP1: track 49.7 -> 53.7 mm, vias 2 -> 0
- net /IO B/DSI0_CN: track 51.0 -> 54.2 mm, vias 2 -> 0
- net /IO B/DSI0_CP: track 51.2 -> 54.2 mm, vias 2 -> 0
- net /IO B/D-: track 69.8 -> 71.6 mm
- net /bi12: track 67.7 -> 69.1 mm, vias 0 -> 2
- net Net-(Module1-Pad21): track 81.4 -> 82.4 mm, vias 3 -> 1
- net /bi13: track 87.3 -> 86.5 mm
- net /IO B/D+: track 71.7 -> 72.2 mm
Other:
- board text added: "JLCJLCJLCJLC"
- board text added: "Thank you for assuming the Party Escort Submission Position"
- board text added: "i have no idea what i'm doing beep boop!"
