File: boardDesigns/CM4Carrier/CM4Carrier.kicad_sch (KiCad schematic)
At the start: 0 parts

Commit message: rev1
Other:
- sheet IO ports: added SHOULDERL, SHOULDERL2, SHOULDERR, SHOULDERR2; removed none

Commit message: some fixes....
small details, should not affect assembly
Other:
- note removed: "TBF: HEADPHONE JACK / SOUND"
Changed lines of the file:
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@@
     (effects (font (size 1.27 1.27)) (justify left bottom))
-  )
-  (text "TBF: HEADPHONE JACK / SOUND" (at 33.02 39.37 0)
-    (effects (font (size 5.08 5.08)) (justify left bottom))
   )
   (text "Connections:\nSD Card\nButtons (Power,A,B,X,Y,Start,Sel)\nJoystick (digital)\n"
@@
     )
     (path "/1d948cd0-f6e4-4bae-aaaf-c0cfc5cdd7a9/b2cd5d1f-ca21-48bf-babb-dc1a8f95ae47"
-      (reference "C27") (unit 1) (value "C") (footprint "Capacitor_SMD:C_0805_2012Metric_Pad1.18x1.45mm_HandSolder")
+      (reference "C27") (unit 1) (value "33n") (footprint "Capacitor_SMD:C_0805_2012Metric_Pad1.18x1.45mm_HandSolder")
     )
     (path "/1d948cd0-f6e4-4bae-aaaf-c0cfc5cdd7a9/e6767d3a-d227-419d-91dc-026b3d9dac29"
-      (reference "C28") (unit 1) (value "C") (footprint "Capacitor_SMD:C_0805_2012Metric_Pad1.18x1.45mm_HandSolder")
+      (reference "C28") (unit 1) (value "33n") (footprint "Capacitor_SMD:C_0805_2012Metric_Pad1.18x1.45mm_HandSolder")
     )
     (path "/1d948cd0-f6e4-4bae-aaaf-c0cfc5cdd7a9/6f6ec9fc-4a4d-464c-abce-93b8e52dde1a"
-      (reference "C29") (unit 1) (value "C") (footprint "Capacitor_SMD:C_0805_2012Metric_Pad1.18x1.45mm_HandSolder")
+      (reference "C29") (unit 1) (value "10u") (footprint "Capacitor_SMD:C_0805_2012Metric_Pad1.18x1.45mm_HandSolder")
     )
     (path "/1d948cd0-f6e4-4bae-aaaf-c0cfc5cdd7a9/c6deeb5d-77bf-402c-b065-b32a672f9056"
@@
     )
     (path "/a75f8253-7851-4062-bd61-8fb400fa95f7/5089a053-a588-4324-9095-4e96b7bfc76c"
-      (reference "R7") (unit 1) (value "R") (footprint "Resistor_SMD:R_0603_1608Metric_Pad0.98x0.95mm_HandSolder")
+      (reference "R7") (unit 1) (value "8.06k") (footprint "Resistor_SMD:R_0603_1608Metric_Pad0.98x0.95mm_HandSolder")
     )
     (path "/a75f8253-7851-4062-bd61-8fb400fa95f7/cee89a7b-591d-45f9-bf30-d44e71dbab9c"
@@
     )
     (path "/a75f8253-7851-4062-bd61-8fb400fa95f7/eb7bd789-7322-48a8-b1a6-c541ff3e11a1"
-      (reference "R9") (unit 1) (value "600k") (footprint "Resistor_SMD:R_0603_1608Metric_Pad0.98x0.95mm_HandSolder")
+      (reference "R9") (unit 1) (value "300k") (footprint "Resistor_SMD:R_0603_1608Metric_Pad0.98x0.95mm_HandSolder")
     )
     (path "/a75f8253-7851-4062-bd61-8fb400fa95f7/deda94a4-012e-4762-8d8b-fc34005f1aa0"
-      (reference "R10") (unit 1) (value "400k") (footprint "Resistor_SMD:R_0603_1608Metric_Pad0.98x0.95mm_HandSolder")
+      (reference "R10") (unit 1) (value "200k") (footprint "Resistor_SMD:R_0603_1608Metric_Pad0.98x0.95mm_HandSolder")
     )
     (path "/a75f8253-7851-4062-bd61-8fb400fa95f7/73e10f49-b2bb-42a8-95a9-fc71580c4820"
@@
     )
     (path "/1d948cd0-f6e4-4bae-aaaf-c0cfc5cdd7a9/c4a10c80-a780-41b4-bb7f-cb081f13cb1f"
-      (reference "R39") (unit 1) (value "R") (footprint "Resistor_SMD:R_0805_2012Metric_Pad1.20x1.40mm_HandSolder")
+      (reference "R39") (unit 1) (value "270") (footprint "Resistor_SMD:R_0805_2012Metric_Pad1.20x1.40mm_HandSolder")
     )
     (path "/1d948cd0-f6e4-4bae-aaaf-c0cfc5cdd7a9/55ce97d2-9972-4d19-b3c1-506993631f1d"
-      (reference "R40") (unit 1) (value "R") (footprint "Resistor_SMD:R_0805_2012Metric_Pad1.20x1.40mm_HandSolder")
+      (reference "R40") (unit 1) (value "270") (footprint "Resistor_SMD:R_0805_2012Metric_Pad1.20x1.40mm_HandSolder")
     )
     (path "/1d948cd0-f6e4-4bae-aaaf-c0cfc5cdd7a9/20795852-5961-4a1e-a58a-e018f5fafd6c"
-      (reference "R41") (unit 1) (value "R") (footprint "Resistor_SMD:R_0805_2012Metric_Pad1.20x1.40mm_HandSolder")
+      (reference "R41") (unit 1) (value "150") (footprint "Resistor_SMD:R_0805_2012Metric_Pad1.20x1.40mm_HandSolder")
     )
     (path "/1d948cd0-f6e4-4bae-aaaf-c0cfc5cdd7a9/438822c6-6002-4506-8be6-1c0133b2e53a"
-      (reference "R42") (unit 1) (value "R") (footprint "Resistor_SMD:R_0805_2012Metric_Pad1.20x1.40mm_HandSolder")
+      (reference "R42") (unit 1) (value "150") (footprint "Resistor_SMD:R_0805_2012Metric_Pad1.20x1.40mm_HandSolder")
     )
     (path "/fbd4ebba-c181-4efc-9928-2457cd7bdbdb/13bebd33-e033-4b3d-99b8-2cb413c10c2b"
@@
     )
     (path "/1d948cd0-f6e4-4bae-aaaf-c0cfc5cdd7a9/e28a4482-9bf6-4674-8ebc-9a8bb92d1a3e"
-      (reference "U1") (unit 1) (value "MIC2025-2YMM") (footprint "Package_SO:MSOP-8_3x3mm_P0.65mm")
+      (reference "U1") (unit 1) (value "MIC2025-1YMM") (footprint "Package_SO:MSOP-8_3x3mm_P0.65mm")
     )
     (path "/a75f8253-7851-4062-bd61-8fb400fa95f7/2a3e3937-f1c9-4371-a1ef-6f37a588e608"
